File: Adlib card/Adlib.kicad_sch (KiCad schematic)
At the start: 60 parts, among them J1 CONN_01X05, P1 IRQ, P2 ADDR, Q1 2N3904, U1 74LS109, U2 74LS138, U3 74LS138, U4 74LS245, U5 74LS04, U6 YM3812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

Commit message: Adlib part
Connections:
- net +12VA: now also U8.11 (V+), U8.11 (V+), U8.11 (V+)
- net -12VA: now also U8.7 (V-), U8.7 (V-), U8.7 (V-)
