File: Mad5160.kicad_sch (KiCad schematic)
At the start: 0 parts

Commit message: Sheet 2
Other:
- added sheet Sheet_2 (Sheet2.kicad_sch)
Changed lines of the file:
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@@
 (kicad_sch (version 20230121) (generator eeschema)
   (paper "A4")
+  (sheet (at 65.405 20.32) (size 40.005 29.845) (fields_autoplaced)
+    (stroke (width 0.1524) (type solid))
+    (fill (color 0 0 0 0.0000))
+    (property "Sheetname" "Sheet_2" (at 65.405 19.6084 0)
+      (effects (font (size 1.27 1.27)) (justify left bottom))
+    )
+    (property "Sheetfile" "Sheet2.kicad_sch" (at 65.405 50.7496 0)
+      (effects (font (size 1.27 1.27)) (justify left top))
+    )
+    (instances
+      (project "Mad5160"
+        (path "/ac3c86ab-084e-42f6-87ca-c4b0142d8ff2" (page "3"))
+      )
+    )
+  )
   (sheet (at 24.765 20.32) (size 33.655 29.845) (fields_autoplaced)
     (stroke (width 0.1524) (type solid))

Commit message: Sheet 2 finished
Other:
- sheet List1 renamed Sheet 1
- sheet Sheet 1: file list1.kicad_sch -> sheet1.kicad_sch
Changed lines of the file:
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@@
     (stroke (width 0.1524) (type solid))
     (fill (color 0 0 0 0.0000))
-    (property "Sheetname" "List1" (at 24.765 19.6084 0)
+    (property "Sheetname" "Sheet 1" (at 24.765 19.6084 0)
       (effects (font (size 1.27 1.27)) (justify left bottom))
     )
-    (property "Sheetfile" "list1.kicad_sch" (at 24.765 50.7496 0)
+    (property "Sheetfile" "sheet1.kicad_sch" (at 24.765 50.7496 0)
       (effects (font (size 1.27 1.27)) (justify left top))
     )

Commit message: Working on Sheet3
Other:
- added sheet Sheet_3 (sheet3.kicad_sch)
Changed lines of the file:
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@@
+    )
+  )
+  (sheet (at 111.125 20.32) (size 41.275 29.845) (fields_autoplaced)
+    (stroke (width 0.1524) (type solid))
+    (fill (color 0 0 0 0.0000))
+    (property "Sheetname" "Sheet_3" (at 111.125 19.6084 0)
+      (effects (font (size 1.27 1.27)) (justify left bottom))
+    )
+    (property "Sheetfile" "sheet3.kicad_sch" (at 111.125 50.7496 0)
+      (effects (font (size 1.27 1.27)) (justify left top))
+    )
+    (instances
+      (project "Mad5160"
+        (path "/ac3c86ab-084e-42f6-87ca-c4b0142d8ff2" (page "4"))
+      )
     )
   )

Commit message: Sheet 4 finished
Other:
- added sheet Sheet_4 (sheet4.kicad_sch)
Changed lines of the file:
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@@
 (kicad_sch (version 20230121) (generator eeschema)
   (paper "A4")
+  (sheet (at 156.845 20.32) (size 41.91 29.845) (fields_autoplaced)
+    (stroke (width 0.1524) (type solid))
+    (fill (color 0 0 0 0.0000))
+    (property "Sheetname" "Sheet_4" (at 156.845 19.6084 0)
+      (effects (font (size 1.27 1.27)) (justify left bottom))
+    )
+    (property "Sheetfile" "sheet4.kicad_sch" (at 156.845 50.7496 0)
+      (effects (font (size 1.27 1.27)) (justify left top))
+    )
+    (instances
+      (project "Mad5160"
+        (path "/ac3c86ab-084e-42f6-87ca-c4b0142d8ff2" (page "5"))
+      )
+    )
+  )
   (sheet (at 65.405 20.32) (size 40.005 29.845) (fields_autoplaced)
     (stroke (width 0.1524) (type solid))

Commit message: Sheet 5 symbols
Other:
- added sheet Sheet_5 (sheet5.kicad_sch)
Changed lines of the file:
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@@
+    )
+  )
+  (sheet (at 202.565 20.32) (size 42.545 29.845) (fields_autoplaced)
+    (stroke (width 0.1524) (type solid))
+    (fill (color 0 0 0 0.0000))
+    (property "Sheetname" "Sheet_5" (at 202.565 19.6084 0)
+      (effects (font (size 1.27 1.27)) (justify left bottom))
+    )
+    (property "Sheetfile" "sheet5.kicad_sch" (at 202.565 50.7496 0)
+      (effects (font (size 1.27 1.27)) (justify left top))
+    )
+    (instances
+      (project "Mad5160"
+        (path "/ac3c86ab-084e-42f6-87ca-c4b0142d8ff2" (page "6"))
+      )
     )
   )

Commit message: Working on sheet 6
Other:
- added sheet Sheet_6 (sheet6.kicad_sch)
Changed lines of the file:
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@@
+    )
+  )
+  (sheet (at 24.765 71.12) (size 34.29 27.305) (fields_autoplaced)
+    (stroke (width 0.1524) (type solid))
+    (fill (color 0 0 0 0.0000))
+    (property "Sheetname" "Sheet_6" (at 24.765 70.4084 0)
+      (effects (font (size 1.27 1.27)) (justify left bottom))
+    )
+    (property "Sheetfile" "sheet6.kicad_sch" (at 24.765 99.0096 0)
+      (effects (font (size 1.27 1.27)) (justify left top))
+    )
+    (instances
+      (project "Mad5160"
+        (path "/ac3c86ab-084e-42f6-87ca-c4b0142d8ff2" (page "7"))
+      )
     )
   )

Commit message: Sheet 7
Other:
- added sheet Sheet_7 (sheet7.kicad_sch)
Changed lines of the file:
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@@
+    )
+  )
+  (sheet (at 65.405 71.12) (size 40.005 26.67) (fields_autoplaced)
+    (stroke (width 0.1524) (type solid))
+    (fill (color 0 0 0 0.0000))
+    (property "Sheetname" "Sheet_7" (at 65.405 70.4084 0)
+      (effects (font (size 1.27 1.27)) (justify left bottom))
+    )
+    (property "Sheetfile" "sheet7.kicad_sch" (at 65.405 98.3746 0)
+      (effects (font (size 1.27 1.27)) (justify left top))
+    )
+    (instances
+      (project "Mad5160"
+        (path "/ac3c86ab-084e-42f6-87ca-c4b0142d8ff2" (page "8"))
+      )
     )
   )

Commit message: Sheet 8 finished
Other:
- added sheet Sheet_8 (sheet8.kicad_sch)
Changed lines of the file:
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@@
+    )
+  )
+  (sheet (at 110.49 71.12) (size 41.91 26.67) (fields_autoplaced)
+    (stroke (width 0.1524) (type solid))
+    (fill (color 0 0 0 0.0000))
+    (property "Sheetname" "Sheet_8" (at 110.49 70.4084 0)
+      (effects (font (size 1.27 1.27)) (justify left bottom))
+    )
+    (property "Sheetfile" "sheet8.kicad_sch" (at 110.49 98.3746 0)
+      (effects (font (size 1.27 1.27)) (justify left top))
+    )
+    (instances
+      (project "Mad5160"
+        (path "/ac3c86ab-084e-42f6-87ca-c4b0142d8ff2" (page "9"))
+      )
     )
   )
