File: Mad5160.kicad_sch (KiCad schematic)
At the start: 0 parts

Commit message: Sheet 9 finished, almost there
Other:
- added sheet Sheet_10 (sheet10.kicad_sch)
- added sheet Sheet_9 (sheet9.kicad_sch)
Changed lines of the file:
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@@
+    )
+  )
+  (sheet (at 156.845 71.12) (size 41.91 26.67) (fields_autoplaced)
+    (stroke (width 0.1524) (type solid))
+    (fill (color 0 0 0 0.0000))
+    (property "Sheetname" "Sheet_9" (at 156.845 70.4084 0)
+      (effects (font (size 1.27 1.27)) (justify left bottom))
+    )
+    (property "Sheetfile" "sheet9.kicad_sch" (at 156.845 98.3746 0)
+      (effects (font (size 1.27 1.27)) (justify left top))
+    )
+    (instances
+      (project "Mad5160"
+        (path "/ac3c86ab-084e-42f6-87ca-c4b0142d8ff2" (page "10"))
+      )
     )
   )
@@
       )
     )
+  )
+  (sheet (at 201.93 71.12) (size 43.18 26.67) (fields_autoplaced)
+    (stroke (width 0.1524) (type solid))
+    (fill (color 0 0 0 0.0000))
+    (property "Sheetname" "Sheet_10" (at 201.93 70.4084 0)
+      (effects (font (size 1.27 1.27)) (justify left bottom))
+    )
+    (property "Sheetfile" "sheet10.kicad_sch" (at 201.93 98.3746 0)
+      (effects (font (size 1.27 1.27)) (justify left top))
+    )
+    (instances
+      (project "Mad5160"
+        (path "/ac3c86ab-084e-42f6-87ca-c4b0142d8ff2" (page "11"))
+      )
+    )
