File: Sheet2.kicad_sch (KiCad schematic)
At the start: 0 parts

Commit message: Sheet 2 finished
Parts:
- added R4: 220, madXT_early:resistor, symbol Device:R
- added R5: 180, madXT_early:resistor, symbol Device:R
- added RN5: 4.7K, Package_DIP:DIP-16_W7.62mm, symbol Mad5150_early:Resistor_Network
- added TD1: ~, Connector_PinHeader_2.54mm:PinHeader_1x04_P2.54mm_Vertical, symbol Mad5150_early:TD2
- added U57: LS20_U57, Package_DIP:DIP-14_W7.62mm, symbol Mad5150_early:LS20_U57
- added U69: S00_U69, Package_DIP:DIP-14_W7.62mm, symbol Mad5150_early:S00_U69
- added U70: S74_U70, Package_DIP:DIP-14_W7.62mm, symbol Mad5150_early:S74_U70
- added U71: LS04_U71, Package_DIP:DIP-14_W7.62mm, symbol Mad5150_early:LS04_U71
- added U72: LS10_U72, Package_DIP:DIP-14_W7.62mm, symbol Mad5150_early:LS10_U72
- added U73: S74_U70, Package_DIP:DIP-14_W7.62mm, symbol Mad5150_early:LS74_U73
- added U74: LS00_U74, Package_DIP:DIP-14_W7.62mm, symbol Mad5150_early:LS00_U74
- added U86: S74_U70, Package_DIP:DIP-14_W7.62mm, symbol Mad5150_early:LS74_U86
- added U87: S08_U87, Package_DIP:DIP-14_W7.62mm, symbol Mad5150_early:S08_U87
- added U88: LS175, Package_DIP:DIP-16_W7.62mm, symbol Mad5150_early:LS175_U88
- added U89: LS04_U71, Package_DIP:DIP-14_W7.62mm, symbol Mad5150_early:LS04_U89
Connections:
- net CLK: now also U88.9 (Cp), U89.9
- net CLK88: now also U89.1
- net HRQDMA: now also U57.5, U73.1 (~{R})
- net I/O CHCK: now also RN5.10, U74.12, U74.8, U74.9
- net I/O CHRDY: now also RN5.2, U70.10 (~{S})
- net N.P. INSTLSW: now also U69.13
- net N.P. NPI: now also U69.12
- net RESET: now also U89.3
- net XD7: now also U86.12 (D)
- net ~{DACKOBRD}': now also U72.3
- net ~{ENABLEI/OCK}': now also U89.13
- net ~{LOCK}': now also U57.1
- net ~{PCK}': now also U72.9
- net ~{S0}': now also U57.4
- net ~{S1}': now also U57.2
- net ~{WRTNMIREG}': now also U86.11 (C)
- net ~{XIOR}': now also U72.13
- net ~{XIOW}': now also U72.1
- net ~{XMEMR}': now also U71.11
- new net: R4.1, R5.2, TD1.4 (7NS), U74.1
- new net: U73.3 (C), U74.2, U89.2
- new net: U70.13 (~{R}), U87.1, U88.11 (~{Q2})
- new net: U71.2, U88.13 (D3)
- new net: U73.2 (D), U88.15 (Q3)
- new net: U74.5, U88.7 (Q1)
- new net: U57.6, U71.1
- new net: U86.9 (Q), U87.9
- new net: TD1.1 (IN), U89.8
- new net: U72.11, U74.10, U74.11
- new net: U74.13, U89.12
- new net: U69.11, U72.10
- new net: U70.11 (C), U72.12
- new net: U70.8 (~{Q}), U87.2
- new net: U72.2, U72.6
- new net: U72.8, U87.10
- new net: U73.4 (~{S}), U73.6 (~{Q})
- new net +5V: R5.1, RN5.16, RN5.16, U70.12 (D), U86.10 (~{S})
- new net +XMEMR: U71.10, U71.5, U72.4
- new net AENBRD: U72.5, U74.4, U88.2 (Q0), U88.5 (D1)
- new net DCLK: U74.3
- new net GND: R4.2, TD1.2 (GND)
- new net HOLDA: U73.5 (Q), U88.4 (D0)
- new net NMI: U87.8
- new net RDYTODMA: U87.3
- new net RESETDRV: U71.12
- new net ~{AEN}': U88.3 (~{Q0})
- new net ~{DMAAEN}': U74.6
- new net ~{DMAWAIT}': U88.6 (~{Q1})
- new net ~{RDY}'/WAIT: U70.9 (Q), U88.12 (D2)
- new net ~{RESETDRV}': U71.13, U86.13 (~{R}), U88.1 (~{Mr}), U89.4
- new net ~{YMEMR}': U71.6
- no-connect marks 0 -> 3

Commit message: Working on Sheet3
Parts:
- removed unit 2 of U57
Other:
- moved on the sheet: U71G, U72D, U74E
Changed lines of the file:
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@@
     )
   )
-  (symbol (lib_id "Mad5150_early:LS04_U71") (at 133.35 -57.15 0) (unit 7)
-    (in_bom yes) (on_board yes) (dnp no) (fields_autoplaced)
-    (property "Reference" "U71" (at 139.7 -58.42 0)
-      (effects (font (size 1.27 1.27)) (justify left))
-    )
-    (property "Value" "LS04_U71" (at 139.7 -55.88 0)
-      (effects (font (size 1.27 1.27)) (justify left))
-    )
-    (property "Footprint" "Package_DIP:DIP-14_W7.62mm" (at 133.35 -57.15 0)
-      (effects (font (size 1.27 1.27)) hide)
-    )
-    (property "Datasheet" "http://www.ti.com/lit/gpn/sn74LS04" (at 133.35 -57.15 0)
+  (symbol (lib_id "Mad5150_early:LS04_U71") (at 154.94 -60.96 0) (unit 7)
+    (in_bom yes) (on_board yes) (dnp no) (fields_autoplaced)
+    (property "Reference" "U71" (at 161.29 -62.23 0)
+      (effects (font (size 1.27 1.27)) (justify left))
+    )
+    (property "Value" "LS04_U71" (at 161.29 -59.69 0)
+      (effects (font (size 1.27 1.27)) (justify left))
+    )
+    (property "Footprint" "Package_DIP:DIP-14_W7.62mm" (at 154.94 -60.96 0)
+      (effects (font (size 1.27 1.27)) hide)
+    )
+    (property "Datasheet" "http://www.ti.com/lit/gpn/sn74LS04" (at 154.94 -60.96 0)
       (effects (font (size 1.27 1.27)) hide)
     )
@@
     )
   )
-  (symbol (lib_id "Mad5150_early:LS00_U74") (at 226.06 -91.44 0) (unit 5)
-    (in_bom yes) (on_board yes) (dnp no) (fields_autoplaced)
-    (property "Reference" "U74" (at 232.41 -92.71 0)
-      (effects (font (size 1.27 1.27)) (justify left))
-    )
-    (property "Value" "LS00_U74" (at 232.41 -90.17 0)
-      (effects (font (size 1.27 1.27)) (justify left))
-    )
-    (property "Footprint" "Package_DIP:DIP-14_W7.62mm" (at 226.06 -91.44 0)
-      (effects (font (size 1.27 1.27)) hide)
-    )
-    (property "Datasheet" "http://www.ti.com/lit/gpn/sn74ls00" (at 226.06 -91.44 0)
+  (symbol (lib_id "Mad5150_early:LS00_U74") (at 223.52 -69.85 0) (unit 5)
+    (in_bom yes) (on_board yes) (dnp no) (fields_autoplaced)
+    (property "Reference" "U74" (at 229.87 -71.12 0)
+      (effects (font (size 1.27 1.27)) (justify left))
+    )
+    (property "Value" "LS00_U74" (at 229.87 -68.58 0)
+      (effects (font (size 1.27 1.27)) (justify left))
+    )
+    (property "Footprint" "Package_DIP:DIP-14_W7.62mm" (at 223.52 -69.85 0)
+      (effects (font (size 1.27 1.27)) hide)
+    )
+    (property "Datasheet" "http://www.ti.com/lit/gpn/sn74ls00" (at 223.52 -69.85 0)
       (effects (font (size 1.27 1.27)) hide)
     )
@@
     )
   )
-  (symbol (lib_id "Mad5150_early:LS10_U72") (at 179.07 -106.68 0) (unit 4)
-    (in_bom yes) (on_board yes) (dnp no) (fields_autoplaced)
-    (property "Reference" "U72" (at 185.42 -107.95 0)
-      (effects (font (size 1.27 1.27)) (justify left))
-    )
-    (property "Value" "LS10_U72" (at 185.42 -105.41 0)
-      (effects (font (size 1.27 1.27)) (justify left))
-    )
-    (property "Footprint" "Package_DIP:DIP-14_W7.62mm" (at 179.07 -106.68 0)
-      (effects (font (size 1.27 1.27)) hide)
-    )
-    (property "Datasheet" "http://www.ti.com/lit/gpn/sn74LS10" (at 179.07 -106.68 0)
+  (symbol (lib_id "Mad5150_early:LS10_U72") (at 176.53 -60.96 0) (unit 4)
+    (in_bom yes) (on_board yes) (dnp no) (fields_autoplaced)
+    (property "Reference" "U72" (at 182.88 -62.23 0)
+      (effects (font (size 1.27 1.27)) (justify left))
+    )
+    (property "Value" "LS10_U72" (at 182.88 -59.69 0)
+      (effects (font (size 1.27 1.27)) (justify left))
+    )
+    (property "Footprint" "Package_DIP:DIP-14_W7.62mm" (at 176.53 -60.96 0)
+      (effects (font (size 1.27 1.27)) hide)
+    )
+    (property "Datasheet" "http://www.ti.com/lit/gpn/sn74LS10" (at 176.53 -60.96 0)
       (effects (font (size 1.27 1.27)) hide)
     )
@@
         )
       )
-    )
-  )
-  (symbol (lib_id "Mad5150_early:LS20_U57") (at 356.235 -140.97 0) (unit 2)
-    (in_bom yes) (on_board yes) (dnp no) (fields_autoplaced)
-    (property "Reference" "U57" (at 356.2253 -148.59 0)
-      (effects (font (size 1.27 1.27)))
-    )
-    (property "Value" "LS20_U57" (at 356.2253 -146.05 0)
-      (effects (font (size 1.27 1.27)))
-    )
-    (property "Footprint" "Package_DIP:DIP-14_W7.62mm" (at 356.235 -140.97 0)
-      (effects (font (size 1.27 1.27)) hide)
-    )
-    (property "Datasheet" "http://www.ti.com/lit/gpn/sn74LS20" (at 356.235 -140.97 0)
-      (effects (font (size 1.27 1.27)) hide)
-    )
-    (pin "10")
-    (pin "13")
-    (pin "5")
-    (pin "8")
-    (pin "9")
-    (pin "12")
-    (pin "1")
-    (pin "6")
-    (pin "2")
-    (pin "4")
-    (pin "14")
-    (pin "7")
-    (instances
-      (project "Mad5160"
-        (path "/ac3c86ab-084e-42f6-87ca-c4b0142d8ff2/297b9b6a-a175-4c69-ab04-e1a6c5a6c538"
-          (reference "U57") (unit 2)
-        )
-      )

Commit message: Sheet 3 finished
Parts:
- removed unit 2 of U69
- removed unit 3 of U69
- removed unit 1 of U69
- renumbered TD1 to TD2
Connections:
- net +5V: now also U57.14 (VCC), U69.14 (VCC), U70.14 (VCC), U71.14 (VCC), U72.14 (VCC), U73.14 (VCC), U74.14 (VCC), U86.14 (VCC), U87.14 (VCC), U88.16 (VCC), U89.14 (VCC)
- net GND: now also U57.7 (GND), U69.7 (GND), U70.7 (GND), U71.7 (GND), U72.7 (GND), U73.7 (GND), U74.7 (GND), U86.7 (GND), U87.7 (GND), U88.8 (GND), U89.7 (GND)
Other:
- moved on the sheet: R4, R5, RN5B, RN5J, TD2, U57A, U57C, U69D, U69E, U70B, U70C, U71A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

Commit message: Sheet 4 finished
Parts:
- removed unit 2 of U71
Connections:
- net ~{DACKOBRD}' renamed ~{DA0K0BRD}'
Changed lines of the file:
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@@
     )
   )
-  (global_label "~{DACKOBRD}'" (shape input) (at 45.085 65.405 180) (fields_autoplaced)
+  (global_label "~{DA0K0BRD}'" (shape input) (at 45.085 65.405 180) (fields_autoplaced)
     (effects (font (size 1.27 1.27)) (justify right))
-    (property "Intersheetrefs" "${INTERSHEET_REFS}" (at 31.4559 65.405 0)
+    (property "Intersheetrefs" "${INTERSHEET_REFS}" (at 31.6374 65.405 0)
       (effects (font (size 1.27 1.27)) (justify right) hide)
     )
@@
         )
       )
-    )
-  )
-  (symbol (lib_id "Mad5150_early:LS04_U71") (at 132.715 -138.43 0) (unit 2)
-    (in_bom yes) (on_board yes) (dnp no) (fields_autoplaced)
-    (property "Reference" "U71" (at 132.715 -146.05 0)
-      (effects (font (size 1.27 1.27)))
-    )
-    (property "Value" "LS04_U71" (at 132.715 -143.51 0)
-      (effects (font (size 1.27 1.27)))
-    )
-    (property "Footprint" "Package_DIP:DIP-14_W7.62mm" (at 132.715 -138.43 0)
-      (effects (font (size 1.27 1.27)) hide)
-    )
-    (property "Datasheet" "http://www.ti.com/lit/gpn/sn74LS04" (at 132.715 -138.43 0)
-      (effects (font (size 1.27 1.27)) hide)
-    )
-    (pin "2")
-    (pin "9")
-    (pin "10")
-    (pin "11")
-    (pin "12")
-    (pin "13")
-    (pin "1")
-    (pin "5")
-    (pin "3")
-    (pin "4")
-    (pin "6")
-    (pin "8")
-    (pin "14")
-    (pin "7")
-    (instances
-      (project "Mad5160"
-        (path "/ac3c86ab-084e-42f6-87ca-c4b0142d8ff2/297b9b6a-a175-4c69-ab04-e1a6c5a6c538"
-          (reference "U71") (unit 2)
-        )
-      )

Commit message: Working on sheet 6
Parts:
- removed unit 1 of U86
- removed unit 5 of U89
Changed lines of the file:
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@@
-    )
-  )
-  (symbol (lib_id "Mad5150_early:LS04_U89") (at 309.245 -107.95 0) (unit 5)
-    (in_bom yes) (on_board yes) (dnp no) (fields_autoplaced)
-    (property "Reference" "U89" (at 309.245 -115.57 0)
-      (effects (font (size 1.27 1.27)))
-    )
-    (property "Value" "LS04_U71" (at 309.245 -113.03 0)
-      (effects (font (size 1.27 1.27)))
-    )
-    (property "Footprint" "Package_DIP:DIP-14_W7.62mm" (at 309.245 -107.95 0)
-      (effects (font (size 1.27 1.27)) hide)
-    )
-    (property "Datasheet" "http://www.ti.com/lit/gpn/sn74LS04" (at 309.245 -107.95 0)
-      (effects (font (size 1.27 1.27)) hide)
-    )
-    (pin "11")
-    (pin "4")
-    (pin "7")
-    (pin "6")
-    (pin "10")
-    (pin "8")
-    (pin "14")
-    (pin "2")
-    (pin "3")
-    (pin "12")
-    (pin "13")
-    (pin "1")
-    (pin "5")
-    (pin "9")
-    (instances
-      (project "Mad5160"
-        (path "/ac3c86ab-084e-42f6-87ca-c4b0142d8ff2/297b9b6a-a175-4c69-ab04-e1a6c5a6c538"
-          (reference "U89") (unit 5)
-        )
-      )
     )
   )
@@
         )
       )
-    )
-  )
-  (symbol (lib_id "Mad5150_early:LS74_U86") (at 584.835 -165.1 0) (unit 1)
-    (in_bom yes) (on_board yes) (dnp no) (fields_autoplaced)
-    (property "Reference" "U86" (at 587.0291 -173.99 0)
-      (effects (font (size 1.27 1.27)) (justify left))
-    )
-    (property "Value" "S74_U70" (at 587.0291 -171.45 0)
-      (effects (font (size 1.27 1.27)) (justify left))
-    )
-    (property "Footprint" "Package_DIP:DIP-14_W7.62mm" (at 584.835 -165.1 0)
-      (effects (font (size 1.27 1.27)) hide)
-    )
-    (property "Datasheet" "74xx/74hc_hct74.pdf" (at 584.835 -165.1 0)
-      (effects (font (size 1.27 1.27)) hide)
-    )
-    (pin "1")
-    (pin "2")
-    (pin "5")
-    (pin "6")
-    (pin "10")
-    (pin "12")
-    (pin "13")
-    (pin "8")
-    (pin "9")
-    (pin "14")
-    (pin "11")
-    (pin "7")
-    (pin "3")
-    (pin "4")
-    (instances
-      (project "Mad5160"
-        (path "/ac3c86ab-084e-42f6-87ca-c4b0142d8ff2/297b9b6a-a175-4c69-ab04-e1a6c5a6c538"
-          (reference "U86") (unit 1)
-        )
-      )

Commit message: Sheet 8 finished
Parts:
- removed unit 2 of U73
- removed unit 4 of U87
Changed lines of the file:
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@@
-    )
-  )
-  (symbol (lib_id "Mad5150_early:S08_U87") (at 269.875 -117.475 0) (unit 4)
-    (in_bom yes) (on_board yes) (dnp no) (fields_autoplaced)
-    (property "Reference" "U87" (at 269.8667 -124.46 0)
-      (effects (font (size 1.27 1.27)))
-    )
-    (property "Value" "S08_U87" (at 269.8667 -121.92 0)
-      (effects (font (size 1.27 1.27)))
-    )
-    (property "Footprint" "Package_DIP:DIP-14_W7.62mm" (at 269.875 -117.475 0)
-      (effects (font (size 1.27 1.27)) hide)
-    )
-    (property "Datasheet" "" (at 269.875 -117.475 0)
-      (effects (font (size 1.27 1.27)) hide)
-    )
-    (pin "14")
-    (pin "5")
-    (pin "11")
-    (pin "10")
-    (pin "2")
-    (pin "12")
-    (pin "4")
-    (pin "6")
-    (pin "7")
-    (pin "8")
-    (pin "3")
-    (pin "9")
-    (pin "1")
-    (pin "13")
-    (instances
-      (project "Mad5160"
-        (path "/ac3c86ab-084e-42f6-87ca-c4b0142d8ff2/297b9b6a-a175-4c69-ab04-e1a6c5a6c538"
-          (reference "U87") (unit 4)
-        )
-      )
     )
   )
@@
         )
       )
-    )
-  )
-  (symbol (lib_id "Mad5150_early:LS74_U73") (at 547.37 -145.415 0) (unit 2)
-    (in_bom yes) (on_board yes) (dnp no) (fields_autoplaced)
-    (property "Reference" "U73" (at 549.5641 -153.67 0)
-      (effects (font (size 1.27 1.27)) (justify left))
-    )
-    (property "Value" "S74_U70" (at 549.5641 -151.13 0)
-      (effects (font (size 1.27 1.27)) (justify left))
-    )
-    (property "Footprint" "Package_DIP:DIP-14_W7.62mm" (at 547.37 -145.415 0)
-      (effects (font (size 1.27 1.27)) hide)
-    )
-    (property "Datasheet" "74xx/74hc_hct74.pdf" (at 547.37 -145.415 0)
-      (effects (font (size 1.27 1.27)) hide)
-    )
-    (pin "11")
-    (pin "3")
-    (pin "4")
-    (pin "12")
-    (pin "7")
-    (pin "10")
-    (pin "14")
-    (pin "6")
-    (pin "5")
-    (pin "13")
-    (pin "8")
-    (pin "2")
-    (pin "1")
-    (pin "9")
-    (instances
-      (project "Mad5160"
-        (path "/ac3c86ab-084e-42f6-87ca-c4b0142d8ff2/297b9b6a-a175-4c69-ab04-e1a6c5a6c538"
-          (reference "U73") (unit 2)
-        )
-      )

Commit message: Sheet 9 finished, almost there
Parts:
- removed unit 1 of U70
- removed unit 4 of U71
- removed unit 3 of U89
Changed lines of the file:
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@@
-    )
-  )
-  (symbol (lib_id "Mad5150_early:LS04_U71") (at 132.715 -106.045 0) (unit 4)
-    (in_bom yes) (on_board yes) (dnp no) (fields_autoplaced)
-    (property "Reference" "U71" (at 132.715 -113.03 0)
-      (effects (font (size 1.27 1.27)))
-    )
-    (property "Value" "LS04_U71" (at 132.715 -110.49 0)
-      (effects (font (size 1.27 1.27)))
-    )
-    (property "Footprint" "Package_DIP:DIP-14_W7.62mm" (at 132.715 -106.045 0)
-      (effects (font (size 1.27 1.27)) hide)
-    )
-    (property "Datasheet" "http://www.ti.com/lit/gpn/sn74LS04" (at 132.715 -106.045 0)
-      (effects (font (size 1.27 1.27)) hide)
-    )
-    (pin "2")
-    (pin "9")
-    (pin "10")
-    (pin "11")
-    (pin "12")
-    (pin "13")
-    (pin "1")
-    (pin "5")
-    (pin "3")
-    (pin "4")
-    (pin "6")
-    (pin "8")
-    (pin "14")
-    (pin "7")
-    (instances
-      (project "Mad5160"
-        (path "/ac3c86ab-084e-42f6-87ca-c4b0142d8ff2/297b9b6a-a175-4c69-ab04-e1a6c5a6c538"
-          (reference "U71") (unit 4)
-        )
-      )
     )
   )
@@
     )
   )
-  (symbol (lib_id "Mad5150_early:LS04_U89") (at 307.975 -132.715 0) (unit 3)
-    (in_bom yes) (on_board yes) (dnp no) (fields_autoplaced)
-    (property "Reference" "U89" (at 307.975 -139.7 0)
-      (effects (font (size 1.27 1.27)))
-    )
-    (property "Value" "LS04_U71" (at 307.975 -137.16 0)
-      (effects (font (size 1.27 1.27)))
-    )
-    (property "Footprint" "Package_DIP:DIP-14_W7.62mm" (at 307.975 -132.715 0)
-      (effects (font (size 1.27 1.27)) hide)
-    )
-    (property "Datasheet" "http://www.ti.com/lit/gpn/sn74LS04" (at 307.975 -132.715 0)
-      (effects (font (size 1.27 1.27)) hide)
-    )
-    (pin "11")
-    (pin "4")
-    (pin "7")
-    (pin "6")
-    (pin "10")
-    (pin "8")
-    (pin "14")
-    (pin "2")
-    (pin "3")
-    (pin "12")
-    (pin "13")
-    (pin "1")
-    (pin "5")
-    (pin "9")
-    (instances
-      (project "Mad5160"
-        (path "/ac3c86ab-084e-42f6-87ca-c4b0142d8ff2/297b9b6a-a175-4c69-ab04-e1a6c5a6c538"
-          (reference "U89") (unit 3)
-        )
-      )
-    )
-  )
   (symbol (lib_id "Mad5150_early:LS20_U57") (at 153.67 264.16 0) (unit 3)
     (in_bom yes) (on_board yes) (dnp no) (fields_autoplaced)
@@
         )
       )
-    )
-  )
-  (symbol (lib_id "Mad5150_early:S74_U70") (at 443.865 -159.385 0) (unit 1)
-    (in_bom yes) (on_board yes) (dnp no) (fields_autoplaced)
-    (property "Reference" "U70" (at 446.0591 -167.64 0)
-      (effects (font (size 1.27 1.27)) (justify left))
-    )
-    (property "Value" "S74_U70" (at 446.0591 -165.1 0)
-      (effects (font (size 1.27 1.27)) (justify left))
-    )
-    (property "Footprint" "Package_DIP:DIP-14_W7.62mm" (at 443.865 -159.385 0)
-      (effects (font (size 1.27 1.27)) hide)
-    )
-    (property "Datasheet" "74xx/74hc_hct74.pdf" (at 443.865 -159.385 0)
-      (effects (font (size 1.27 1.27)) hide)
-    )
-    (pin "3")
-    (pin "10")
-    (pin "5")
-    (pin "1")
-    (pin "6")
-    (pin "2")
-    (pin "8")
-    (pin "9")
-    (pin "12")
-    (pin "7")
-    (pin "13")
-    (pin "4")
-    (pin "14")
-    (pin "11")
-    (instances
-      (project "Mad5160"
-        (path "/ac3c86ab-084e-42f6-87ca-c4b0142d8ff2/297b9b6a-a175-4c69-ab04-e1a6c5a6c538"
-          (reference "U70") (unit 1)
-        )
-      )

Commit message: Sheet 10 done
Parts:
- RN5: symbol Mad5150_early:Resistor_Network -> Mad5150_early:Resistor_Network_1
Changed lines of the file:
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@@
     )
   )
-  (symbol (lib_id "Mad5150_early:Resistor_Network") (at 55.88 168.275 0) (unit 10)
-    (in_bom yes) (on_board yes) (dnp no) (fields_autoplaced)
-    (property "Reference" "RN5" (at 57.15 167.005 0)
-      (effects (font (size 1.27 1.27)) (justify left))
-    )
-    (property "Value" "4.7K" (at 57.15 169.545 0)
+  (symbol (lib_id "Mad5150_early:Resistor_Network_1") (at 55.88 168.275 0) (unit 10)
+    (in_bom yes) (on_board yes) (dnp no) (fields_autoplaced)
+    (property "Reference" "RN5" (at 58.42 167.005 0)
+      (effects (font (size 1.27 1.27)) (justify left))
+    )
+    (property "Value" "4.7K" (at 58.42 169.545 0)
       (effects (font (size 1.27 1.27)) (justify left))
     )
@@
       (effects (font (size 1.27 1.27)) hide)
     )
-    (property "Datasheet" "" (at 55.88 168.275 0)
+    (property "Datasheet" "" (at 56.515 167.64 0)
       (effects (font (size 1.27 1.27)) hide)
     )
@@
     )
   )
-  (symbol (lib_id "Mad5150_early:Resistor_Network") (at 133.985 36.195 180) (unit 2)
+  (symbol (lib_id "Mad5150_early:Resistor_Network_1") (at 133.985 36.195 180) (unit 2)
     (in_bom yes) (on_board yes) (dnp no) (fields_autoplaced)
     (property "Reference" "RN5" (at 135.89 34.925 0)
@@
       (effects (font (size 1.27 1.27)) hide)
     )
-    (property "Datasheet" "" (at 133.985 36.195 0)
-      (effects (font (size 1.27 1.27)) hide)
-    )
+    (property "Datasheet" "" (at 133.35 36.83 0)
+      (effects (font (size 1.27 1.27)) hide)
+    )
