File: Sheet2.kicad_sch (KiCad schematic)
At the start: 15 parts, among them U57 LS20_U57, U69 S00_U69, U70 S74_U70, U71 LS04_U71, U72 LS10_U72, U73 S74_U70, U74 LS00_U74, U86 S74_U70, U87 S08_U87, U88 LS175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

Commit message: Tracing finished
Parts:
- R4, R5: footprint madXT_early:resistor -> mad5150:resistor
- RN5, U88: footprint Package_DIP:DIP-16_W7.62mm -> mad5150:DIP-16_W7.62mm
- TD2: footprint Connector_PinHeader_2.54mm:PinHeader_1x04_P2.54mm_Vertical -> mad5150:TD2
- U57, U69, U70, U71, U72, U73, U74, U86, U87, U89: footprint Package_DIP:DIP-14_W7.62mm -> mad5150:DIP-14_W7.62mm

Commit message: Fixing bugs
Connections:
- net +5V: no longer U70.12 (D)
- net ~{DA0K0BRD}': now also U70.12 (D)
Changed lines of the file:
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@@
   (junction (at 176.53 251.46) (diameter 0) (color 0 0 0 0)
+  )
+  (junction (at 77.47 65.405) (diameter 0) (color 0 0 0 0)
   )
   (junction (at 57.785 276.86) (diameter 0) (color 0 0 0 0)
@@
     (stroke (width 0) (type default))
   )
+  (wire (pts (xy 133.985 55.88) (xy 133.985 65.405))
+    (stroke (width 0) (type default))
+  )
   (wire (pts (xy 182.245 192.405) (xy 182.245 194.945))
     (stroke (width 0) (type default))
@@
     (stroke (width 0) (type default))
   )
-  (wire (pts (xy 153.035 55.88) (xy 158.115 55.88))
+  (wire (pts (xy 133.985 55.88) (xy 158.115 55.88))
     (stroke (width 0) (type default))
   )
@@
   )
   (wire (pts (xy 263.525 63.5) (xy 208.28 63.5))
+    (stroke (width 0) (type default))
+  )
+  (wire (pts (xy 77.47 65.405) (xy 133.985 65.405))
     (stroke (width 0) (type default))
   )
@@
         )
       )
-    )
-  )
-  (symbol (lib_id "power:+5V") (at 153.035 55.88 90) (unit 1)
-    (in_bom yes) (on_board yes) (dnp no) (fields_autoplaced)
-    (property "Reference" "#PWR023" (at 156.845 55.88 0)
-      (effects (font (size 1.27 1.27)) hide)
-    )
-    (property "Value" "+5V" (at 149.225 55.88 90)
-      (effects (font (size 1.27 1.27)) (justify left))
-    )
-    (property "Footprint" "" (at 153.035 55.88 0)
-      (effects (font (size 1.27 1.27)) hide)
-    )
-    (property "Datasheet" "" (at 153.035 55.88 0)
-      (effects (font (size 1.27 1.27)) hide)
-    )
-    (pin "1")
-    (instances
-      (project "Mad5160"
-        (path "/ac3c86ab-084e-42f6-87ca-c4b0142d8ff2/297b9b6a-a175-4c69-ab04-e1a6c5a6c538"
-          (reference "#PWR023") (unit 1)
-        )
-      )

Commit message: Fixing, fixing...
Parts:
- added U22: 74LS04, mad5150:DIP-14_W7.62mm, symbol 74xx:74LS04
- added U90: LS32_U58, mad5150:DIP-14_W7.62mm, symbol Mad5150_early:LS32_U90
Connections:
- net +5V: now also U90.14 (VCC)
- net GND: now also U90.7 (GND)
- net ~{XIOW}': now also U90.13
- net at U57.6: now also U90.9; no longer U71.1
- new net: U22.5, U90.11
- new net: U22.6, U90.10
- new net: U71.1, U90.8
- new net ~{DMACS}': U90.12
- no-connect marks 3 -> 9
Other:
- moved on the sheet: U57A, U71A

Commit message: Gerbers
Parts:
- U70: value S74_U70 -> 74S74N
- U73, U86: value S74_U70 -> 74LS74AN
Changed lines of the file:
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@@
       (effects (font (size 1.27 1.27)) (justify left))
     )
-    (property "Value" "S74_U70" (at 205.105 262.89 0)
+    (property "Value" "74S74N" (at 205.105 262.89 0)
       (effects (font (size 1.27 1.27)) (justify left))
     )
@@
       (effects (font (size 1.27 1.27)) (justify left))
     )
-    (property "Value" "S74_U70" (at 142.5291 152.4 0)
+    (property "Value" "74LS74AN" (at 142.5291 152.4 0)
       (effects (font (size 1.27 1.27)) (justify left))
     )
@@
       (effects (font (size 1.27 1.27)) (justify left))
     )
-    (property "Value" "S74_U70" (at 270.51 264.16 0)
+    (property "Value" "74LS74AN" (at 270.51 264.16 0)
       (effects (font (size 1.27 1.27)) (justify left))
     )
@@
       (effects (font (size 1.27 1.27)) (justify left))
     )
-    (property "Value" "S74_U70" (at 167.9291 52.07 0)
+    (property "Value" "74S74N" (at 167.9291 52.07 0)
       (effects (font (size 1.27 1.27)) (justify left))
     )
@@
       (effects (font (size 1.27 1.27)) (justify left))
     )
-    (property "Value" "S74_U70" (at 247.015 262.89 0)
+    (property "Value" "74LS74AN" (at 247.015 262.89 0)
       (effects (font (size 1.27 1.27)) (justify left))
     )
@@
       (effects (font (size 1.27 1.27)) (justify left))
     )
-    (property "Value" "S74_U70" (at 181.8991 114.3 0)
-      (effects (font (size 1.27 1.27)) (justify left))
-    )
+    (property "Value" "74LS74AN" (at 181.8991 114.3 0)
+      (effects (font (size 1.27 1.27)) (justify left))
+    )

Commit message: Version 1.0 fix
Connections:
- net I/O CHCK: no longer RN5.10, U74.9
- new net ~{I/O CHCK}': RN5.10, U74.9
Changed lines of the file:
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@@
     )
   )
-  (global_label "I{slash}O CHCK" (shape input) (at 45.72 161.925 180) (fields_autoplaced)
+  (global_label "~{I{slash}O CHCK}'" (shape input) (at 45.72 161.925 180) (fields_autoplaced)
     (effects (font (size 1.27 1.27)) (justify right))
-    (property "Intersheetrefs" "${INTERSHEET_REFS}" (at 33.3609 161.925 0)
+    (property "Intersheetrefs" "${INTERSHEET_REFS}" (at 32.7561 161.925 0)
       (effects (font (size 1.27 1.27)) (justify right) hide)
     )
