File: sheet1.kicad_sch (KiCad schematic)
At the start: 18 parts, among them U1 8284A, U2 LS245, U22 74LS04, U25 8259A, U3 8088, U4 8087, U5 LS373, U6 LS244, U7 LS373, U8 8288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

Commit message: Begin tracing
Parts:
- C1: footprint Capacitor_THT:DX_5R5HxxxxU_D11.5mm_P10.00mm -> madXT_early:VR
- C6, C8: footprint Capacitor_THT:C_Disc_D7.0mm_W2.5mm_P5.00mm -> madXT_early:cap_unipolar
Changed lines of the file:
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@@
       (effects (font (size 1.27 1.27)))
     )
-    (property "Footprint" "Capacitor_THT:C_Disc_D7.0mm_W2.5mm_P5.00mm" (at 180.34 51.1048 0)
+    (property "Footprint" "madXT_early:cap_unipolar" (at 180.34 51.1048 0)
       (effects (font (size 1.27 1.27)) hide)
     )
@@
       (effects (font (size 1.27 1.27)))
     )
-    (property "Footprint" "Capacitor_THT:DX_5R5HxxxxU_D11.5mm_P10.00mm" (at 102.235 85.09 0)
+    (property "Footprint" "madXT_early:VR" (at 102.235 85.09 0)
       (effects (font (size 1.27 1.27)) hide)
     )
@@
       (effects (font (size 1.27 1.27)) (justify right))
     )
-    (property "Footprint" "Capacitor_THT:C_Disc_D7.0mm_W2.5mm_P5.00mm" (at 159.0548 141.605 0)
-      (effects (font (size 1.27 1.27)) hide)
-    )
+    (property "Footprint" "madXT_early:cap_unipolar" (at 159.0548 141.605 0)
+      (effects (font (size 1.27 1.27)) hide)
+    )

Commit message: Update 03/05/2024
Parts:
- U4: footprint Package_DIP:DIP-40_W15.24mm_Socket_LongPads -> Package_DIP:DIP-40_W15.24mm_Socket
Changed lines of the file:
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@@
       (effects (font (size 1.27 1.27) bold))
     )
-    (property "Footprint" "Package_DIP:DIP-40_W15.24mm_Socket_LongPads" (at 179.705 208.28 0)
+    (property "Footprint" "Package_DIP:DIP-40_W15.24mm_Socket" (at 179.705 208.28 0)
       (effects (font (size 1.27 1.27)) hide)
     )

Commit message: Tracing finished
Parts:
- C1: footprint madXT_early:VR -> mad5150:VR
- C6, C8: footprint madXT_early:cap_unipolar -> mad5150:cap_unipolar
- R1, R2: footprint madXT_early:resistor -> mad5150:resistor
- RN1, RN5: footprint Package_DIP:DIP-16_W7.62mm -> mad5150:DIP-16_W7.62mm
- U1: footprint Package_DIP:DIP-18_W7.62mm -> mad5150:DIP-18_W7.62mm
- U2, U5, U6, U7, U8: footprint Package_DIP:DIP-20_W7.62mm -> mad5150:DIP-20_W7.62mm
- U22: footprint Package_DIP:DIP-14_W7.62mm -> mad5150:DIP-14_W7.62mm
- U25: footprint Package_DIP:DIP-28_W15.24mm -> mad5150:DIP-28_W15.24mm
- U3: footprint Package_DIP:DIP-40_W15.24mm -> mad5150:DIP-40_W15.24mm
- U4: footprint Package_DIP:DIP-40_W15.24mm_Socket -> mad5150:DIP-40_W15.24mm_Socket
- Y1: footprint Crystal:Crystal_HC49-U_Horizontal -> mad5150:Crystal_HC49-U_Horizontal

Commit message: Fixing bugs
Connections:
- net AENBRD: now also U5.1 (~{OE}), U6.1 (OEa), U7.1 (~{OE})
- net ~{AEN}': no longer U5.1 (~{OE}), U6.1 (OEa), U7.1 (~{OE})
Changed lines of the file:
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@@
   (junction (at 195.58 154.94) (diameter 0) (color 0 0 0 0)
   )
+  (junction (at 245.745 215.9) (diameter 0) (color 0 0 0 0)
+  )
   (junction (at 248.285 150.495) (diameter 0) (color 0 0 0 0)
   )
@@
   )
   (junction (at 95.25 85.09) (diameter 0) (color 0 0 0 0)
-  )
-  (junction (at 245.745 223.52) (diameter 0) (color 0 0 0 0)
   )
   (junction (at 195.58 152.4) (diameter 0) (color 0 0 0 0)
@@
     (stroke (width 0) (type default))
   )
-  (wire (pts (xy 105.41 223.52) (xy 245.745 223.52))
-    (stroke (width 0) (type default))
-  )
   (wire (pts (xy 329.565 200.66) (xy 337.82 200.66))
     (stroke (width 0) (type default))
@@
     (stroke (width 0) (type default))
   )
-  (wire (pts (xy 102.87 215.9) (xy 266.065 215.9))
+  (wire (pts (xy 102.87 215.9) (xy 245.745 215.9))
     (stroke (width 0) (type default))
   )
@@
     (stroke (width 0) (type default))
   )
-  (wire (pts (xy 245.745 147.955) (xy 245.745 223.52))
+  (wire (pts (xy 245.745 147.955) (xy 245.745 215.9))
     (stroke (width 0) (type default))
   )
@@
     (stroke (width 0) (type default))
   )
+  (wire (pts (xy 245.745 215.9) (xy 266.065 215.9))
+    (stroke (width 0) (type default))
+  )
   (wire (pts (xy 257.175 132.715) (xy 266.7 132.715))
     (stroke (width 0) (type default))
@@
     (stroke (width 0) (type default))
   )
+  (wire (pts (xy 105.41 223.52) (xy 266.065 223.52))
+    (stroke (width 0) (type default))
+  )
   (bus (pts (xy 67.31 212.725) (xy 67.31 215.265))
     (stroke (width 1) (type default))
@@
     (stroke (width 0) (type default))
   )
-  (wire (pts (xy 245.745 223.52) (xy 266.065 223.52))
-    (stroke (width 0) (type default))
-  )

Commit message: Fixing, fixing...
Parts:
- removed unit 3 of U22
Connections:
- no-connect marks 28 -> 26
Changed lines of the file:
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@@
   (no_connect (at 66.04 177.8))
   (no_connect (at 283.21 109.855))
-  (no_connect (at 213.36 268.605))
   (no_connect (at 266.7 97.155))
-  (no_connect (at 198.12 268.605))
   (no_connect (at 182.88 267.97))
   (no_connect (at 263.525 256.54))
@@
         )
       )
-    )
-  )
-  (symbol (lib_id "74xx:74LS04") (at 205.74 268.605 0) (unit 3)
-    (in_bom yes) (on_board yes) (dnp no) (fields_autoplaced)
-    (property "Reference" "U22" (at 205.74 261.62 0)
-      (effects (font (size 1.27 1.27)))
-    )
-    (property "Value" "74LS04" (at 205.74 264.16 0)
-      (effects (font (size 1.27 1.27)))
-    )
-    (property "Footprint" "mad5150:DIP-14_W7.62mm" (at 205.74 268.605 0)
-      (effects (font (size 1.27 1.27)) hide)
-    )
-    (property "Datasheet" "http://www.ti.com/lit/gpn/sn74LS04" (at 205.74 268.605 0)
-      (effects (font (size 1.27 1.27)) hide)
-    )
-    (pin "1")
-    (pin "2")
-    (pin "3")
-    (pin "4")
-    (pin "5")
-    (pin "6")
-    (pin "8")
-    (pin "9")
-    (pin "10")
-    (pin "11")
-    (pin "12")
-    (pin "13")
-    (pin "14")
-    (pin "7")
-    (instances
-      (project "Mad5160"
-        (path "/ac3c86ab-084e-42f6-87ca-c4b0142d8ff2/921209e9-21b1-4dfe-a217-0f57a16b1ecc"
-          (reference "U22") (unit 3)
-        )
-      )

Commit message: Fixing stuff
Parts:
- removed unit 1 of U22
- removed unit 2 of U22
Connections:
- no-connect marks 26 -> 22
Changed lines of the file:
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@@
   (no_connect (at 294.64 97.155))
   (no_connect (at 66.04 175.26))
-  (no_connect (at 139.7 268.605))
   (no_connect (at 266.7 102.235))
   (no_connect (at 266.7 99.695))
@@
   (no_connect (at 294.005 219.71))
   (no_connect (at 190.5 119.38))
-  (no_connect (at 154.94 268.605))
-  (no_connect (at 167.64 267.97))
   (no_connect (at 66.04 97.79))
   (no_connect (at 165.1 119.38))
@@
   (no_connect (at 283.21 109.855))
   (no_connect (at 266.7 97.155))
-  (no_connect (at 182.88 267.97))
   (no_connect (at 263.525 256.54))
   (no_connect (at 254.635 256.54))
@@
     )
   )
-  (symbol (lib_id "74xx:74LS04") (at 147.32 268.605 0) (unit 1)
-    (in_bom yes) (on_board yes) (dnp no) (fields_autoplaced)
-    (property "Reference" "U22" (at 147.32 261.62 0)
-      (effects (font (size 1.27 1.27)))
-    )
-    (property "Value" "74LS04" (at 147.32 264.16 0)
-      (effects (font (size 1.27 1.27)))
-    )
-    (property "Footprint" "mad5150:DIP-14_W7.62mm" (at 147.32 268.605 0)
-      (effects (font (size 1.27 1.27)) hide)
-    )
-    (property "Datasheet" "http://www.ti.com/lit/gpn/sn74LS04" (at 147.32 268.605 0)
-      (effects (font (size 1.27 1.27)) hide)
-    )
-    (pin "1")
-    (pin "2")
-    (pin "3")
-    (pin "4")
-    (pin "5")
-    (pin "6")
-    (pin "8")
-    (pin "9")
-    (pin "10")
-    (pin "11")
-    (pin "12")
-    (pin "13")
-    (pin "14")
-    (pin "7")
-    (instances
-      (project "Mad5160"
-        (path "/ac3c86ab-084e-42f6-87ca-c4b0142d8ff2/921209e9-21b1-4dfe-a217-0f57a16b1ecc"
-          (reference "U22") (unit 1)
-        )
-      )
-    )
-  )
   (symbol (lib_id "Mad5150_early:LS373_U7") (at 279.4 55.88 0) (unit 1)
     (in_bom yes) (on_board yes) (dnp no)
@@
         )
       )
-    )
-  )
-  (symbol (lib_id "74xx:74LS04") (at 175.26 267.97 0) (unit 2)
-    (in_bom yes) (on_board yes) (dnp no) (fields_autoplaced)
-    (property "Reference" "U22" (at 175.26 261.62 0)
-      (effects (font (size 1.27 1.27)))
-    )
-    (property "Value" "74LS04" (at 175.26 264.16 0)
-      (effects (font (size 1.27 1.27)))
-    )
-    (property "Footprint" "mad5150:DIP-14_W7.62mm" (at 175.26 267.97 0)
-      (effects (font (size 1.27 1.27)) hide)
-    )
-    (property "Datasheet" "http://www.ti.com/lit/gpn/sn74LS04" (at 175.26 267.97 0)
-      (effects (font (size 1.27 1.27)) hide)
-    )
-    (pin "1")
-    (pin "2")
-    (pin "3")
-    (pin "4")
-    (pin "5")
-    (pin "6")
-    (pin "8")
-    (pin "9")
-    (pin "10")
-    (pin "11")
-    (pin "12")
-    (pin "13")
-    (pin "14")
-    (pin "7")
-    (instances
-      (project "Mad5160"
-        (path "/ac3c86ab-084e-42f6-87ca-c4b0142d8ff2/921209e9-21b1-4dfe-a217-0f57a16b1ecc"
-          (reference "U22") (unit 2)
-        )
-      )
