File: sheet3.kicad_sch (KiCad schematic)
At the start: 7 parts, among them U24 LS00_U24, U42 LS138, U43 LS138, U45 LS138, U56 LS138, U57 LS20_U57

Commit message: Sheet 3 finished
Parts:
- added E2: E2_Jumper_block, Connector_PinHeader_2.54mm:PinHeader_2x02_P2.54mm_Vertical, symbol Mad5150_early:E2_Jumper_block
- added E3: E3 Jumper Block, Connector_PinHeader_2.54mm:PinHeader_2x04_P2.54mm_Vertical, symbol Mad5150_early:E3 Jumper Block
- added RN2: 8.2K, Package_DIP:DIP-16_W7.62mm, symbol Mad5150_early:RN2
- added RN4: 30, Package_DIP:DIP-16_W7.62mm, symbol Mad5150_early:RN4
- added TD1: TTLDL-20, Package_DIP:DIP-14_W7.62mm, symbol Mad5150_early:TTLDL-20
- added U44: 24S10, Package_DIP:DIP-16_W7.62mm, symbol Mad5150_early:24S10_U44
- added U55: S08_U55, Package_DIP:DIP-14_W7.62mm, symbol Mad5150_early:S08_U55
- added U58: LS32_U58, Package_DIP:DIP-14_W7.62mm, symbol Mad5150_early:LS32_U58
- added U69: S00_U69, Package_DIP:DIP-14_W7.62mm, symbol Mad5150_early:S00_U69
- renumbered E1 to E7
Connections:
- net A16: now also U44.5 (A0)
- net A17: now also U44.6 (A1)
- net A18: now also U44.7 (A2)
- net A19: now also U44.4 (A3)
- net DACK 0: now also U56.4 (G2A), U69.10
- net PLANAR RAM 0: now also U44.3 (A4)
- net PLANAR RAM 1: now also U44.2 (A5)
- net XA14: now also E3.5 (Pin_5)
- net XA15: now also U43.1 (A), E3.3 (Pin_3)
- net XA16: now also U43.2 (B)
- net XA17: now also U43.3 (C)
- net XA18: now also U24.2
- net XA19: now also U43.6 (G1)
- net ~{AEN}': now also U57.9
- net ~{DACK 0 BRD}': now also U24.5, U42.6 (G1)
- net ~{MEMR}': now also U57.10
- net ~{MWTC}': now also U57.12
- net ~{XIOW}': now also U58.10, U58.12
- net ~{XMEMR}': now also U43.4 (G2A), U69.4
- net ~{XMEMW}': now also U69.5
- net ~{CS5}': now reaches U43.10 (Y5)
- net ~{CS4}': now reaches U43.11 (Y4)
- net ~{CS3}': now reaches U43.12 (Y3)
- net ~{CS2}': now reaches U43.13 (Y2)
- net ~{CS1}': now reaches U43.14 (Y1)
- net ~{CS0}': now reaches U43.15 (Y0)
- net at U43.5 (G2B): now also U24.3
- net ~{CS7}': now reaches U43.7 (Y7)
- net ~{CS7}': now also U24.10
- net ~{CS6}': now reaches U43.9 (Y6)
- net ~{CS6}': now also U24.9
- net at U24.1: now also E7.2 (Pin_2), RN2.1
- net ROMADDRSEL: now reaches U24.8
- net at U42.1 (A): now also U56.1 (A), E3.6 (Pin_6), E3.8 (Pin_8)
- net ~{CAS3}': now reaches U42.12 (Y3)
- net ~{CAS2}': now reaches U42.13 (Y2)
- net ~{CAS1}': now reaches U42.14 (Y1)
- net ~{CAS0}': now reaches U42.15 (Y0)
- net at U42.2 (B): now also U56.2 (B), E3.2 (Pin_2), E3.4 (Pin_4)
- net GND: now reaches U42.3 (C)
- net GND: now also E7.1 (Pin_1), U24.7 (GND), U42.8 (GND), U43.8 (GND), U45.8 (GND), U56.8 (GND), E2.1 (Pin_1), E2.3 (Pin_3), TD1.7 (GND), U44.13 (S1), U44.14 (S2), U44.8 (GND), U55.7 (GND), U58.7 (GND)
- net ~{RAMADDRSEL}': now reaches U42.4 (G2A)
- net ~{RAMADDRSEL}': now also U24.6, U56.5 (G2B)
- net ~{CAS}: now reaches U42.5 (G2B)
- net ~{CAS}: now also U69.3
- net at U45.10 (Y5): now also U58.13
- net at U45.11 (Y4): now also U58.9
- net ~{PPICS}': now reaches U45.12 (Y3)
- net ~{T/CCS}': now reaches U45.13 (Y2)
- net ~{INTRCS}': now reaches U45.14 (Y1)
- net ~{DMACS}': now reaches U45.15 (Y0)
- net +5V: now reaches U43.16 (VCC)
- net +5V: now also U24.14 (VCC), U42.16 (VCC), U45.16 (VCC), U56.16 (VCC), U56.3 (C), U57.13, RN2.16, RN2.16, RN2.16, TD1.14 (Vcc), U44.16 (Vcc), U55.14 (VCC), U58.14 (VCC)
- net at U56.10 (Y5): now also U55.12
- net at U56.11 (Y4): now also U55.2
- net RAS: now reaches U56.6 (G1)
- net RAS: now also TD1.1 (IN), U69.6, U69.9
- net at U56.7 (Y7): now also U55.9
- net at U56.9 (Y6): now also U55.5
- net at U57.8: now also U69.1
- net at U24.4: now also U44.12 (Q0)
- new net: E3.1 (Pin_1), U44.10 (Q2)
- new net: E3.7 (Pin_7), U44.11 (Q1)
- new net: RN4.12, U55.8
- new net: E2.2 (Pin_2), RN2.6, U44.1 (A6)
- new net: RN4.11, U55.6
- new net: TD1.8 (100), U69.2
- new net: RN4.14, U55.3
- new net: RN4.13, U55.11
- new net: E2.4 (Pin_4), RN2.7, U44.15 (A7)
- new net ADDRSEL: TD1.10 (60)
- new net ~{RAS0}': RN4.3
- new net ~{RAS1}': RN4.4
- new net ~{RAS2}': RN4.6
- new net ~{RAS3}': RN4.5
- new net ~{REFRESH GATE}: U55.1, U55.10, U55.13, U55.4, U69.8
- new net ~{WRTDMAPGREG}': U58.8
- new net ~{WRTNMIREG}': U58.11
- no-connect marks 2 -> 14
Other:
- moved on the sheet: E7, U24A, U24B, U24C, U24D, U24E, U42A, U42B, U43A, U43B, U45A, U45B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

Commit message: Sheet 4 finished
Connections:
- net DACK 0 renamed DA0K0
- net ~{DACK 0 BRD}' renamed ~{DA0K0BRD}'
Changed lines of the file:
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@@
     )
   )
-  (global_label "~{DACK 0 BRD}'" (shape input) (at 29.845 130.81 180) (fields_autoplaced)
-    (effects (font (size 1.27 1.27)) (justify right))
-    (property "Intersheetrefs" "${INTERSHEET_REFS}" (at 14.4017 130.81 0)
+  (global_label "~{DA0K0BRD}'" (shape input) (at 29.845 130.81 180) (fields_autoplaced)
+    (effects (font (size 1.27 1.27)) (justify right))
+    (property "Intersheetrefs" "${INTERSHEET_REFS}" (at 16.3974 130.81 0)
       (effects (font (size 1.27 1.27)) (justify right) hide)
     )
@@
     )
   )
-  (global_label "DACK 0" (shape input) (at 28.575 184.785 180) (fields_autoplaced)
-    (effects (font (size 1.27 1.27)) (justify right))
-    (property "Intersheetrefs" "${INTERSHEET_REFS}" (at 18.5141 184.785 0)
-      (effects (font (size 1.27 1.27)) (justify right) hide)
-    )
+  (global_label "DA0K0" (shape input) (at 28.575 184.785 180) (fields_autoplaced)
+    (effects (font (size 1.27 1.27)) (justify right))
+    (property "Intersheetrefs" "${INTERSHEET_REFS}" (at 19.5422 184.785 0)
+      (effects (font (size 1.27 1.27)) (justify right) hide)
+    )

Commit message: Sheet 5 symbols
Parts:
- removed unit 4 of U24
Changed lines of the file:
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@@
-    )
-  )
-  (symbol (lib_id "Mad5150_early:LS00_U24") (at 50.8 -88.265 0) (unit 4)
-    (in_bom yes) (on_board yes) (dnp no) (fields_autoplaced)
-    (property "Reference" "U24" (at 50.7917 -95.25 0)
-      (effects (font (size 1.27 1.27)))
-    )
-    (property "Value" "LS00_U24" (at 50.7917 -92.71 0)
-      (effects (font (size 1.27 1.27)))
-    )
-    (property "Footprint" "Package_DIP:DIP-14_W7.62mm" (at 50.8 -88.265 0)
-      (effects (font (size 1.27 1.27)) hide)
-    )
-    (property "Datasheet" "http://www.ti.com/lit/gpn/sn74ls00" (at 50.8 -88.265 0)
-      (effects (font (size 1.27 1.27)) hide)
-    )
-    (pin "1")
-    (pin "3")
-    (pin "4")
-    (pin "8")
-    (pin "13")
-    (pin "5")
-    (pin "14")
-    (pin "6")
-    (pin "10")
-    (pin "9")
-    (pin "11")
-    (pin "12")
-    (pin "7")
-    (pin "2")
-    (instances
-      (project "Mad5160"
-        (path "/ac3c86ab-084e-42f6-87ca-c4b0142d8ff2/66db5a8e-229f-48cb-8657-576a3a35aa17"
-          (reference "U24") (unit 4)
-        )
-      )
     )
   )

Commit message: Working on sheet 6
Parts:
- removed unit 2 of RN4
- removed unit 1 of U58
Changed lines of the file:
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@@
-    )
-  )
-  (symbol (lib_id "Mad5150_early:RN4") (at 77.47 -148.59 0) (unit 2)
-    (in_bom yes) (on_board yes) (dnp no) (fields_autoplaced)
-    (property "Reference" "RN4" (at 80.01 -149.86 0)
-      (effects (font (size 1.27 1.27)) (justify left))
-    )
-    (property "Value" "30" (at 80.01 -147.32 0)
-      (effects (font (size 1.27 1.27)) (justify left))
-    )
-    (property "Footprint" "Package_DIP:DIP-16_W7.62mm" (at 77.47 -148.59 0)
-      (effects (font (size 1.27 1.27)) hide)
-    )
-    (property "Datasheet" "" (at 78.105 -149.225 0)
-      (effects (font (size 1.27 1.27)) hide)
-    )
-    (pin "3")
-    (pin "9")
-    (pin "15")
-    (pin "4")
-    (pin "12")
-    (pin "2")
-    (pin "10")
-    (pin "7")
-    (pin "8")
-    (pin "11")
-    (pin "13")
-    (pin "1")
-    (pin "6")
-    (pin "16")
-    (pin "5")
-    (pin "14")
-    (instances
-      (project "Mad5160"
-        (path "/ac3c86ab-084e-42f6-87ca-c4b0142d8ff2/66db5a8e-229f-48cb-8657-576a3a35aa17"
-          (reference "RN4") (unit 2)
-        )
-      )
     )
   )
@@
         )
       )
-    )
-  )
-  (symbol (lib_id "Mad5150_early:LS32_U58") (at 193.675 -130.175 0) (unit 1)
-    (in_bom yes) (on_board yes) (dnp no) (fields_autoplaced)
-    (property "Reference" "U58" (at 193.675 -137.16 0)
-      (effects (font (size 1.27 1.27)))
-    )
-    (property "Value" "LS32_U58" (at 193.675 -134.62 0)
-      (effects (font (size 1.27 1.27)))
-    )
-    (property "Footprint" "Package_DIP:DIP-14_W7.62mm" (at 193.675 -130.175 0)
-      (effects (font (size 1.27 1.27)) hide)
-    )
-    (property "Datasheet" "http://www.ti.com/lit/gpn/sn74LS32" (at 193.675 -130.175 0)
-      (effects (font (size 1.27 1.27)) hide)
-    )
-    (pin "11")
-    (pin "5")
-    (pin "14")
-    (pin "3")
-    (pin "10")
-    (pin "13")
-    (pin "6")
-    (pin "9")
-    (pin "12")
-    (pin "2")
-    (pin "7")
-    (pin "8")
-    (pin "4")
-    (pin "1")
-    (instances
-      (project "Mad5160"
-        (path "/ac3c86ab-084e-42f6-87ca-c4b0142d8ff2/66db5a8e-229f-48cb-8657-576a3a35aa17"
-          (reference "U58") (unit 1)
-        )
-      )

Commit message: Sheet 7
Parts:
- removed unit 1 of RN4
Changed lines of the file:
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@@
-    )
-  )
-  (symbol (lib_id "Mad5150_early:RN4") (at 66.675 -147.955 0) (unit 1)
-    (in_bom yes) (on_board yes) (dnp no) (fields_autoplaced)
-    (property "Reference" "RN4" (at 68.58 -149.225 0)
-      (effects (font (size 1.27 1.27)) (justify left))
-    )
-    (property "Value" "30" (at 68.58 -146.685 0)
-      (effects (font (size 1.27 1.27)) (justify left))
-    )
-    (property "Footprint" "Package_DIP:DIP-16_W7.62mm" (at 66.675 -147.955 0)
-      (effects (font (size 1.27 1.27)) hide)
-    )
-    (property "Datasheet" "" (at 67.31 -148.59 0)
-      (effects (font (size 1.27 1.27)) hide)
-    )
-    (pin "3")
-    (pin "9")
-    (pin "15")
-    (pin "4")
-    (pin "12")
-    (pin "2")
-    (pin "10")
-    (pin "7")
-    (pin "8")
-    (pin "11")
-    (pin "13")
-    (pin "1")
-    (pin "6")
-    (pin "16")
-    (pin "5")
-    (pin "14")
-    (instances
-      (project "Mad5160"
-        (path "/ac3c86ab-084e-42f6-87ca-c4b0142d8ff2/66db5a8e-229f-48cb-8657-576a3a35aa17"
-          (reference "RN4") (unit 1)
-        )
-      )
     )
   )

Commit message: Sheet 9 finished, almost there
Parts:
- removed unit 9 of RN2
- removed unit 13 of RN2
- removed unit 5 of RN2
- removed unit 4 of RN2
- removed unit 10 of RN2
- removed unit 2 of RN2
- removed unit 3 of RN2
- removed unit 12 of RN2
- removed unit 11 of RN2

Commit message: Sheet 10 done
Connections:
- net +5V: now also RN2.16, RN2.16, RN2.16
- no-connect marks 14 -> 24
Changed lines of the file:
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@@
   (junction (at 55.245 177.165) (diameter 0) (color 0 0 0 0)
   )
+  (no_connect (at 185.42 -114.3))
+  (no_connect (at -47.625 -113.665))
+  (no_connect (at 137.795 -144.145))
   (no_connect (at 163.83 83.185))
   (no_connect (at 144.145 120.65))
   (no_connect (at 99.695 33.655))
+  (no_connect (at -31.115 -94.615))
   (no_connect (at 94.615 123.19))
   (no_connect (at 94.615 118.11))
@@
   (no_connect (at 144.145 123.19))
   (no_connect (at 94.615 120.65))
+  (no_connect (at 185.42 -119.38))
   (no_connect (at 93.98 76.835))
+  (no_connect (at 137.795 -155.575))
+  (no_connect (at 149.86 -155.575))
   (no_connect (at 94.615 115.57))
   (no_connect (at 144.145 128.27))
+  (no_connect (at 200.66 -116.84))
   (no_connect (at 144.145 125.73))
   (no_connect (at 168.91 83.185))
   (no_connect (at 161.29 83.185))
+  (no_connect (at 149.86 -144.145))
+  (no_connect (at -17.145 -95.25))
   (bus_entry (at 196.215 165.735) (size 2.54 -2.54)
     (stroke (width 0) (type default))
@@
     (stroke (width 0) (type default))
   )
+  (wire (pts (xy 59.055 133.35) (xy 118.745 133.35))
+    (stroke (width 0) (type default))
+  )
   (wire (pts (xy 30.48 71.755) (xy 69.85 71.755))
     (stroke (width 0) (type default))
@@
   )
   (wire (pts (xy 98.425 137.16) (xy 98.425 101.6))
-    (stroke (width 0) (type default))
-  )
-  (wire (pts (xy 119.38 133.35) (xy 59.055 133.35))
     (stroke (width 0) (type default))
   )
@@
     (effects (font (size 1.27 1.27)) (justify left bottom))
   )
+  (label "~{CS1}'" (at 260.35 142.24 0) (fields_autoplaced)
+    (effects (font (size 1.27 1.27)) (justify left bottom))
+  )
   (label "~{CS5}'" (at 95.25 155.575 0) (fields_autoplaced)
     (effects (font (size 1.27 1.27)) (justify left bottom))
@@
     (effects (font (size 1.27 1.27)) (justify left bottom))
   )
+  (label "~{CS4}'" (at 260.35 149.86 0) (fields_autoplaced)
+    (effects (font (size 1.27 1.27)) (justify left bottom))
+  )
   (label "~{CS7}'" (at 204.47 163.195 0) (fields_autoplaced)
     (effects (font (size 1.27 1.27)) (justify left bottom))
@@
     (effects (font (size 1.27 1.27)) (justify left bottom))
   )
+  (label "~{CS5}'" (at 260.35 152.4 0) (fields_autoplaced)
+    (effects (font (size 1.27 1.27)) (justify left bottom))
+  )
   (label "~{CS0}'" (at 95.25 142.875 0) (fields_autoplaced)
     (effects (font (size 1.27 1.27)) (justify left bottom))
@@
     (effects (font (size 1.27 1.27)) (justify left bottom))
   )
+  (label "~{CS0}'" (at 260.35 139.7 0) (fields_autoplaced)
+    (effects (font (size 1.27 1.27)) (justify left bottom))
+  )
   (label "~{CS3}'" (at 95.25 150.495 0) (fields_autoplaced)
     (effects (font (size 1.27 1.27)) (justify left bottom))
@@
     (effects (font (size 1.27 1.27)) (justify left bottom))
   )
+  (label "~{CS3}'" (at 260.35 147.32 0) (fields_autoplaced)
+    (effects (font (size 1.27 1.27)) (justify left bottom))
+  )
   (label "~{REFRESH GATE}" (at 148.59 160.02 0) (fields_autoplaced)
     (effects (font (size 1.27 1.27)) (justify left bottom))
@@
     (effects (font (size 1.27 1.27)) (justify left bottom))
   )
+  (label "~{CS6}'" (at 260.35 154.94 0) (fields_autoplaced)
+    (effects (font (size 1.27 1.27)) (justify left bottom))
+  )
   (label "~{CS2}'" (at 95.25 147.955 0) (fields_autoplaced)
+    (effects (font (size 1.27 1.27)) (justify left bottom))
+  )
+  (label "~{CS2}'" (at 260.35 144.78 0) (fields_autoplaced)
+    (effects (font (size 1.27 1.27)) (justify left bottom))
+  )
+  (label "~{CS7}'" (at 260.35 157.48 0) (fields_autoplaced)
     (effects (font (size 1.27 1.27)) (justify left bottom))
   )
@@
     )
   )
-  (symbol (lib_name "LS138_U43_1") (lib_id "Mad5150_early:LS138_U43") (at 81.915 150.495 0) (unit 1)
+  (symbol (lib_id "Mad5150_early:LS138_U43") (at 81.915 150.495 0) (unit 1)
     (in_bom yes) (on_board yes) (dnp no)
     (property "Reference" "U43" (at 81.915 149.225 0)
@@
     )
   )
-  (symbol (lib_name "LS138_U42_1") (lib_id "Mad5150_early:LS138_U42") (at 81.915 113.03 0) (unit 1)
+  (symbol (lib_id "Mad5150_early:LS138_U42") (at 81.915 113.03 0) (unit 1)
     (in_bom yes) (on_board yes) (dnp no)
     (property "Reference" "U42" (at 81.915 109.22 0)
@@
     )
   )
-  (symbol (lib_name "LS138_U45_1") (lib_id "Mad5150_early:LS138_U45") (at 86.995 23.495 0) (unit 1)
+  (symbol (lib_id "Mad5150_early:LS138_U45") (at 86.995 23.495 0) (unit 1)
     (in_bom yes) (on_board yes) (dnp no)
     (property "Reference" "U45" (at 86.995 19.685 0)
@@
     )
   )
+  (symbol (lib_id "power:+5V") (at -47.625 -102.235 180) (unit 1)
+    (in_bom yes) (on_board yes) (dnp no)
+    (property "Reference" "#PWR0250" (at -47.625 -106.045 0)
+      (effects (font (size 1.27 1.27)) hide)
+    )
+    (property "Value" "+5V" (at -47.625 -98.425 0)
+      (effects (font (size 1.27 1.27)))
+    )
+    (property "Footprint" "" (at -47.625 -102.235 0)
+      (effects (font (size 1.27 1.27)) hide)
+    )
+    (property "Datasheet" "" (at -47.625 -102.235 0)
+      (effects (font (size 1.27 1.27)) hide)
+    )
+    (pin "1")
+    (instances
+      (project "Mad5160"
+        (path "/ac3c86ab-084e-42f6-87ca-c4b0142d8ff2/66db5a8e-229f-48cb-8657-576a3a35aa17"
+          (reference "#PWR0250") (unit 1)
+        )
+      )
+    )
+  )
   (symbol (lib_id "Mad5150_early:LS138_U45") (at 155.575 -46.99 0) (unit 2)
     (in_bom yes) (on_board yes) (dnp no) (fields_autoplaced)
@@
     )
   )
+  (symbol (lib_id "power:+5V") (at -31.115 -83.185 180) (unit 1)
+    (in_bom yes) (on_board yes) (dnp no)
+    (property "Reference" "#PWR0251" (at -31.115 -86.995 0)
+      (effects (font (size 1.27 1.27)) hide)
+    )
+    (property "Value" "+5V" (at -31.115 -79.375 0)
+      (effects (font (size 1.27 1.27)))
+    )
+    (property "Footprint" "" (at -31.115 -83.185 0)
+      (effects (font (size 1.27 1.27)) hide)
+    )
+    (property "Datasheet" "" (at -31.115 -83.185 0)
+      (effects (font (size 1.27 1.27)) hide)
+    )
+    (pin "1")
+    (instances
+      (project "Mad5160"
+        (path "/ac3c86ab-084e-42f6-87ca-c4b0142d8ff2/66db5a8e-229f-48cb-8657-576a3a35aa17"
+          (reference "#PWR0251") (unit 1)
+        )
+      )
+    )
+  )
   (symbol (lib_id "power:+5V") (at 118.11 123.19 90) (unit 1)
     (in_bom yes) (on_board yes) (dnp no)
@@
         )
       )
+    )
+  )
+  (symbol (lib_id "power:+5V") (at -17.145 -83.82 180) (unit 1)
+    (in_bom yes) (on_board yes) (dnp no)
+    (property "Reference" "#PWR0252" (at -17.145 -87.63 0)
+      (effects (font (size 1.27 1.27)) hide)
+    )
+    (property "Value" "+5V" (at -17.145 -80.01 0)
+      (effects (font (size 1.27 1.27)))
+    )
+    (property "Footprint" "" (at -17.145 -83.82 0)
+      (effects (font (size 1.27 1.27)) hide)
+    )
+    (property "Datasheet" "" (at -17.145 -83.82 0)
+      (effects (font (size 1.27 1.27)) hide)
+    )
+    (pin "1")
+    (instances
+      (project "Mad5160"
+        (path "/ac3c86ab-084e-42f6-87ca-c4b0142d8ff2/66db5a8e-229f-48cb-8657-576a3a35aa17"
+          (reference "#PWR0252") (unit 1)
+        )
+      )

Commit message: Update 010502024
Parts:
- removed E7: E7_Jumper_block, Connector_PinHeader_2.54mm:PinHeader_2x01_P2.54mm_Vertical, symbol Mad5150_early:E7_Jumper_block
- added E1: E1_Jumper_block, Connector_PinHeader_2.54mm:PinHeader_2x01_P2.54mm_Vertical, symbol Mad5150_early:E1_Jumper_block
Connections:
- net GND: now also E1.1 (Pin_1)
- net at RN2.1, U24.1: now also E1.2 (Pin_2)
- net ~{MEMR}' renamed ~{YMEMR}'
- no-connect marks 24 -> 30
Other:
- moved on the sheet: E2, E3, RN2A, RN2F, RN2G, RN2H, RN2N, RN2O, RN4C, RN4D, RN4E, RN4F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
