File: sheet3.kicad_sch (KiCad schematic)
At the start: 16 parts, among them U24 LS00_U24, U42 LS138, U43 LS138, U44 24S10, U45 LS138, U55 S08_U55, U56 LS138, U57 LS20_U57, U58 LS32_U58, U69 S00_U69

Commit message: Tracing for version 1.0 finished
Parts:
- TD1: footprint Package_DIP:DIP-14_W7.62mm -> madXT_early:time_delay
Changed lines of the file:
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@@
       (effects (font (size 1.27 1.27) bold) (justify left))
     )
-    (property "Footprint" "Package_DIP:DIP-14_W7.62mm" (at 193.04 86.995 0)
+    (property "Footprint" "madXT_early:time_delay" (at 193.04 86.995 0)
       (effects (font (size 1.27 1.27)) hide)
     )
@@
       (effects (font (size 1.27 1.27) bold) (justify left))
     )
-    (property "Footprint" "Package_DIP:DIP-14_W7.62mm" (at 160.655 257.81 0)
-      (effects (font (size 1.27 1.27)) hide)
-    )
+    (property "Footprint" "madXT_early:time_delay" (at 160.655 257.81 0)
+      (effects (font (size 1.27 1.27)) hide)
+    )

Commit message: Tracing finished
Parts:
- E1: footprint Connector_PinHeader_2.54mm:PinHeader_2x01_P2.54mm_Vertical -> mad5150:PinHeader_2x01_P2.54mm_Vertical
- E2: footprint Connector_PinHeader_2.54mm:PinHeader_2x02_P2.54mm_Vertical -> mad5150:PinHeader_2x02_P2.54mm_Vertical
- E3: footprint Connector_PinHeader_2.54mm:PinHeader_2x04_P2.54mm_Vertical -> mad5150:PinHeader_2x04_P2.54mm_Vertical
- RN2, RN4, U42, U43, U44, U45, U56: footprint Package_DIP:DIP-16_W7.62mm -> mad5150:DIP-16_W7.62mm
- TD1: footprint madXT_early:time_delay -> mad5150:time_delay
- U24, U55, U57, U58, U69: footprint Package_DIP:DIP-14_W7.62mm -> mad5150:DIP-14_W7.62mm

Commit message: Fixing stuff
Parts:
- removed unit 2 of U58
Connections:
- no-connect marks 30 -> 27
Changed lines of the file:
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@@
   (junction (at 64.135 187.96) (diameter 0) (color 0 0 0 0)
   )
-  (no_connect (at 277.495 277.495))
   (no_connect (at 109.22 163.83))
   (no_connect (at 247.65 250.19))
@@
   (no_connect (at 153.035 133.985))
   (no_connect (at 103.505 131.445))
-  (no_connect (at 277.495 272.415))
   (no_connect (at 102.87 87.63))
   (no_connect (at 280.67 250.19))
@@
   (no_connect (at 103.505 126.365))
   (no_connect (at 153.035 139.065))
-  (no_connect (at 292.735 274.955))
   (no_connect (at 109.22 153.67))
   (no_connect (at 153.035 136.525))
@@
         )
       )
-    )
-  )
-  (symbol (lib_id "Mad5150_early:LS32_U58") (at 285.115 274.955 0) (unit 2)
-    (in_bom yes) (on_board yes) (dnp no) (fields_autoplaced)
-    (property "Reference" "U58" (at 285.115 267.335 0)
-      (effects (font (size 1.27 1.27)))
-    )
-    (property "Value" "LS32_U58" (at 285.115 269.875 0)
-      (effects (font (size 1.27 1.27)))
-    )
-    (property "Footprint" "mad5150:DIP-14_W7.62mm" (at 285.115 274.955 0)
-      (effects (font (size 1.27 1.27)) hide)
-    )
-    (property "Datasheet" "http://www.ti.com/lit/gpn/sn74LS32" (at 285.115 274.955 0)
-      (effects (font (size 1.27 1.27)) hide)
-    )
-    (pin "11")
-    (pin "5")
-    (pin "14")
-    (pin "3")
-    (pin "10")
-    (pin "13")
-    (pin "6")
-    (pin "9")
-    (pin "12")
-    (pin "2")
-    (pin "7")
-    (pin "8")
-    (pin "4")
-    (pin "1")
-    (instances
-      (project "Mad5160"
-        (path "/ac3c86ab-084e-42f6-87ca-c4b0142d8ff2/66db5a8e-229f-48cb-8657-576a3a35aa17"
-          (reference "U58") (unit 2)
-        )
-      )

Commit message: Gerbers
Parts:
- U56: value LS138 -> 74S138
Changed lines of the file:
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@@
       (effects (font (size 1.27 1.27)))
     )
-    (property "Value" "LS138" (at 140.335 137.16 0)
+    (property "Value" "74S138" (at 140.335 137.16 0)
       (effects (font (size 1.27 1.27) bold))
     )
@@
       (effects (font (size 1.27 1.27)) (justify left))
     )
-    (property "Value" "LS138" (at 102.87 257.81 0)
+    (property "Value" "74S138" (at 102.87 257.81 0)
       (effects (font (size 1.27 1.27) bold) (justify left))
     )
