File: sheet4.kicad_sch (KiCad schematic)
At the start: 7 parts, among them U10 LS670_U10, U11 LS373, U12 LS244, U22 74LS04, U28 8237A-5_U28, U71 LS04_U71

Commit message: Sheet 10 done
Parts:
- RN5: symbol Mad5150_early:Resistor_Network -> Mad5150_early:Resistor_Network_1
Changed lines of the file:
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@@
     )
   )
-  (symbol (lib_id "Mad5150_early:Resistor_Network") (at 176.53 68.58 270) (unit 5)
+  (symbol (lib_id "Mad5150_early:Resistor_Network_1") (at 176.53 68.58 270) (unit 5)
     (in_bom yes) (on_board yes) (dnp no)
     (property "Reference" "RN5" (at 176.53 66.04 90)
@@
       (effects (font (size 1.27 1.27)) hide)
     )
-    (property "Datasheet" "" (at 176.53 68.58 0)
+    (property "Datasheet" "" (at 177.165 69.215 0)
       (effects (font (size 1.27 1.27)) hide)
     )

Commit message: Update 010502024
Changed lines of the file:
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@@
     (effects (font (size 1.27 1.27)) (justify right bottom))
-  )
-  (label "TERMINAL COUNT" (at 223.52 60.325 0) (fields_autoplaced)
-    (effects (font (size 1.27 1.27)) (justify left bottom))
   )
   (label "A10" (at 205.105 140.97 180) (fields_autoplaced)

Commit message: Tracing for version 1.0 finished
Connections:
- net XA5: now also U28.38 (A5); no longer U28.36 (~{EOP})
Changed lines of the file:
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@@
+    (stroke (width 0) (type default))
+  )
+  (wire (pts (xy 95.25 32.385) (xy 104.14 32.385))
     (stroke (width 0) (type default))
   )
@@
   )
   (bus (pts (xy 160.655 140.97) (xy 160.655 143.51))
-    (stroke (width 0) (type default))
-  )
-  (wire (pts (xy 95.25 32.385) (xy 104.14 32.385))
     (stroke (width 0) (type default))
   )
@@
     (pin "11")
     (pin "25")
-    (pin "36")
+    (pin "38")
     (pin "24")
     (pin "19")

Commit message: Tracing finished
Parts:
- RN5, U10: footprint Package_DIP:DIP-16_W7.62mm -> mad5150:DIP-16_W7.62mm
- U11, U12: footprint Package_DIP:DIP-20_W7.62mm -> mad5150:DIP-20_W7.62mm
- U22, U71: footprint Package_DIP:DIP-14_W7.62mm -> mad5150:DIP-14_W7.62mm
- U28: footprint Package_DIP:DIP-40_W15.24mm -> mad5150:DIP-40_W15.24mm
Changed lines of the file:
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@@
       (effects (font (size 1.27 1.27)))
     )
-    (property "Footprint" "Package_DIP:DIP-16_W7.62mm" (at 186.055 133.35 0)
+    (property "Footprint" "mad5150:DIP-16_W7.62mm" (at 186.055 133.35 0)
       (effects (font (size 1.27 1.27)) hide)
     )
@@
       (effects (font (size 1.27 1.27) bold) (justify left))
     )
-    (property "Footprint" "Package_DIP:DIP-20_W7.62mm" (at 271.145 143.51 0)
+    (property "Footprint" "mad5150:DIP-20_W7.62mm" (at 271.145 143.51 0)
       (effects (font (size 1.27 1.27)) hide)
     )
@@
       (effects (font (size 1.27 1.27) bold))
     )
-    (property "Footprint" "Package_DIP:DIP-20_W7.62mm" (at 184.785 35.56 0)
+    (property "Footprint" "mad5150:DIP-20_W7.62mm" (at 184.785 35.56 0)
       (effects (font (size 1.27 1.27)) hide)
     )
@@
       (effects (font (size 1.27 1.27)))
     )
-    (property "Footprint" "Package_DIP:DIP-14_W7.62mm" (at 226.06 67.945 0)
+    (property "Footprint" "mad5150:DIP-14_W7.62mm" (at 226.06 67.945 0)
       (effects (font (size 1.27 1.27)) hide)
     )
@@
       (effects (font (size 1.27 1.27)))
     )
-    (property "Footprint" "Package_DIP:DIP-16_W7.62mm" (at 176.53 68.58 0)
+    (property "Footprint" "mad5150:DIP-16_W7.62mm" (at 176.53 68.58 0)
       (effects (font (size 1.27 1.27)) hide)
     )
@@
       (effects (font (size 1.27 1.27) bold))
     )
-    (property "Footprint" "Package_DIP:DIP-20_W7.62mm" (at 186.055 140.97 0)
+    (property "Footprint" "mad5150:DIP-20_W7.62mm" (at 186.055 140.97 0)
       (effects (font (size 1.27 1.27)) hide)
     )
@@
       (effects (font (size 1.27 1.27)) (justify left))
     )
-    (property "Footprint" "Package_DIP:DIP-16_W7.62mm" (at 248.285 165.1 0)
+    (property "Footprint" "mad5150:DIP-16_W7.62mm" (at 248.285 165.1 0)
       (effects (font (size 1.27 1.27)) hide)
     )
@@
       (effects (font (size 1.27 1.27)))
     )
-    (property "Footprint" "Package_DIP:DIP-40_W15.24mm" (at 80.01 95.885 0)
+    (property "Footprint" "mad5150:DIP-40_W15.24mm" (at 80.01 95.885 0)
       (effects (font (size 1.27 1.27)) hide)
     )
@@
       (effects (font (size 1.27 1.27)))
     )
-    (property "Footprint" "Package_DIP:DIP-14_W7.62mm" (at 196.85 60.325 0)
+    (property "Footprint" "mad5150:DIP-14_W7.62mm" (at 196.85 60.325 0)
       (effects (font (size 1.27 1.27)) hide)
     )
@@
       (effects (font (size 1.27 1.27) bold) (justify left))
     )
-    (property "Footprint" "Package_DIP:DIP-20_W7.62mm" (at 225.425 139.7 0)
-      (effects (font (size 1.27 1.27)) hide)
-    )
+    (property "Footprint" "mad5150:DIP-20_W7.62mm" (at 225.425 139.7 0)
+      (effects (font (size 1.27 1.27)) hide)
+    )
