File: sheet7.kicad_sch (KiCad schematic)
At the start: 18 parts, among them U59 64K x1 bit RAM 4164, U60 64K x1 bit RAM 4164, U61 64K x1 bit RAM 4164, U62 64K x1 bit RAM 4164, U63 64K x1 bit RAM 4164, U64 64K x1 bit RAM 4164, U65 64K x1 bit RAM 4164, U66 64K x1 bit RAM 4164, U67 64K x1 bit RAM 4164, U75 64K x1 bit RAM 4164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

Commit message: Sheet 8 finished
Connections:
- net MDPIN: now also U59.2 (D), U75.2 (D)
- net MDPOUT: now also U59.14 (Q), U75.14 (Q)
Changed lines of the file:
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@@
+    (stroke (width 0) (type default))
+  )
+  (bus_entry (at 415.925 203.2) (size 2.54 2.54)
     (stroke (width 0) (type default))
   )
@@
     (stroke (width 0) (type default))
   )
+  (bus_entry (at 460.375 205.74) (size 2.54 -2.54)
+    (stroke (width 0) (type default))
+  )
   (bus_entry (at 257.175 130.175) (size -2.54 2.54)
     (stroke (width 0) (type default))
@@
     (stroke (width 0) (type default))
   )
+  (bus_entry (at 415.925 155.575) (size 2.54 2.54)
+    (stroke (width 0) (type default))
+  )
   (bus_entry (at 368.935 70.485) (size 2.54 2.54)
     (stroke (width 0) (type default))
@@
     (stroke (width 0) (type default))
   )
+  (bus_entry (at 460.375 158.115) (size 2.54 -2.54)
+    (stroke (width 0) (type default))
+  )
   (bus_entry (at 415.925 183.515) (size 2.54 2.54)
     (stroke (width 0) (type default))
@@
     (stroke (width 0) (type default))
   )
-  (bus (pts (xy 415.925 183.515) (xy 415.925 205.74))
+  (bus (pts (xy 415.925 183.515) (xy 415.925 203.2))
     (stroke (width 0) (type default))
   )
@@
     (stroke (width 0) (type default))
   )
+  (wire (pts (xy 456.565 158.115) (xy 460.375 158.115))
+    (stroke (width 0) (type default))
+  )
   (wire (pts (xy 371.475 278.765) (xy 380.365 278.765))
     (stroke (width 0) (type default))
@@
     (stroke (width 0) (type default))
   )
+  (bus (pts (xy 415.925 203.2) (xy 415.925 205.74))
+    (stroke (width 0) (type default))
+  )
   (wire (pts (xy 412.75 103.505) (xy 379.73 103.505))
     (stroke (width 0) (type default))
@@
     (stroke (width 0) (type default))
   )
+  (bus (pts (xy 462.915 155.575) (xy 462.915 169.545))
+    (stroke (width 0) (type default))
+  )
   (wire (pts (xy 277.495 313.69) (xy 286.385 313.69))
     (stroke (width 0) (type default))
@@
     (stroke (width 0) (type default))
   )
+  (wire (pts (xy 456.565 205.74) (xy 460.375 205.74))
+    (stroke (width 0) (type default))
+  )
   (bus (pts (xy 415.925 135.89) (xy 415.925 147.955))
     (stroke (width 0) (type default))
@@
     (stroke (width 0) (type default))
   )
-  (bus (pts (xy 462.915 121.92) (xy 462.915 169.545))
+  (bus (pts (xy 462.915 121.92) (xy 462.915 155.575))
     (stroke (width 0) (type default))
   )
@@
     (stroke (width 0) (type default))
   )
+  (wire (pts (xy 418.465 205.74) (xy 427.355 205.74))
+    (stroke (width 0) (type default))
+  )
   (bus (pts (xy 368.935 273.685) (xy 368.935 276.225))
     (stroke (width 0) (type default))
@@
     (stroke (width 0) (type default))
   )
+  (bus (pts (xy 415.925 155.575) (xy 415.925 158.115))
+    (stroke (width 0) (type default))
+  )
   (bus (pts (xy 274.955 260.985) (xy 274.955 263.525))
     (stroke (width 0) (type default))
   )
+  (wire (pts (xy 418.465 158.115) (xy 427.355 158.115))
+    (stroke (width 0) (type default))
+  )
   (wire (pts (xy 277.495 328.93) (xy 286.385 328.93))
     (stroke (width 0) (type default))
@@
     (stroke (width 0) (type default))
   )
-  (bus (pts (xy 462.915 169.545) (xy 462.915 217.17))
+  (bus (pts (xy 462.915 169.545) (xy 462.915 203.2))
     (stroke (width 0) (type default))
   )
@@
     (stroke (width 0) (type default))
   )
-  (bus (pts (xy 415.925 147.955) (xy 415.925 158.115))
+  (bus (pts (xy 415.925 147.955) (xy 415.925 155.575))
     (stroke (width 0) (type default))
   )
@@
   )
   (bus (pts (xy 274.955 278.765) (xy 274.955 290.83))
+    (stroke (width 0) (type default))
+  )
+  (bus (pts (xy 462.915 203.2) (xy 462.915 217.17))
     (stroke (width 0) (type default))
   )
@@
     (effects (font (size 1.27 1.27)) (justify right bottom))
   )
+  (label "MDPOUT" (at 457.2 158.115 0) (fields_autoplaced)
+    (effects (font (size 1.27 1.27)) (justify left bottom))
+  )
   (label "MA4" (at 285.75 273.685 180) (fields_autoplaced)
     (effects (font (size 1.27 1.27)) (justify right bottom))
@@
   (label "MA2" (at 426.72 78.105 180) (fields_autoplaced)
     (effects (font (size 1.27 1.27)) (justify right bottom))
+  )
+  (label "MDPIN" (at 421.005 158.115 0) (fields_autoplaced)
+    (effects (font (size 1.27 1.27)) (justify left bottom))
   )
   (label "MA5" (at 379.73 323.85 180) (fields_autoplaced)
@@
     (effects (font (size 1.27 1.27)) (justify right bottom))
   )
+  (label "MDPOUT" (at 457.2 205.74 0) (fields_autoplaced)
+    (effects (font (size 1.27 1.27)) (justify left bottom))
+  )
   (label "MA7" (at 426.72 233.68 180) (fields_autoplaced)
     (effects (font (size 1.27 1.27)) (justify right bottom))
@@
     (effects (font (size 1.27 1.27)) (justify right bottom))
   )
+  (label "MDPIN" (at 421.005 205.74 0) (fields_autoplaced)
+    (effects (font (size 1.27 1.27)) (justify left bottom))
+  )
   (label "~{CAS2}" (at 285.75 67.945 180) (fields_autoplaced)

Commit message: Tracing finished
Parts:
- U59, U60, U61, U62, U63, U64, U65, U66, U67, U75, U76, U77, U78, U79, U80, U81, U82, U83: footprint Package_DIP:DIP-16_W7.62mm -> mad5150:Ram_socket_IC
Changed lines of the file:
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@@
       (effects (font (size 1.27 1.27)))
     )
-    (property "Footprint" "Package_DIP:DIP-16_W7.62mm" (at 386.08 99.695 0)
+    (property "Footprint" "mad5150:Ram_socket_IC" (at 386.08 99.695 0)
       (effects (font (size 1.27 1.27)) hide)
     )
@@
       (effects (font (size 1.27 1.27)))
     )
-    (property "Footprint" "Package_DIP:DIP-16_W7.62mm" (at 386.08 290.195 0)
+    (property "Footprint" "mad5150:Ram_socket_IC" (at 386.08 290.195 0)
       (effects (font (size 1.27 1.27)) hide)
     )
@@
       (effects (font (size 1.27 1.27)))
     )
-    (property "Footprint" "Package_DIP:DIP-16_W7.62mm" (at 292.1 52.07 0)
+    (property "Footprint" "mad5150:Ram_socket_IC" (at 292.1 52.07 0)
       (effects (font (size 1.27 1.27)) hide)
     )
@@
       (effects (font (size 1.27 1.27)))
     )
-    (property "Footprint" "Package_DIP:DIP-16_W7.62mm" (at 433.07 242.57 0)
+    (property "Footprint" "mad5150:Ram_socket_IC" (at 433.07 242.57 0)
       (effects (font (size 1.27 1.27)) hide)
     )
@@
       (effects (font (size 1.27 1.27)))
     )
-    (property "Footprint" "Package_DIP:DIP-16_W7.62mm" (at 433.07 290.195 0)
+    (property "Footprint" "mad5150:Ram_socket_IC" (at 433.07 290.195 0)
       (effects (font (size 1.27 1.27)) hide)
     )
@@
       (effects (font (size 1.27 1.27)))
     )
-    (property "Footprint" "Package_DIP:DIP-16_W7.62mm" (at 433.07 99.695 0)
+    (property "Footprint" "mad5150:Ram_socket_IC" (at 433.07 99.695 0)
       (effects (font (size 1.27 1.27)) hide)
     )
@@
       (effects (font (size 1.27 1.27)))
     )
-    (property "Footprint" "Package_DIP:DIP-16_W7.62mm" (at 386.08 242.57 0)
+    (property "Footprint" "mad5150:Ram_socket_IC" (at 386.08 242.57 0)
       (effects (font (size 1.27 1.27)) hide)
     )
@@
       (effects (font (size 1.27 1.27)))
     )
-    (property "Footprint" "Package_DIP:DIP-16_W7.62mm" (at 292.1 242.57 0)
+    (property "Footprint" "mad5150:Ram_socket_IC" (at 292.1 242.57 0)
       (effects (font (size 1.27 1.27)) hide)
     )
@@
       (effects (font (size 1.27 1.27)))
     )
-    (property "Footprint" "Package_DIP:DIP-16_W7.62mm" (at 292.1 99.695 0)
+    (property "Footprint" "mad5150:Ram_socket_IC" (at 292.1 99.695 0)
       (effects (font (size 1.27 1.27)) hide)
     )
@@
       (effects (font (size 1.27 1.27)))
     )
-    (property "Footprint" "Package_DIP:DIP-16_W7.62mm" (at 339.09 52.07 0)
+    (property "Footprint" "mad5150:Ram_socket_IC" (at 339.09 52.07 0)
       (effects (font (size 1.27 1.27)) hide)
     )
@@
       (effects (font (size 1.27 1.27)))
     )
-    (property "Footprint" "Package_DIP:DIP-16_W7.62mm" (at 292.1 290.195 0)
+    (property "Footprint" "mad5150:Ram_socket_IC" (at 292.1 290.195 0)
       (effects (font (size 1.27 1.27)) hide)
     )
@@
       (effects (font (size 1.27 1.27)))
     )
-    (property "Footprint" "Package_DIP:DIP-16_W7.62mm" (at 433.07 194.945 0)
+    (property "Footprint" "mad5150:Ram_socket_IC" (at 433.07 194.945 0)
       (effects (font (size 1.27 1.27)) hide)
     )
@@
       (effects (font (size 1.27 1.27)))
     )
-    (property "Footprint" "Package_DIP:DIP-16_W7.62mm" (at 433.07 52.07 0)
+    (property "Footprint" "mad5150:Ram_socket_IC" (at 433.07 52.07 0)
       (effects (font (size 1.27 1.27)) hide)
     )
@@
       (effects (font (size 1.27 1.27)))
     )
-    (property "Footprint" "Package_DIP:DIP-16_W7.62mm" (at 339.09 290.195 0)
+    (property "Footprint" "mad5150:Ram_socket_IC" (at 339.09 290.195 0)
       (effects (font (size 1.27 1.27)) hide)
     )
@@
       (effects (font (size 1.27 1.27)))
     )
-    (property "Footprint" "Package_DIP:DIP-16_W7.62mm" (at 339.09 242.57 0)
+    (property "Footprint" "mad5150:Ram_socket_IC" (at 339.09 242.57 0)
       (effects (font (size 1.27 1.27)) hide)
     )
@@
       (effects (font (size 1.27 1.27)))
     )
-    (property "Footprint" "Package_DIP:DIP-16_W7.62mm" (at 433.07 147.32 0)
+    (property "Footprint" "mad5150:Ram_socket_IC" (at 433.07 147.32 0)
       (effects (font (size 1.27 1.27)) hide)
     )
@@
       (effects (font (size 1.27 1.27)))
     )
-    (property "Footprint" "Package_DIP:DIP-16_W7.62mm" (at 339.09 99.695 0)
+    (property "Footprint" "mad5150:Ram_socket_IC" (at 339.09 99.695 0)
       (effects (font (size 1.27 1.27)) hide)
     )
@@
       (effects (font (size 1.27 1.27)))
     )
-    (property "Footprint" "Package_DIP:DIP-16_W7.62mm" (at 386.08 52.07 0)
-      (effects (font (size 1.27 1.27)) hide)
-    )
+    (property "Footprint" "mad5150:Ram_socket_IC" (at 386.08 52.07 0)
+      (effects (font (size 1.27 1.27)) hide)
+    )
