File: sheet10.kicad_sch (KiCad schematic)
At the start: 1 part, among them J1 ISA Bus connector

Commit message: Sheet 10 done
Parts:
- added C10, C11, C12, C13, C14, C15, C16, C19, C28, C3, C37, C46, C54, C56, C58, C60, C61, C63: 10uF 25V, symbol Device:C_Polarized
- added C17, C18, C20, C21, C22, C23, C24, C25, C26, C27, C29, C30, C31, C32, C33, C34, C35, C36, C38, C39, C40, C41, C42, C43, C44, C45, C47, C48, C49, C5, C50, C51, C52, C55, C57, C59, C62, C64, C65, C66, C67: 0.047pF, symbol Device:C
- added C68: 10uF, symbol Device:C
- added J10: AT POWER CONNECTOR, symbol Connector:Conn_01x12_Pin
- added J2, J3, J4, J5, J6, J7: ISA Bus connector, madXT_early:isa_edge_slot, symbol Mad5150_early:ISA
- added J8: ISA Bus connector, madXT_early:isa_edge_slot, symbol Mad5150_early:ISA_slot_8
Connections:
- net I/O CHCK: now reaches J1.A1 (I/OCHCK)
- net I/O CHCK: now also J2.A1 (I/OCHCK), J3.A1 (I/OCHCK), J4.A1 (I/OCHCK), J5.A1 (I/OCHCK), J6.A1 (I/OCHCK), J7.A1 (I/OCHCK), J8.A1 (I/OCHCK)
- net I/O CHRDY: now reaches J1.A10 (I/OCHRDY)
- net I/O CHRDY: now also J2.A10 (I/OCHRDY), J3.A10 (I/OCHRDY), J4.A10 (I/OCHRDY), J5.A10 (I/OCHRDY), J6.A10 (I/OCHRDY), J7.A10 (I/OCHRDY), J8.A10 (I/OCHRDY)
- net AEN: now reaches J1.A11 (AEN)
- net AEN: now also J2.A11 (AEN), J3.A11 (AEN), J4.A11 (AEN), J5.A11 (AEN), J6.A11 (AEN), J7.A11 (AEN), J8.A11 (AEN)
- net A19: now reaches J1.A12 (A19)
- net A19: now also J2.A12 (A19), J3.A12 (A19), J4.A12 (A19), J5.A12 (A19), J6.A12 (A19), J7.A12 (A19)
- net A18: now reaches J1.A13 (A18)
- net A18: now also J2.A13 (A18), J3.A13 (A18), J4.A13 (A18), J5.A13 (A18), J6.A13 (A18), J7.A13 (A18)
- net A17: now reaches J1.A14 (A17)
- net A17: now also J2.A14 (A17), J3.A14 (A17), J4.A14 (A17), J5.A14 (A17), J6.A14 (A17), J7.A14 (A17)
- net A16: now reaches J1.A15 (A16)
- net A16: now also J2.A15 (A16), J3.A15 (A16), J4.A15 (A16), J5.A15 (A16), J6.A15 (A16), J7.A15 (A16)
- net A15: now reaches J1.A16 (A15)
- net A15: now also J2.A16 (A15), J3.A16 (A15), J4.A16 (A15), J5.A16 (A15), J6.A16 (A15), J7.A16 (A15)
- net A14: now reaches J1.A17 (A14)
- net A14: now also J2.A17 (A14), J3.A17 (A14), J4.A17 (A14), J5.A17 (A14), J6.A17 (A14), J7.A17 (A14)
- net A13: now reaches J1.A18 (A13)
- net A13: now also J2.A18 (A13), J3.A18 (A13), J4.A18 (A13), J5.A18 (A13), J6.A18 (A13), J7.A18 (A13)
- net A12: now reaches J1.A19 (A12)
- net A12: now also J2.A19 (A12), J3.A19 (A12), J4.A19 (A12), J5.A19 (A12), J6.A19 (A12), J7.A19 (A12)
- net D7: now reaches J1.A2 (D7)
- net D7: now also J2.A2 (D7), J3.A2 (D7), J4.A2 (D7), J5.A2 (D7), J6.A2 (D7), J7.A2 (D7)
- net A11: now reaches J1.A20 (A11)
- net A11: now also J2.A20 (A11), J3.A20 (A11), J4.A20 (A11), J5.A20 (A11), J6.A20 (A11), J7.A20 (A11)
- net A10: now reaches J1.A21 (A10)
- net A10: now also J2.A21 (A10), J3.A21 (A10), J4.A21 (A10), J5.A21 (A10), J6.A21 (A10), J7.A21 (A10)
- net A9: now reaches J1.A22 (A9)
- net A9: now also J2.A22 (A9), J3.A22 (A9), J4.A22 (A9), J5.A22 (A9), J6.A22 (A9), J7.A22 (A9)
- net A8: now reaches J1.A23 (A8)
- net A8: now also J2.A23 (A8), J3.A23 (A8), J4.A23 (A8), J5.A23 (A8), J6.A23 (A8), J7.A23 (A8)
- net A7: now reaches J1.A24 (A7)
- net A7: now also J2.A24 (A7), J3.A24 (A7), J4.A24 (A7), J5.A24 (A7), J6.A24 (A7), J7.A24 (A7)
- net A6: now reaches J1.A25 (A6)
- net A6: now also J2.A25 (A6), J3.A25 (A6), J4.A25 (A6), J5.A25 (A6), J6.A25 (A6), J7.A25 (A6)
- net A5: now reaches J1.A26 (A5)
- net A5: now also J2.A26 (A5), J3.A26 (A5), J4.A26 (A5), J5.A26 (A5), J6.A26 (A5), J7.A26 (A5)
- net A4: now reaches J1.A27 (A4)
- net A4: now also J2.A27 (A4), J3.A27 (A4), J4.A27 (A4), J5.A27 (A4), J6.A27 (A4), J7.A27 (A4)
- net A3: now reaches J1.A28 (A3)
- net A3: now also J2.A28 (A3), J3.A28 (A3), J4.A28 (A3), J5.A28 (A3), J6.A28 (A3), J7.A28 (A3)
- net A2: now reaches J1.A29 (A2)
- net A2: now also J2.A29 (A2), J3.A29 (A2), J4.A29 (A2), J5.A29 (A2), J6.A29 (A2), J7.A29 (A2)
- net D6: now reaches J1.A3 (D6)
- net D6: now also J2.A3 (D6), J3.A3 (D6), J4.A3 (D6), J5.A3 (D6), J6.A3 (D6), J7.A3 (D6)
- net A1: now reaches J1.A30 (A1)
- net A1: now also J2.A30 (A1), J3.A30 (A1), J4.A30 (A1), J5.A30 (A1), J6.A30 (A1), J7.A30 (A1)
- net A0: now reaches J1.A31 (A0)
- net A0: now also J2.A31 (A0), J3.A31 (A0), J4.A31 (A0), J5.A31 (A0), J6.A31 (A0), J7.A31 (A0)
- net D5: now reaches J1.A4 (D5)
- net D5: now also J2.A4 (D5), J3.A4 (D5), J4.A4 (D5), J5.A4 (D5), J6.A4 (D5), J7.A4 (D5)
- net D4: now reaches J1.A5 (D4)
- net D4: now also J2.A5 (D4), J3.A5 (D4), J4.A5 (D4), J5.A5 (D4), J6.A5 (D4), J7.A5 (D4)
- net D3: now reaches J1.A6 (D3)
- net D3: now also J2.A6 (D3), J3.A6 (D3), J4.A6 (D3), J5.A6 (D3), J6.A6 (D3), J7.A6 (D3)
- net D2: now reaches J1.A7 (D2)
- net D2: now also J2.A7 (D2), J3.A7 (D2), J4.A7 (D2), J5.A7 (D2), J6.A7 (D2), J7.A7 (D2)
- net D1: now reaches J1.A8 (D1)
- net D1: now also J2.A8 (D1), J3.A8 (D1), J4.A8 (D1), J5.A8 (D1), J6.A8 (D1), J7.A8 (D1)
- net D0: now reaches J1.A9 (D0)
- net D0: now also J2.A9 (D0), J3.A9 (D0), J4.A9 (D0), J5.A9 (D0), J6.A9 (D0), J7.A9 (D0)
- net GND: now reaches J1.B1 (GND)
- net GND: now also J1.B10 (GND), J1.B31 (GND), C10.2, C11.2, C12.2, C13.2, C14.2, C15.2, C16.2, C17.2, C18.2, C19.2, C20.2, C21.2, C22.2, C23.2, C24.2, C25.2, C26.2, C27.2, C28.2, C29.2, C3.2, C30.2, C31.2, C32.2, C33.2, C34.2, C35.2, C36.2, C37.2, C38.2, C39.2, C40.2, C41.2, C42.2, C43.2, C44.2, C45.2, C46.2, C47.2, C48.2, C49.2, C5.2, C50.2, C51.2, C52.2, C54.2, C55.2, C56.2, C57.2, C58.2, C59.2, C60.2, C61.2, C62.2, C63.2, C64.2, C65.2, C66.2, C67.2, C68.2, J10.5 (Pin_5), J10.6 (Pin_6), J10.7 (Pin_7), J10.8 (Pin_8), J2.B1 (GND), J2.B10 (GND), J2.B31 (GND), J3.B1 (GND), J3.B10 (GND), J3.B31 (GND), J4.B1 (GND), J4.B10 (GND), J4.B31 (GND), J5.B1 (GND), J5.B10 (GND), J5.B31 (GND), J6.B1 (GND), J6.B10 (GND), J6.B31 (GND), J7.B1 (GND), J7.B10 (GND), J7.B31 (GND), J8.B1 (GND), J8.B10 (GND), J8.B31 (GND)
- net ~{MEMW}': now reaches J1.B11 (~{MEMW})
- net ~{MEMW}': now also J2.B11 (~{MEMW}), J3.B11 (~{MEMW}), J4.B11 (~{MEMW}), J5.B11 (~{MEMW}), J6.B11 (~{MEMW}), J7.B11 (~{MEMW})
- net ~{MEMR}': now reaches J1.B12 (~{MEMR})
- net ~{MEMR}': now also J2.B12 (~{MEMR}), J3.B12 (~{MEMR}), J4.B12 (~{MEMR}), J5.B12 (~{MEMR}), J6.B12 (~{MEMR}), J7.B12 (~{MEMR})
- net ~{IOW}': now reaches J1.B13 (~{IOW})
- net ~{IOW}': now also J2.B13 (~{IOW}), J3.B13 (~{IOW}), J4.B13 (~{IOW}), J5.B13 (~{IOW}), J6.B13 (~{IOW}), J7.B13 (~{IOW})
- net ~{IOR}': now reaches J1.B14 (~{IOR})
- net ~{IOR}': now also J2.B14 (~{IOR}), J3.B14 (~{IOR}), J4.B14 (~{IOR}), J5.B14 (~{IOR}), J6.B14 (~{IOR}), J7.B14 (~{IOR})
- net ~{DA0K3}': now reaches J1.B15 (~{DACK3})
- net ~{DA0K3}': now also J2.B15 (~{DACK3}), J3.B15 (~{DACK3}), J4.B15 (~{DACK3}), J5.B15 (~{DACK3}), J6.B15 (~{DACK3}), J7.B15 (~{DACK3}), J8.B15 (~{DACK3})
- net DRQ3: now reaches J1.B16 (DRQ3)
- net DRQ3: now also J2.B16 (DRQ3), J3.B16 (DRQ3), J4.B16 (DRQ3), J5.B16 (DRQ3), J6.B16 (DRQ3), J7.B16 (DRQ3), J8.B16 (DRQ3)
- net ~{DA0K1}': now reaches J1.B17 (~{DACK1})
- net ~{DA0K1}': now also J2.B17 (~{DACK1}), J3.B17 (~{DACK1}), J4.B17 (~{DACK1}), J5.B17 (~{DACK1}), J6.B17 (~{DACK1}), J7.B17 (~{DACK1}), J8.B17 (~{DACK1})
- net DRQ1: now reaches J1.B18 (DRQ1)
- net DRQ1: now also J2.B18 (DRQ1), J3.B18 (DRQ1), J4.B18 (DRQ1), J5.B18 (DRQ1), J6.B18 (DRQ1), J7.B18 (DRQ1), J8.B18 (DRQ1)
- net ~{DACK0}': now reaches J1.B19 (~{DACK0})
- net ~{DACK0}': now also J2.B19 (~{DACK0}), J3.B19 (~{DACK0}), J4.B19 (~{DACK0}), J5.B19 (~{DACK0}), J6.B19 (~{DACK0}), J7.B19 (~{DACK0}), J8.B19 (~{DACK0})
- net RESETDRV: now reaches J1.B2 (RESETDRV)
- net RESETDRV: now also J2.B2 (RESETDRV), J3.B2 (RESETDRV), J4.B2 (RESETDRV), J5.B2 (RESETDRV), J6.B2 (RESETDRV), J7.B2 (RESETDRV), J8.B2 (RESETDRV)
- net CLK: now reaches J1.B20 (CLK)
- net CLK: now also J2.B20 (CLK), J3.B20 (CLK), J4.B20 (CLK), J5.B20 (CLK), J6.B20 (CLK), J7.B20 (CLK), J8.B20 (CLK)
- net IRQ7: now reaches J1.B21 (IRQ7)
- net IRQ7: now also J2.B21 (IRQ7), J3.B21 (IRQ7), J4.B21 (IRQ7), J5.B21 (IRQ7), J6.B21 (IRQ7), J7.B21 (IRQ7), J8.B21 (IRQ7)
- net IRQ6: now reaches J1.B22 (IRQ6)
- net IRQ6: now also J2.B22 (IRQ6), J3.B22 (IRQ6), J4.B22 (IRQ6), J5.B22 (IRQ6), J6.B22 (IRQ6), J7.B22 (IRQ6), J8.B22 (IRQ6)
- net IRQ5: now reaches J1.B23 (IRQ5)
- net IRQ5: now also J2.B23 (IRQ5), J3.B23 (IRQ5), J4.B23 (IRQ5), J5.B23 (IRQ5), J6.B23 (IRQ5), J7.B23 (IRQ5), J8.B23 (IRQ5)
- net IRQ4: now reaches J1.B24 (IRQ4)
- net IRQ4: now also J2.B24 (IRQ4), J3.B24 (IRQ4), J4.B24 (IRQ4), J5.B24 (IRQ4), J6.B24 (IRQ4), J7.B24 (IRQ4), J8.B24 (IRQ4)
- net IRQ3: now reaches J1.B25 (IRQ3)
- net IRQ3: now also J2.B25 (IRQ3), J3.B25 (IRQ3), J4.B25 (IRQ3), J5.B25 (IRQ3), J6.B25 (IRQ3), J7.B25 (IRQ3), J8.B25 (IRQ3)
- net ~{DA0K2}': now reaches J1.B26 (~{DACK2})
- net ~{DA0K2}': now also J2.B26 (~{DACK2}), J3.B26 (~{DACK2}), J4.B26 (~{DACK2}), J5.B26 (~{DACK2}), J6.B26 (~{DACK2}), J7.B26 (~{DACK2}), J8.B26 (~{DACK2})
- net T/C: now reaches J1.B27 (T/C)
- net T/C: now also J2.B27 (T/C), J3.B27 (T/C), J4.B27 (T/C), J5.B27 (T/C), J6.B27 (T/C), J7.B27 (T/C), J8.B27 (T/C)
- net ALE: now reaches J1.B28 (ALE)
- net ALE: now also J2.B28 (ALE), J3.B28 (ALE), J4.B28 (ALE), J5.B28 (ALE), J6.B28 (ALE), J7.B28 (ALE), J8.B28 (ALE)
- net +5V: now reaches J1.B29 (+5V)
- net +5V: now also J1.B3 (+5V), C10.1, C11.1, C12.1, C13.1, C14.1, C15.1, C16.1, C17.1, C18.1, C19.1, C20.1, C21.1, C22.1, C23.1, C24.1, C25.1, C26.1, C27.1, C28.1, C29.1, C3.1, C30.1, C31.1, C32.1, C33.1, C34.1, C35.1, C36.1, C37.1, C38.1, C39.1, C40.1, C41.1, C42.1, C43.1, C44.1, C45.1, C46.1, C47.1, C48.1, C49.1, C5.1, C50.1, C51.1, C52.1, C54.1, C59.1, C60.1, C61.1, C62.1, C63.1, C64.1, C65.1, C66.1, J10.10 (Pin_10), J10.11 (Pin_11), J10.12 (Pin_12), J2.B29 (+5V), J2.B3 (+5V), J3.B29 (+5V), J3.B3 (+5V), J4.B29 (+5V), J4.B3 (+5V), J5.B29 (+5V), J5.B3 (+5V), J6.B29 (+5V), J6.B3 (+5V), J7.B29 (+5V), J7.B3 (+5V), J8.B29 (+5V), J8.B3 (+5V)
- net OSC: now reaches J1.B30 (OSC)
- net OSC: now also J2.B30 (OSC), J3.B30 (OSC), J4.B30 (OSC), J5.B30 (OSC), J6.B30 (OSC), J7.B30 (OSC), J8.B30 (OSC)
- net IRQ2: now reaches J1.B4 (IRQ2)
- net IRQ2: now also J2.B4 (IRQ2), J3.B4 (IRQ2), J4.B4 (IRQ2), J5.B4 (IRQ2), J6.B4 (IRQ2), J7.B4 (IRQ2), J8.B4 (IRQ2)
- net -5V: now reaches J1.B5 (-5V)
- net -5V: now also C67.1, C68.1, J10.9 (Pin_9), J2.B5 (-5V), J3.B5 (-5V), J4.B5 (-5V), J5.B5 (-5V), J6.B5 (-5V), J7.B5 (-5V), J8.B5 (-5V)
- net DRQ2: now reaches J1.B6 (DRQ2)
- net DRQ2: now also J2.B6 (DRQ2), J3.B6 (DRQ2), J4.B6 (DRQ2), J5.B6 (DRQ2), J6.B6 (DRQ2), J7.B6 (DRQ2), J8.B6 (DRQ2)
- net -12V: now reaches J1.B7 (-12V)
- net -12V: now also C57.1, C58.1, J10.4 (Pin_4), J2.B7 (-12V), J3.B7 (-12V), J4.B7 (-12V), J5.B7 (-12V), J6.B7 (-12V), J7.B7 (-12V), J8.B7 (-12V)
- net +12V: now reaches J1.B9 (+12V)
- net +12V: now also C55.1, C56.1, J10.3 (Pin_3), J2.B9 (+12V), J3.B9 (+12V), J4.B9 (+12V), J5.B9 (+12V), J6.B9 (+12V), J7.B9 (+12V), J8.B9 (+12V)
- new net PWRGOOD: J10.1 (Pin_1)
- new net XA0: J8.A31 (XA0)
- new net XA1: J8.A30 (XA1)
- new net XA10: J8.A21 (XA10)
- new net XA11: J8.A20 (XA11)
- new net XA12: J8.A19 (XA12)
- new net XA13: J8.A18 (XA13)
- new net XA14: J8.A17 (XA14)
- new net XA15: J8.A16 (XA15)
- new net XA16: J8.A15 (XA16)
- new net XA17: J8.A14 (XA17)
- new net XA18: J8.A13 (XA18)
- new net XA19: J8.A12 (XA19)
- new net XA2: J8.A29 (XA2)
- new net XA3: J8.A28 (XA3)
- new net XA4: J8.A27 (XA4)
- new net XA5: J8.A26 (XA5)
- new net XA6: J8.A25 (XA6)
- new net XA7: J8.A24 (XA7)
- new net XA8: J8.A23 (XA8)
- new net XA9: J8.A22 (XA9)
- new net XD0: J8.A9 (XD0)
- new net XD1: J8.A8 (XD1)
- new net XD2: J8.A7 (XD2)
- new net XD3: J8.A6 (XD3)
- new net XD4: J8.A5 (XD4)
- new net XD5: J8.A4 (XD5)
- new net XD6: J8.A3 (XD6)
- new net XD7: J8.A2 (XD7)
- new net ~{CARDSLCTD}': J8.B8 (~{CARDSLCTD})
- new net ~{XIOR}': J8.B14 (~{XIOR})
- new net ~{XIOW}': J8.B13 (~{XIOW})
- new net ~{YMEMR}': J8.B12 (~{YMEMR})
- new net ~{YMEMW}': J8.B11 (~{YMEMW})
- no-connect marks 0 -> 1
Other:
- moved on the sheet: J1

Commit message: At connector
Parts:
- J10: footprint (none) -> madXT_early:AT_power_connector
Changed lines of the file:
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@@
       (effects (font (size 1.27 1.27)))
     )
-    (property "Footprint" "" (at 352.425 213.36 0)
+    (property "Footprint" "madXT_early:AT_power_connector" (at 352.425 213.36 0)
       (effects (font (size 1.27 1.27)) hide)
     )

Commit message: Update 010502024
Parts:
- C10, C11, C12, C13, C14, C15, C16, C19, C28, C3, C37, C46, C54, C56, C58, C60, C61, C63, C68: footprint (none) -> madXT_early:Cap_unipolar_3pin
- C17, C18, C20, C21, C22, C23, C24, C25, C26, C27, C29, C30, C31, C32, C33, C34, C35, C36, C38, C39, C40, C41, C42, C43, C44, C45, C47, C48, C49, C5, C50, C51, C52, C55, C57, C59, C62, C64, C65, C66, C67: value 0.047pF -> 0.047uF; footprint (none) -> Capacitor_THT:C_Disc_D7.0mm_W2.5mm_P5.00mm

Commit message: Begin tracing
Parts:
- removed C68: 10uF, madXT_early:Cap_unipolar_3pin, symbol Device:C
- added C68: 10uF 25V, madXT_early:cap_tantalum, symbol Device:C_Polarized
- C10, C11, C12, C13, C14, C15, C16, C19, C28, C3, C37, C46, C54, C56, C58, C60, C61, C63: footprint madXT_early:Cap_unipolar_3pin -> madXT_early:cap_tantalum
- C17, C18, C20, C21, C22, C23, C24, C25, C26, C27, C29, C30, C31, C32, C33, C34, C35, C36, C38, C39, C40, C41, C42, C43, C44, C45, C47, C48, C49, C5, C50, C51, C52, C55, C57, C59, C62, C64, C65, C66, C67: footprint Capacitor_THT:C_Disc_D7.0mm_W2.5mm_P5.00mm -> madXT_early:cap_unipolar
Connections:
- net -12V: now also C58.2; no longer C58.1
- net -5V: now also C68.2
- net GND: now also C58.1, C68.1; no longer C58.2

Commit message: Update 03/05/2024
Parts:
- C10, C11, C12, C13, C14, C15, C16, C19, C28, C3, C37, C46, C54, C56, C61, C63: footprint madXT_early:cap_tantalum -> madXT_early:cap_tantalum_pos
- C58, C68: footprint madXT_early:cap_tantalum -> madXT_early:cap_tantalum_neg
- C59: renamed from C60; footprint madXT_early:cap_tantalum -> madXT_early:cap_tantalum_pos
- renumbered C59 to C60
Changed lines of the file:
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@@
   (symbol (lib_id "Device:C_Polarized") (at 332.74 149.86 0) (unit 1)
     (in_bom yes) (on_board yes) (dnp no)
-    (property "Reference" "C60" (at 330.835 142.875 0)
+    (property "Reference" "C59" (at 330.835 142.875 0)
       (effects (font (size 1.27 1.27)) (justify left))
     )
@@
       (effects (font (size 1.27 1.27)) (justify left))
     )
-    (property "Footprint" "madXT_early:cap_tantalum" (at 333.7052 153.67 0)
+    (property "Footprint" "madXT_early:cap_tantalum_pos" (at 333.7052 153.67 0)
       (effects (font (size 1.27 1.27)) hide)
     )
@@
       (project "Mad5160"
         (path "/ac3c86ab-084e-42f6-87ca-c4b0142d8ff2/68a30030-8dd9-4071-b44e-d748bd61ffe4"
-          (reference "C60") (unit 1)
+          (reference "C59") (unit 1)
         )
       )
@@
       (effects (font (size 1.27 1.27)) (justify left))
     )
-    (property "Footprint" "madXT_early:cap_tantalum" (at 298.7802 153.67 0)
+    (property "Footprint" "madXT_early:cap_tantalum_pos" (at 298.7802 153.67 0)
       (effects (font (size 1.27 1.27)) hide)
     )
@@
       (effects (font (size 1.27 1.27)) (justify left))
     )
-    (property "Footprint" "madXT_early:cap_tantalum" (at 284.8102 153.67 0)
+    (property "Footprint" "madXT_early:cap_tantalum_pos" (at 284.8102 153.67 0)
       (effects (font (size 1.27 1.27)) hide)
     )
@@
       (effects (font (size 1.27 1.27)) (justify left))
     )
-    (property "Footprint" "madXT_early:cap_tantalum" (at 263.8552 153.67 0)
+    (property "Footprint" "madXT_early:cap_tantalum_pos" (at 263.8552 153.67 0)
       (effects (font (size 1.27 1.27)) hide)
     )
@@
       (effects (font (size 1.27 1.27)) (justify left))
     )
-    (property "Footprint" "madXT_early:cap_tantalum" (at 185.7502 257.81 0)
+    (property "Footprint" "madXT_early:cap_tantalum_pos" (at 185.7502 257.81 0)
       (effects (font (size 1.27 1.27)) hide)
     )
@@
       (effects (font (size 1.27 1.27)) (justify left))
     )
-    (property "Footprint" "madXT_early:cap_tantalum" (at 242.9002 153.67 0)
+    (property "Footprint" "madXT_early:cap_tantalum_pos" (at 242.9002 153.67 0)
       (effects (font (size 1.27 1.27)) hide)
     )
@@
       (effects (font (size 1.27 1.27)) (justify left))
     )
-    (property "Footprint" "madXT_early:cap_tantalum" (at 347.6752 153.67 0)
+    (property "Footprint" "madXT_early:cap_tantalum_pos" (at 347.6752 153.67 0)
       (effects (font (size 1.27 1.27)) hide)
     )
@@
       (effects (font (size 1.27 1.27)) (justify left))
     )
-    (property "Footprint" "madXT_early:cap_tantalum" (at 291.7952 153.67 0)
+    (property "Footprint" "madXT_early:cap_tantalum_pos" (at 291.7952 153.67 0)
       (effects (font (size 1.27 1.27)) hide)
     )
@@
       (effects (font (size 1.27 1.27)) (justify left))
     )
-    (property "Footprint" "madXT_early:cap_tantalum" (at 270.8402 153.67 0)
+    (property "Footprint" "madXT_early:cap_tantalum_pos" (at 270.8402 153.67 0)
       (effects (font (size 1.27 1.27)) hide)
     )
@@
       (effects (font (size 1.27 1.27)) (justify left))
     )
-    (property "Footprint" "madXT_early:cap_tantalum" (at 225.0948 250.19 0)
+    (property "Footprint" "madXT_early:cap_tantalum_neg" (at 225.0948 250.19 0)
       (effects (font (size 1.27 1.27)) hide)
     )
@@
       (effects (font (size 1.27 1.27)) (justify left))
     )
-    (property "Footprint" "madXT_early:cap_tantalum" (at 263.8298 250.19 0)
+    (property "Footprint" "madXT_early:cap_tantalum_neg" (at 263.8298 250.19 0)
       (effects (font (size 1.27 1.27)) hide)
     )
@@
       (effects (font (size 1.27 1.27)) (justify left))
     )
-    (property "Footprint" "madXT_early:cap_tantalum" (at 249.8852 153.67 0)
+    (property "Footprint" "madXT_early:cap_tantalum_pos" (at 249.8852 153.67 0)
       (effects (font (size 1.27 1.27)) hide)
     )
@@
       (effects (font (size 1.27 1.27)) (justify left))
     )
-    (property "Footprint" "madXT_early:cap_tantalum" (at 326.7202 153.67 0)
+    (property "Footprint" "madXT_early:cap_tantalum_pos" (at 326.7202 153.67 0)
       (effects (font (size 1.27 1.27)) hide)
     )
@@
       (effects (font (size 1.27 1.27)) (justify left))
     )
-    (property "Footprint" "madXT_early:cap_tantalum" (at 256.8702 153.67 0)
+    (property "Footprint" "madXT_early:cap_tantalum_pos" (at 256.8702 153.67 0)
       (effects (font (size 1.27 1.27)) hide)
     )
@@
       (effects (font (size 1.27 1.27)) (justify left))
     )
-    (property "Footprint" "madXT_early:cap_tantalum" (at 305.7652 153.67 0)
+    (property "Footprint" "madXT_early:cap_tantalum_pos" (at 305.7652 153.67 0)
       (effects (font (size 1.27 1.27)) hide)
     )
@@
       (effects (font (size 1.27 1.27)) (justify left))
     )
-    (property "Footprint" "madXT_early:cap_tantalum" (at 312.7502 153.67 0)
+    (property "Footprint" "madXT_early:cap_tantalum_pos" (at 312.7502 153.67 0)
       (effects (font (size 1.27 1.27)) hide)
     )
@@
       (effects (font (size 1.27 1.27)) (justify left))
     )
-    (property "Footprint" "madXT_early:cap_tantalum" (at 340.6902 153.67 0)
+    (property "Footprint" "madXT_early:cap_tantalum_pos" (at 340.6902 153.67 0)
       (effects (font (size 1.27 1.27)) hide)
     )
@@
       (effects (font (size 1.27 1.27)) (justify left))
     )
-    (property "Footprint" "madXT_early:cap_tantalum" (at 277.8252 153.67 0)
+    (property "Footprint" "madXT_early:cap_tantalum_pos" (at 277.8252 153.67 0)
       (effects (font (size 1.27 1.27)) hide)
     )
@@
   (symbol (lib_id "Device:C") (at 372.745 172.085 0) (unit 1)
     (in_bom yes) (on_board yes) (dnp no)
-    (property "Reference" "C59" (at 370.84 165.1 0)
+    (property "Reference" "C60" (at 370.84 165.1 0)
       (effects (font (size 1.27 1.27)) (justify left))
     )
@@
       (project "Mad5160"
         (path "/ac3c86ab-084e-42f6-87ca-c4b0142d8ff2/68a30030-8dd9-4071-b44e-d748bd61ffe4"
-          (reference "C59") (unit 1)
+          (reference "C60") (unit 1)
         )
       )
@@
       (effects (font (size 1.27 1.27)) (justify left))
     )
-    (property "Footprint" "madXT_early:cap_tantalum" (at 319.7352 153.67 0)
+    (property "Footprint" "madXT_early:cap_tantalum_pos" (at 319.7352 153.67 0)
       (effects (font (size 1.27 1.27)) hide)
     )

Commit message: Tracing for version 1.0 finished
Parts:
- added U90: SPARE, madXT_early:spare, symbol Mad5150_early:spare_IC
Connections:
- new net: U90.1, U90.17
- new net: U90.10, U90.26
- new net: U90.11, U90.27
- new net: U90.12, U90.28
- new net: U90.13, U90.29
- new net: U90.14, U90.30
- new net: U90.15, U90.31
- new net: U90.16, U90.32
- new net: U90.18, U90.2
- new net: U90.19, U90.3
- new net: U90.20, U90.4
- new net: U90.21, U90.5
- new net: U90.22, U90.6
- new net: U90.23, U90.24, U90.33, U90.34, U90.7, U90.8
- new net: U90.25, U90.9
Other:
- moved on the sheet: J10

Commit message: Tracing finished
Parts:
- C10, C11, C12, C13, C14, C15, C16, C19, C28, C3, C37, C46, C54, C56, C59, C61, C63: footprint madXT_early:cap_tantalum_pos -> mad5150:cap_tantalum_pos
- C17, C18, C20, C21, C22, C23, C24, C25, C26, C27, C29, C30, C31, C32, C33, C34, C35, C36, C38, C39, C40, C41, C42, C43, C44, C45, C47, C48, C49, C5, C50, C51, C52, C55, C57, C60, C62, C64, C65, C66, C67: footprint madXT_early:cap_unipolar -> mad5150:cap_unipolar
- C58, C68: footprint madXT_early:cap_tantalum_neg -> mad5150:cap_tantalum_neg
- J1, J2, J3, J4, J5, J6, J7, J8: footprint madXT_early:isa_edge_slot -> mad5150:isa_edge_slot
- J10: footprint madXT_early:AT_power_connector -> mad5150:AT_power_connector
- U90: footprint madXT_early:spare -> mad5150:spare
