File: sheet5.kicad_sch (KiCad schematic)
At the start: 11 parts, among them U13 LS243_U13, U14 LS244, U15 LS245, U16 LS244, U17 LS244, U18 27C256 (32KX8), U19 27C256 (32KX8), U23 LS27_U23, U24 LS00_U24, U9 LS244

Commit message: Sheet 5 finished
Parts:
- U13: footprint Package_DIP:DIP-12_W7.62mm_LongPads -> Package_DIP:DIP-14_W7.62mm_LongPads
Connections:
- net XA10: now also U16.12 (O3a)
- net XA11: now also U16.14 (O2a)
- net XA12: now also U16.18 (O0a)
- net XA13: now also U14.9 (O0b)
- net XA14: now also U14.12 (O3a)
- net XA8: now also U16.5 (O2b), U23.13
- net XA9: now also U16.7 (O1b), U23.2
- net GND: now reaches U15.10 (GND)
- net GND: now also U13.7 (GND), U14.1 (OEa), U14.10 (GND), U14.19 (OEb), U16.1 (OEa), U16.10 (GND), U16.19 (OEb), U17.10 (GND), U18.14 (GND), U19.14 (GND), U23.7 (GND)
- net +5V: now reaches U15.20 (VCC)
- net +5V: now also RN1.16, RN1.16, RN1.16, RN1.16, RN1.16, U13.14 (VCC), U14.20 (VCC), U16.20 (VCC), U17.20 (VCC), U18.28 (VCC), U19.28 (VCC), U23.14 (VCC)
- net XD0: now reaches U19.11 (D0)
- net XD0: now also U15.18 (B0), U18.11 (D0)
- net XD1: now reaches U19.12 (D1)
- net XD1: now also U15.17 (B1), U18.12 (D1)
- net XD2: now reaches U19.13 (D2)
- net XD2: now also U15.16 (B2), U18.13 (D2)
- net XD3: now reaches U19.15 (D3)
- net XD3: now also U15.15 (B3), U18.15 (D3)
- net XD4: now reaches U19.16 (D4)
- net XD4: now also U15.14 (B4), U18.16 (D4)
- net XD5: now reaches U19.17 (D5)
- net XD5: now also U15.13 (B5), U18.17 (D5)
- net XD6: now reaches U19.18 (D6)
- net XD6: now also U15.12 (B6), U18.18 (D6)
- net XD7: now reaches U19.19 (D7)
- net XD7: now also U15.11 (B7), U18.19 (D7)
- net ~{XMEMW}': now reaches RN1.3
- net ~{XMEMW}': now also U13.5 (A2), U14.2 (I0a)
- net ~{XIOR}': now reaches RN1.4
- net ~{XIOR}': now also U13.6 (A3), U23.1
- net at U9.1 (OEa): now also U15.19 (CE), U9.19 (OEb)
- net at U23.3: now also U23.12
- net at U23.4: now also U24.11
- net ROMADDRSEL: now reaches U23.5
- net at U23.6: now also U15.1 (A->B)
- net ~{XIOW}': now reaches RN1.2
- net ~{XIOW}': now also U13.4 (A1)
- net ~{CARDSLCTD}': now reaches RN1.10
- net ~{CARDSLCTD}': now also U24.13
- net ~{DA0K0BRD}': now reaches U16.11 (I0b)
- net A9: now reaches U16.13 (I1b)
- net A8: now reaches U16.15 (I2b)
- net CLK: now reaches U16.16 (O1a)
- net AENBRD: now reaches U16.17 (I3b)
- net A12: now reaches U16.2 (I0a)
- net AEN: now reaches U16.3 (O3b)
- net CLK88: now reaches U16.4 (I1a)
- net A11: now reaches U16.6 (I2a)
- net A10: now reaches U16.8 (I3a)
- net ~{DACK0}': now reaches U16.9 (O0b)
- net ~{DMAAEN}': now reaches U13.1 (OEa)
- net ~{DMAAEN}': now also U13.13 (OEb)
- net ~{IOW}': now reaches U13.10 (B1)
- net ~{MEMR}': now reaches U13.11 (B0)
- net ~{XMEMR}': now reaches U13.3 (A0)
- net ~{XMEMR}': now also RN1.1
- net ~{IOR}': now reaches U13.8 (B3)
- net ~{MEMW}': now reaches U13.9 (B2)
- net ~{INTA}': now reaches U24.12
- net D0: now reaches U15.2 (A0)
- net D1: now reaches U15.3 (A1)
- net D2: now reaches U15.4 (A2)
- net D3: now reaches U15.5 (A3)
- net D4: now reaches U15.6 (A4)
- net D5: now reaches U15.7 (A5)
- net D6: now reaches U15.8 (A6)
- net D7: now reaches U15.9 (A7)
- net A13: now reaches U14.11 (I0b)
- net A15: now reaches U14.13 (I1b)
- net XA16: now reaches U14.14 (O2a)
- net A17: now reaches U14.15 (I2b)
- net XA18: now reaches U14.16 (O1a)
- net A19: now reaches U14.17 (I3b)
- net ~{YMEMW}': now reaches U14.18 (O0a)
- net XA19: now reaches U14.3 (O3b)
- net A18: now reaches U14.4 (I1a)
- net XA17: now reaches U14.5 (O2b)
- net A16: now reaches U14.6 (I2a)
- net XA15: now reaches U14.7 (O1b)
- net A14: now reaches U14.8 (I3a)
Other:
- moved on the sheet: RN1A, RN1B, RN1C, RN1D, RN1J, U13A, U13B, U14A, U14B, U15A, U15B, U16A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

Commit message: Working on sheet 6
Parts:
- removed unit 3 of U23
- renumbered U9 to U17
Changed lines of the file:
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@@
   (symbol (lib_id "Mad5150_early:LS244_U17") (at 62.865 34.925 0) (unit 1)
     (in_bom yes) (on_board yes) (dnp no) (fields_autoplaced)
-    (property "Reference" "U9" (at 62.865 19.685 0)
+    (property "Reference" "U17" (at 62.865 19.685 0)
       (effects (font (size 1.27 1.27)))
     )
@@
       (project "Mad5160"
         (path "/ac3c86ab-084e-42f6-87ca-c4b0142d8ff2/c44b5552-e284-433f-baff-8fd8b9b71db6"
-          (reference "U9") (unit 1)
+          (reference "U17") (unit 1)
         )
       )
@@
         )
       )
-    )
-  )
-  (symbol (lib_id "Mad5150_early:LS27_U23") (at 453.39 62.865 0) (unit 3)
-    (in_bom yes) (on_board yes) (dnp no) (fields_autoplaced)
-    (property "Reference" "U23" (at 453.39 53.975 0)
-      (effects (font (size 1.27 1.27)))
-    )
-    (property "Value" "LS27_U23" (at 453.39 56.515 0)
-      (effects (font (size 1.27 1.27)))
-    )
-    (property "Footprint" "Package_DIP:DIP-14_W7.62mm" (at 452.12 73.025 0)
-      (effects (font (size 1.27 1.27)) hide)
-    )
-    (property "Datasheet" "http://www.ti.com/lit/gpn/sn74LS27" (at 453.39 70.485 0)
-      (effects (font (size 1.27 1.27)) hide)
-    )
-    (pin "7")
-    (pin "11")
-    (pin "8")
-    (pin "4")
-    (pin "3")
-    (pin "10")
-    (pin "13")
-    (pin "9")
-    (pin "1")
-    (pin "6")
-    (pin "14")
-    (pin "12")
-    (pin "5")
-    (pin "2")
-    (instances
-      (project "Mad5160"
-        (path "/ac3c86ab-084e-42f6-87ca-c4b0142d8ff2/c44b5552-e284-433f-baff-8fd8b9b71db6"
-          (reference "U23") (unit 3)
-        )
-      )

Commit message: Sheet 10 done
Parts:
- RN1: symbol Mad5150_early:Resistor_Network -> Mad5150_early:Resistor_Network_1
Changed lines of the file:
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@@
     )
   )
-  (symbol (lib_id "Mad5150_early:Resistor_Network") (at 226.06 208.28 180) (unit 3)
+  (symbol (lib_id "Mad5150_early:Resistor_Network_1") (at 226.06 208.28 180) (unit 3)
     (in_bom yes) (on_board yes) (dnp no) (fields_autoplaced)
     (property "Reference" "RN1" (at 228.6 207.01 0)
@@
     )
   )
-  (symbol (lib_id "Mad5150_early:Resistor_Network") (at 236.855 208.28 180) (unit 4)
-    (in_bom yes) (on_board yes) (dnp no) (fields_autoplaced)
-    (property "Reference" "RN1" (at 239.395 207.01 0)
+  (symbol (lib_id "Mad5150_early:Resistor_Network_1") (at 236.855 208.28 180) (unit 4)
+    (in_bom yes) (on_board yes) (dnp no) (fields_autoplaced)
+    (property "Reference" "RN1" (at 238.76 207.01 0)
       (effects (font (size 1.27 1.27)) (justify right))
     )
-    (property "Value" "4.7K" (at 239.395 209.55 0)
+    (property "Value" "4.7K" (at 238.76 209.55 0)
       (effects (font (size 1.27 1.27)) (justify right))
     )
@@
     )
   )
-  (symbol (lib_id "Mad5150_early:Resistor_Network") (at 215.9 208.28 180) (unit 2)
+  (symbol (lib_id "Mad5150_early:Resistor_Network_1") (at 215.9 208.28 180) (unit 2)
     (in_bom yes) (on_board yes) (dnp no) (fields_autoplaced)
     (property "Reference" "RN1" (at 218.44 207.01 0)
@@
     )
   )
-  (symbol (lib_id "Mad5150_early:Resistor_Network") (at 76.2 238.125 180) (unit 10)
+  (symbol (lib_id "Mad5150_early:Resistor_Network_1") (at 76.2 238.125 180) (unit 10)
     (in_bom yes) (on_board yes) (dnp no) (fields_autoplaced)
     (property "Reference" "RN1" (at 78.74 236.855 0)
@@
     )
   )
-  (symbol (lib_id "Mad5150_early:Resistor_Network") (at 205.105 208.28 180) (unit 1)
+  (symbol (lib_id "Mad5150_early:Resistor_Network_1") (at 205.105 208.28 180) (unit 1)
     (in_bom yes) (on_board yes) (dnp no) (fields_autoplaced)
     (property "Reference" "RN1" (at 207.01 207.01 0)

Commit message: Update 010502024
Connections:
- net AENBRD: now also U15.19 (CE), U17.1 (OEa), U17.19 (OEb)
Changed lines of the file:
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@@
   (junction (at 205.74 250.19) (diameter 0) (color 0 0 0 0)
   )
+  (junction (at 43.18 148.59) (diameter 0) (color 0 0 0 0)
+  )
   (junction (at 122.555 34.925) (diameter 0) (color 0 0 0 0)
   )
@@
     (stroke (width 0) (type default))
   )
-  (wire (pts (xy 43.18 206.375) (xy 43.18 53.34))
+  (wire (pts (xy 43.18 206.375) (xy 43.18 148.59))
     (stroke (width 0) (type default))
   )
@@
     (stroke (width 0) (type default))
   )
-  (wire (pts (xy 38.735 148.59) (xy 48.26 148.59))
+  (wire (pts (xy 38.735 148.59) (xy 43.18 148.59))
     (stroke (width 0) (type default))
   )
@@
     (stroke (width 0) (type default))
   )
+  (wire (pts (xy 43.18 148.59) (xy 43.18 53.34))
+    (stroke (width 0) (type default))
+  )
   (bus (pts (xy 248.285 73.66) (xy 248.285 76.2))
     (stroke (width 0) (type default))
@@
     (stroke (width 0) (type default))
   )
+  (wire (pts (xy 65.405 51.435) (xy 65.405 53.34))
+    (stroke (width 0) (type default))
+  )
   (wire (pts (xy 74.295 225.425) (xy 95.885 225.425))
     (stroke (width 0) (type default))
@@
     (stroke (width 0) (type default))
   )
+  (wire (pts (xy 43.18 148.59) (xy 48.26 148.59))
+    (stroke (width 0) (type default))
+  )
   (bus (pts (xy 237.49 177.8) (xy 237.49 180.34))
     (stroke (width 0) (type default))
@@
     (stroke (width 0) (type default))
   )
-  (wire (pts (xy 65.405 53.34) (xy 65.405 51.435))
-    (stroke (width 0) (type default))
-  )

Commit message: Update 03/05/2024
Parts:
- U13: footprint Package_DIP:DIP-14_W7.62mm_LongPads -> Package_DIP:DIP-14_W7.62mm
Changed lines of the file:
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@@
       (effects (font (size 1.27 1.27) bold))
     )
-    (property "Footprint" "Package_DIP:DIP-14_W7.62mm_LongPads" (at 61.595 225.425 0)
+    (property "Footprint" "Package_DIP:DIP-14_W7.62mm" (at 61.595 225.425 0)
       (effects (font (size 1.27 1.27)) hide)
     )
@@
       (effects (font (size 1.27 1.27) bold) (justify left))
     )
-    (property "Footprint" "Package_DIP:DIP-14_W7.62mm_LongPads" (at 205.74 267.97 0)
+    (property "Footprint" "Package_DIP:DIP-14_W7.62mm" (at 205.74 267.97 0)
       (effects (font (size 1.27 1.27)) hide)
     )

Commit message: Tracing finished
Parts:
- RN1: footprint Package_DIP:DIP-16_W7.62mm -> mad5150:DIP-16_W7.62mm
- U13, U23, U24: footprint Package_DIP:DIP-14_W7.62mm -> mad5150:DIP-14_W7.62mm
- U14, U15, U16, U17: footprint Package_DIP:DIP-20_W7.62mm -> mad5150:DIP-20_W7.62mm
- U18, U19: footprint Package_DIP:DIP-28_W15.24mm -> mad5150:DIP-28_W15.24mm
Changed lines of the file:
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@@
       (effects (font (size 1.27 1.27)) (justify left))
     )
-    (property "Footprint" "Package_DIP:DIP-20_W7.62mm" (at 189.23 267.97 0)
+    (property "Footprint" "mad5150:DIP-20_W7.62mm" (at 189.23 267.97 0)
       (effects (font (size 1.27 1.27)) hide)
     )
@@
       (effects (font (size 1.27 1.27)) (justify left))
     )
-    (property "Footprint" "Package_DIP:DIP-28_W15.24mm" (at 250.19 300.99 0)
+    (property "Footprint" "mad5150:DIP-28_W15.24mm" (at 250.19 300.99 0)
       (effects (font (size 1.27 1.27)) hide)
     )
@@
       (effects (font (size 1.27 1.27)))
     )
-    (property "Footprint" "Package_DIP:DIP-28_W15.24mm" (at 136.525 144.78 0)
+    (property "Footprint" "mad5150:DIP-28_W15.24mm" (at 136.525 144.78 0)
       (effects (font (size 1.27 1.27)) hide)
     )
@@
       (effects (font (size 1.27 1.27)) (justify right))
     )
-    (property "Footprint" "Package_DIP:DIP-16_W7.62mm" (at 226.06 208.28 0)
+    (property "Footprint" "mad5150:DIP-16_W7.62mm" (at 226.06 208.28 0)
       (effects (font (size 1.27 1.27)) hide)
     )
@@
       (effects (font (size 1.27 1.27) bold) (justify left))
     )
-    (property "Footprint" "Package_DIP:DIP-20_W7.62mm" (at 131.445 263.525 0)
+    (property "Footprint" "mad5150:DIP-20_W7.62mm" (at 131.445 263.525 0)
       (effects (font (size 1.27 1.27)) hide)
     )
@@
       (effects (font (size 1.27 1.27)) (justify right))
     )
-    (property "Footprint" "Package_DIP:DIP-16_W7.62mm" (at 236.855 208.28 0)
+    (property "Footprint" "mad5150:DIP-16_W7.62mm" (at 236.855 208.28 0)
       (effects (font (size 1.27 1.27)) hide)
     )
@@
       (effects (font (size 1.27 1.27) bold))
     )
-    (property "Footprint" "Package_DIP:DIP-20_W7.62mm" (at 62.865 34.925 0)
+    (property "Footprint" "mad5150:DIP-20_W7.62mm" (at 62.865 34.925 0)
       (effects (font (size 1.27 1.27)) hide)
     )
@@
       (effects (font (size 1.27 1.27)))
     )
-    (property "Footprint" "Package_DIP:DIP-14_W7.62mm" (at 144.145 219.71 0)
+    (property "Footprint" "mad5150:DIP-14_W7.62mm" (at 144.145 219.71 0)
       (effects (font (size 1.27 1.27)) hide)
     )
@@
       (effects (font (size 1.27 1.27)) (justify right))
     )
-    (property "Footprint" "Package_DIP:DIP-16_W7.62mm" (at 215.9 208.28 0)
+    (property "Footprint" "mad5150:DIP-16_W7.62mm" (at 215.9 208.28 0)
       (effects (font (size 1.27 1.27)) hide)
     )
@@
       (effects (font (size 1.27 1.27)) (justify right))
     )
-    (property "Footprint" "Package_DIP:DIP-16_W7.62mm" (at 76.2 238.125 0)
+    (property "Footprint" "mad5150:DIP-16_W7.62mm" (at 76.2 238.125 0)
       (effects (font (size 1.27 1.27)) hide)
     )
@@
       (effects (font (size 1.27 1.27) bold) (justify left))
     )
-    (property "Footprint" "Package_DIP:DIP-20_W7.62mm" (at 169.545 263.525 0)
+    (property "Footprint" "mad5150:DIP-20_W7.62mm" (at 169.545 263.525 0)
       (effects (font (size 1.27 1.27)) hide)
     )
@@
       (effects (font (size 1.27 1.27) bold))
     )
-    (property "Footprint" "Package_DIP:DIP-20_W7.62mm" (at 62.23 144.78 0)
+    (property "Footprint" "mad5150:DIP-20_W7.62mm" (at 62.23 144.78 0)
       (effects (font (size 1.27 1.27)) hide)
     )
@@
       (effects (font (size 1.27 1.27)))
     )
-    (property "Footprint" "Package_DIP:DIP-28_W15.24mm" (at 136.525 90.805 0)
+    (property "Footprint" "mad5150:DIP-28_W15.24mm" (at 136.525 90.805 0)
       (effects (font (size 1.27 1.27)) hide)
     )
@@
       (effects (font (size 1.27 1.27)) (justify left))
     )
-    (property "Footprint" "Package_DIP:DIP-28_W15.24mm" (at 276.86 300.99 0)
+    (property "Footprint" "mad5150:DIP-28_W15.24mm" (at 276.86 300.99 0)
       (effects (font (size 1.27 1.27)) hide)
     )
@@
       (effects (font (size 1.27 1.27)) (justify left))
     )
-    (property "Footprint" "Package_DIP:DIP-14_W7.62mm" (at 226.06 273.685 0)
+    (property "Footprint" "mad5150:DIP-14_W7.62mm" (at 226.06 273.685 0)
       (effects (font (size 1.27 1.27)) hide)
     )
@@
       (effects (font (size 1.27 1.27) bold))
     )
-    (property "Footprint" "Package_DIP:DIP-14_W7.62mm" (at 61.595 225.425 0)
+    (property "Footprint" "mad5150:DIP-14_W7.62mm" (at 61.595 225.425 0)
       (effects (font (size 1.27 1.27)) hide)
     )
@@
       (effects (font (size 1.27 1.27) bold) (justify left))
     )
-    (property "Footprint" "Package_DIP:DIP-20_W7.62mm" (at 150.495 263.525 0)
+    (property "Footprint" "mad5150:DIP-20_W7.62mm" (at 150.495 263.525 0)
       (effects (font (size 1.27 1.27)) hide)
     )
@@
       (effects (font (size 1.27 1.27)))
     )
-    (property "Footprint" "Package_DIP:DIP-14_W7.62mm" (at 93.98 247.015 0)
+    (property "Footprint" "mad5150:DIP-14_W7.62mm" (at 93.98 247.015 0)
       (effects (font (size 1.27 1.27)) hide)
     )
@@
       (effects (font (size 1.27 1.27)) (justify right))
     )
-    (property "Footprint" "Package_DIP:DIP-16_W7.62mm" (at 205.105 208.28 0)
+    (property "Footprint" "mad5150:DIP-16_W7.62mm" (at 205.105 208.28 0)
       (effects (font (size 1.27 1.27)) hide)
     )
@@
       (effects (font (size 1.27 1.27) bold) (justify left))
     )
-    (property "Footprint" "Package_DIP:DIP-14_W7.62mm" (at 205.74 267.97 0)
+    (property "Footprint" "mad5150:DIP-14_W7.62mm" (at 205.74 267.97 0)
       (effects (font (size 1.27 1.27)) hide)
     )
@@
       (effects (font (size 1.27 1.27)))
     )
-    (property "Footprint" "Package_DIP:DIP-20_W7.62mm" (at 61.595 190.5 0)
+    (property "Footprint" "mad5150:DIP-20_W7.62mm" (at 61.595 190.5 0)
       (effects (font (size 1.27 1.27)) hide)
     )
@@
       (effects (font (size 1.27 1.27)))
     )
-    (property "Footprint" "Package_DIP:DIP-14_W7.62mm" (at 116.84 217.17 0)
+    (property "Footprint" "mad5150:DIP-14_W7.62mm" (at 116.84 217.17 0)
       (effects (font (size 1.27 1.27)) hide)
     )
@@
       (effects (font (size 1.27 1.27) bold))
     )
-    (property "Footprint" "Package_DIP:DIP-20_W7.62mm" (at 62.865 96.52 0)
-      (effects (font (size 1.27 1.27)) hide)
-    )
+    (property "Footprint" "mad5150:DIP-20_W7.62mm" (at 62.865 96.52 0)
+      (effects (font (size 1.27 1.27)) hide)
+    )
