File: sheet5.kicad_sch (KiCad schematic)
At the start: 10 parts, among them U13 LS243_U13, U14 LS244, U15 LS245, U16 LS244, U17 LS244, U18 27C256 (32KX8), U19 27C256 (32KX8), U23 LS27_U23, U24 LS00_U24

Commit message: Fixing stuff
Connections:
- net ~{XIOR}': now also RN1.3; no longer RN1.4
- net ~{XMEMW}': now also RN1.4; no longer RN1.3
Changed lines of the file:
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@@
   (junction (at 226.06 200.66) (diameter 0) (color 0 0 0 0)
   )
+  (junction (at 215.9 220.345) (diameter 0) (color 0 0 0 0)
+  )
   (junction (at 227.33 278.13) (diameter 0) (color 0 0 0 0)
   )
-  (junction (at 215.9 220.345) (diameter 0) (color 0 0 0 0)
-  )
   (junction (at 161.925 193.04) (diameter 0) (color 0 0 0 0)
   )
@@
     (stroke (width 0) (type default))
   )
-  (wire (pts (xy 265.43 220.345) (xy 265.43 220.98))
-    (stroke (width 0) (type default))
-  )
   (bus (pts (xy 248.285 68.58) (xy 248.285 71.12))
     (stroke (width 0) (type default))
@@
     (stroke (width 0) (type default))
   )
+  (wire (pts (xy 101.6 247.015) (xy 130.81 247.015))
+    (stroke (width 0) (type default))
+  )
+  (wire (pts (xy 205.74 250.19) (xy 205.74 252.73))
+    (stroke (width 0) (type default))
+  )
+  (wire (pts (xy 250.825 35.56) (xy 267.335 35.56))
+    (stroke (width 0) (type default))
+  )
+  (wire (pts (xy 130.81 247.015) (xy 130.81 212.09))
+    (stroke (width 0) (type default))
+  )
+  (bus (pts (xy 248.285 60.96) (xy 248.285 63.5))
+    (stroke (width 0) (type default))
+  )
+  (wire (pts (xy 59.055 203.2) (xy 59.055 208.915))
+    (stroke (width 0) (type default))
+  )
+  (bus (pts (xy 161.925 109.22) (xy 161.925 111.76))
+    (stroke (width 0) (type default))
+  )
   (wire (pts (xy 215.9 213.995) (xy 215.9 220.345))
-    (stroke (width 0) (type default))
-  )
-  (wire (pts (xy 101.6 247.015) (xy 130.81 247.015))
-    (stroke (width 0) (type default))
-  )
-  (wire (pts (xy 205.74 250.19) (xy 205.74 252.73))
-    (stroke (width 0) (type default))
-  )
-  (wire (pts (xy 250.825 35.56) (xy 267.335 35.56))
-    (stroke (width 0) (type default))
-  )
-  (wire (pts (xy 130.81 247.015) (xy 130.81 212.09))
-    (stroke (width 0) (type default))
-  )
-  (bus (pts (xy 248.285 60.96) (xy 248.285 63.5))
-    (stroke (width 0) (type default))
-  )
-  (wire (pts (xy 59.055 203.2) (xy 59.055 208.915))
-    (stroke (width 0) (type default))
-  )
-  (bus (pts (xy 161.925 109.22) (xy 161.925 111.76))
     (stroke (width 0) (type default))
   )
@@
         (path "/ac3c86ab-084e-42f6-87ca-c4b0142d8ff2/c44b5552-e284-433f-baff-8fd8b9b71db6"
           (reference "U15") (unit 2)
+        )
+      )
+    )
+  )
+  (symbol (lib_id "Mad5150_early:Resistor_Network_1") (at 236.855 208.28 180) (unit 3)
+    (in_bom yes) (on_board yes) (dnp no) (fields_autoplaced)
+    (property "Reference" "RN1" (at 239.395 207.01 0)
+      (effects (font (size 1.27 1.27)) (justify right))
+    )
+    (property "Value" "4.7K" (at 239.395 209.55 0)
+      (effects (font (size 1.27 1.27)) (justify right))
+    )
+    (property "Footprint" "mad5150:DIP-16_W7.62mm" (at 236.855 208.28 0)
+      (effects (font (size 1.27 1.27)) hide)
+    )
+    (property "Datasheet" "" (at 236.22 208.915 0)
+      (effects (font (size 1.27 1.27)) hide)
+    )
+    (pin "1")
+    (pin "16")
+    (pin "16")
+    (pin "2")
+    (pin "16")
+    (pin "3")
+    (pin "16")
+    (pin "4")
+    (pin "16")
+    (pin "5")
+    (pin "16")
+    (pin "6")
+    (pin "16")
+    (pin "7")
+    (pin "16")
+    (pin "8")
+    (pin "16")
+    (pin "9")
+    (pin "10")
+    (pin "16")
+    (pin "11")
+    (pin "16")
+    (pin "12")
+    (pin "16")
+    (pin "13")
+    (pin "16")
+    (pin "14")
+    (pin "16")
+    (pin "15")
+    (pin "16")
+    (instances
+      (project "Mad5160"
+        (path "/ac3c86ab-084e-42f6-87ca-c4b0142d8ff2/c44b5552-e284-433f-baff-8fd8b9b71db6"
+          (reference "RN1") (unit 3)
+        )
+      )
+    )
+  )
+  (symbol (lib_id "Mad5150_early:Resistor_Network_1") (at 226.06 208.28 180) (unit 4)
+    (in_bom yes) (on_board yes) (dnp no) (fields_autoplaced)
+    (property "Reference" "RN1" (at 227.965 207.01 0)
+      (effects (font (size 1.27 1.27)) (justify right))
+    )
+    (property "Value" "4.7K" (at 227.965 209.55 0)
+      (effects (font (size 1.27 1.27)) (justify right))
+    )
+    (property "Footprint" "mad5150:DIP-16_W7.62mm" (at 226.06 208.28 0)
+      (effects (font (size 1.27 1.27)) hide)
+    )
+    (property "Datasheet" "" (at 225.425 208.915 0)
+      (effects (font (size 1.27 1.27)) hide)
+    )
+    (pin "1")
+    (pin "16")
+    (pin "16")
+    (pin "2")
+    (pin "16")
+    (pin "3")
+    (pin "16")
+    (pin "4")
+    (pin "16")
+    (pin "5")
+    (pin "16")
+    (pin "6")
+    (pin "16")
+    (pin "7")
+    (pin "16")
+    (pin "8")
+    (pin "16")
+    (pin "9")
+    (pin "10")
+    (pin "16")
+    (pin "11")
+    (pin "16")
+    (pin "12")
+    (pin "16")
+    (pin "13")
+    (pin "16")
+    (pin "14")
+    (pin "16")
+    (pin "15")
+    (pin "16")
+    (instances
+      (project "Mad5160"
+        (path "/ac3c86ab-084e-42f6-87ca-c4b0142d8ff2/c44b5552-e284-433f-baff-8fd8b9b71db6"
+          (reference "RN1") (unit 4)
         )
       )
@@
     )
   )
-  (symbol (lib_id "Mad5150_early:Resistor_Network_1") (at 226.06 208.28 180) (unit 3)
-    (in_bom yes) (on_board yes) (dnp no) (fields_autoplaced)
-    (property "Reference" "RN1" (at 228.6 207.01 0)
-      (effects (font (size 1.27 1.27)) (justify right))
-    )
-    (property "Value" "4.7K" (at 228.6 209.55 0)
-      (effects (font (size 1.27 1.27)) (justify right))
-    )
-    (property "Footprint" "mad5150:DIP-16_W7.62mm" (at 226.06 208.28 0)
-      (effects (font (size 1.27 1.27)) hide)
-    )
-    (property "Datasheet" "" (at 225.425 208.915 0)
-      (effects (font (size 1.27 1.27)) hide)
-    )
-    (pin "1")
-    (pin "16")
-    (pin "16")
-    (pin "2")
-    (pin "16")
-    (pin "3")
-    (pin "16")
-    (pin "4")
-    (pin "16")
-    (pin "5")
-    (pin "16")
-    (pin "6")
-    (pin "16")
-    (pin "7")
-    (pin "16")
-    (pin "8")
-    (pin "16")
-    (pin "9")
-    (pin "10")
-    (pin "16")
-    (pin "11")
-    (pin "16")
-    (pin "12")
-    (pin "16")
-    (pin "13")
-    (pin "16")
-    (pin "14")
-    (pin "16")
-    (pin "15")
-    (pin "16")
-    (instances
-      (project "Mad5160"
-        (path "/ac3c86ab-084e-42f6-87ca-c4b0142d8ff2/c44b5552-e284-433f-baff-8fd8b9b71db6"
-          (reference "RN1") (unit 3)
-        )
-      )
-    )
-  )
   (symbol (lib_id "Mad5150_early:LS244_U17") (at 131.445 263.525 0) (unit 2)
     (in_bom yes) (on_board yes) (dnp no) (fields_autoplaced)
@@
         )
       )
-    )
-  )
-  (symbol (lib_id "Mad5150_early:Resistor_Network_1") (at 236.855 208.28 180) (unit 4)
-    (in_bom yes) (on_board yes) (dnp no) (fields_autoplaced)
-    (property "Reference" "RN1" (at 238.76 207.01 0)
-      (effects (font (size 1.27 1.27)) (justify right))
-    )
-    (property "Value" "4.7K" (at 238.76 209.55 0)
-      (effects (font (size 1.27 1.27)) (justify right))
-    )
-    (property "Footprint" "mad5150:DIP-16_W7.62mm" (at 236.855 208.28 0)
-      (effects (font (size 1.27 1.27)) hide)
-    )
-    (property "Datasheet" "" (at 236.22 208.915 0)
-      (effects (font (size 1.27 1.27)) hide)
-    )
-    (pin "1")
-    (pin "16")
-    (pin "16")
-    (pin "2")
-    (pin "16")
-    (pin "3")
-    (pin "16")
-    (pin "4")
-    (pin "16")
-    (pin "5")
-    (pin "16")
-    (pin "6")
-    (pin "16")
-    (pin "7")
-    (pin "16")
-    (pin "8")
-    (pin "16")
-    (pin "9")
-    (pin "10")
-    (pin "16")
-    (pin "11")
-    (pin "16")
-    (pin "12")
-    (pin "16")
-    (pin "13")
-    (pin "16")
-    (pin "14")
-    (pin "16")
-    (pin "15")
-    (pin "16")
-    (instances
-      (project "Mad5160"
-        (path "/ac3c86ab-084e-42f6-87ca-c4b0142d8ff2/c44b5552-e284-433f-baff-8fd8b9b71db6"
-          (reference "RN1") (unit 4)
-        )
-      )
