File: sheet6.kicad_sch (KiCad schematic)
At the start: 32 parts, among them U20 S280_U20, U23 LS27_U23, U30 64K x1 bit RAM 4164, U31 64K x1 bit RAM 4164, U32 64K x1 bit RAM 4164, U33 64K x1 bit RAM 4164, U34 64K x1 bit RAM 4164, U35 64K x1 bit RAM 4164, U36 64K x1 bit RAM 4164, U37 64K x1 bit RAM 4164, U38 64K x1 bit RAM 4164, U39 LS158_U39, U40 LS158_U39, U46 64K x1 bit RAM 4164, U47 64K x1 bit RAM 4164, U48 64K x1 bit RAM 4164, U49 64K x1 bit RAM 4164, U50 64K x1 bit RAM 4164, U51 64K x1 bit RAM 4164, U52 64K x1 bit RAM 4164, U53 64K x1 bit RAM 4164, U54 64K x1 bit RAM 4164, U58 LS32_U58, U84 LS158_U39, U86 S74_U70, U87 S08_U87, U89 LS04_U71, U9 LS245

Commit message: Sheet 7
Parts:
- added unit 1 of RN4
Connections:
- net ~{CAS0} is gone; now on net ~{CAS0}': U31.15 (~{CAS}), U32.15 (~{CAS}), U33.15 (~{CAS}), U34.15 (~{CAS}), U35.15 (~{CAS}), U36.15 (~{CAS}), U37.15 (~{CAS}), U38.15 (~{CAS})
- net ~{CAS1} is gone; now on net ~{CAS1}': U47.15 (~{CAS}), U48.15 (~{CAS}), U49.15 (~{CAS}), U50.15 (~{CAS}), U51.15 (~{CAS}), U52.15 (~{CAS}), U53.15 (~{CAS}), U54.15 (~{CAS})
- net ~{RAS0} is gone; now on net ~{RAS0}': U31.4 (~{RAS}), U32.4 (~{RAS}), U33.4 (~{RAS}), U34.4 (~{RAS}), U35.4 (~{RAS}), U36.4 (~{RAS}), U37.4 (~{RAS}), U38.4 (~{RAS})
- net ~{RAS1} is gone; now on net ~{RAS1}': U47.4 (~{RAS}), U48.4 (~{RAS}), U49.4 (~{RAS}), U50.4 (~{RAS}), U51.4 (~{RAS}), U52.4 (~{RAS}), U53.4 (~{RAS}), U54.4 (~{RAS})
- net +5V: now also U20.14 (VCC), U30.8 (Vcc), U31.8 (Vcc), U32.8 (Vcc), U33.8 (Vcc), U34.8 (Vcc), U35.8 (Vcc), U36.8 (Vcc), U37.8 (Vcc), U38.8 (Vcc), U39.16 (VCC), U40.16 (VCC), U46.8 (Vcc), U47.8 (Vcc), U48.8 (Vcc), U49.8 (Vcc), U50.8 (Vcc), U51.8 (Vcc), U52.8 (Vcc), U53.8 (Vcc), U54.8 (Vcc), U84.16 (VCC), U9.20 (VCC)
- net MA0: now also RN3.2, U30.5 (A0), U46.5 (A0)
- net MA1: now also RN3.5, U30.7 (A1), U46.7 (A1)
- net MA2: now also RN3.3, U30.6 (A2), U46.6 (A2)
- net MA3: now also RN3.6, U30.12 (A3), U46.12 (A3)
- net MA4: now also RN3.4, U30.11 (A4), U46.11 (A4)
- net MA5: now also RN3.7, U30.10 (A5), U46.10 (A5)
- net MA6: now also RN3.1, U30.13 (A6), U46.13 (A6)
- net MA7: now also RN3.8, U30.9 (A7), U46.9 (A7)
- net MD0: now also U20.8 (A), U31.14 (Q), U47.14 (Q)
- net MD1: now also U20.9 (B), U32.14 (Q), U48.14 (Q)
- net MD2: now also U20.10 (C), U33.14 (Q), U49.14 (Q)
- net MD3: now also U20.11 (D), U34.14 (Q), U50.14 (Q)
- net MD4: now also U20.12 (E), U35.14 (Q), U51.14 (Q)
- net MD5: now also U20.13 (F), U36.14 (Q), U52.14 (Q)
- net MD6: now also U20.1 (G), U37.14 (Q), U53.14 (Q)
- net MD7: now also U20.2 (H), U38.14 (Q), U54.14 (Q)
- net ~{CAS0}': now also U30.15 (~{CAS})
- net ~{CAS1}': now also U46.15 (~{CAS})
- net ~{RAS0}': now also U30.4 (~{RAS})
- net ~{RAS1}': now also U46.4 (~{RAS})
- net ~{WE}': now also U30.3 (~{WE}), U46.3 (~{WE}), RN4.1
- net MA8: now reaches U32.1 (A8)
- net MA8: now also RN4.2, U30.1 (A8), U31.1 (A8), U33.1 (A8), U34.1 (A8), U35.1 (A8), U36.1 (A8), U37.1 (A8), U38.1 (A8), U46.1 (A8), U47.1 (A8), U48.1 (A8), U49.1 (A8), U50.1 (A8), U51.1 (A8), U52.1 (A8), U53.1 (A8), U54.1 (A8)
- net GND: now reaches U32.16 (GND)
- net GND: now also U20.7 (GND), U30.16 (GND), U31.16 (GND), U33.16 (GND), U34.16 (GND), U35.16 (GND), U36.16 (GND), U37.16 (GND), U38.16 (GND), U39.15 (E), U39.8 (GND), U40.15 (E), U40.8 (GND), U46.16 (GND), U47.16 (GND), U48.16 (GND), U49.16 (GND), U50.16 (GND), U51.16 (GND), U52.16 (GND), U53.16 (GND), U54.16 (GND), U58.2, U84.15 (E), U84.8 (GND), U9.10 (GND)
- net ~{XMEMR}': now reaches U9.1 (A->B)
- net ~{XMEMR}': now also U86.3 (C)
- net ~{RAMADDRSEL}': now reaches U9.19 (CE)
- net ~{RAMADDRSEL}': now also U23.11
- net at U20.4 (I): now also U87.6
- net MDPIN: now reaches U20.5 (Even)
- net MDPIN: now also U30.2 (D), U46.2 (D)
- net at U20.6 (Odd): now also U23.10, U23.9
- net ~{XMEMW}': now reaches U58.1
- net at U58.3: now also RN4.16
- net ADDRSEL: now reaches U84.1 (S)
- net ADDRSEL: now also U39.1 (S), U40.1 (S)
- net XA16: now reaches U84.2 (I0a)
- net XA17: now reaches U84.3 (I1a)
- net MDPOUT: now reaches U30.14 (Q)
- net MDPOUT: now also U46.14 (Q), U87.4
- net BA2: now reaches RN3.14
- net BA2: now also U39.7 (Zb)
- net at U23.8: now also U86.2 (D)
- net BA6: now reaches RN3.16
- net BA6: now also U39.12 (Zc)
- net BA3: now reaches RN3.11
- net BA3: now also U40.7 (Zb)
- net BA4: now reaches RN3.13
- net BA4: now also U39.9 (Zd)
- net at U86.1 (~{R}): now also U89.10
- net ~{PCK}': now reaches U86.4 (~{S})
- net ~{PCK}': now also U86.6 (~{Q})
- net PCK: now reaches U86.5 (Q)
- net ~{ENBRAMPCK}': now reaches U89.11
- net XA11: now reaches U39.10 (I1d)
- net XA4: now reaches U39.11 (I0d)
- net XA13: now reaches U39.13 (I1c)
- net XA6: now reaches U39.14 (I0c)
- net XA0: now reaches U39.2 (I0a)
- net XA14: now reaches U39.3 (I1a)
- net XA14: now also E4.1 (Pin_1), E4.3 (Pin_3), E4.4 (Pin_4)
- net BA0: now reaches U39.4 (Za)
- net BA0: now also RN3.15
- net XA2: now reaches U39.5 (I0b)
- net XA9: now reaches U39.6 (I1b)
- net BA5: now reaches RN3.10
- net BA5: now also U40.9 (Zd)
- net XA12: now reaches U40.10 (I1d)
- net XA5: now reaches U40.11 (I0d)
- net BA7: now reaches U40.12 (Zc)
- net BA7: now also RN3.9
- net XA15: now reaches U40.13 (I1c)
- net XA7: now reaches U40.14 (I0c)
- net XA7: now also E4.2 (Pin_2)
- net XA1: now reaches U40.2 (I0a)
- net XA8: now reaches U40.3 (I1a)
- net BA1: now reaches U40.4 (Za)
- net BA1: now also RN3.12
- net XA3: now reaches U40.5 (I0b)
- net XA10: now reaches U40.6 (I1b)
- net +XMEMR: now reaches U87.5
- no-connect marks 3 -> 9
Other:
- moved on the sheet: E4, RN3A, RN3B, RN3C, RN3D, RN3E, RN3F, RN3H, RN4B, RN5A, U20B, U23C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

Commit message: Sheet 10 done
Parts:
- RN5: symbol Mad5150_early:Resistor_Network -> Mad5150_early:Resistor_Network_1
Changed lines of the file:
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@@
     (pin "10")
     (pin "8")
-    (pin "3")
     (pin "9")
     (pin "14")
@@
     (pin "2")
     (pin "7")
-    (pin "3")
     (instances
       (project "Mad5160"
@@
     )
   )
-  (symbol (lib_id "Mad5150_early:Resistor_Network") (at 110.49 251.46 180) (unit 1)
+  (symbol (lib_id "Mad5150_early:Resistor_Network_1") (at 110.49 251.46 180) (unit 1)
     (in_bom yes) (on_board yes) (dnp no) (fields_autoplaced)
     (property "Reference" "RN5" (at 113.03 250.19 0)
@@
       (effects (font (size 1.27 1.27)) hide)
     )
-    (property "Datasheet" "" (at 110.49 251.46 0)
-      (effects (font (size 1.27 1.27)) hide)
-    )
+    (property "Datasheet" "" (at 109.855 252.095 0)
+      (effects (font (size 1.27 1.27)) hide)
+    )

Commit message: Tracing finished
Parts:
- E4: footprint madXT_early:E4 -> mad5150:E4
- RN3, RN4, RN5, U39, U40: footprint Package_DIP:DIP-16_W7.62mm -> mad5150:DIP-16_W7.62mm
- U20, U23, U58, U86, U87, U89: footprint Package_DIP:DIP-14_W7.62mm -> mad5150:DIP-14_W7.62mm
- U30, U31, U32, U33, U34, U35, U36, U37, U38, U46, U47, U48, U49, U50, U51, U52, U53, U54: footprint Package_DIP:DIP-16_W7.62mm -> mad5150:Ram_socket_IC
- U84: footprint Package_DIP:DIP-16_W7.62mm_Socket -> mad5150:DIP-16_W7.62mm_Socket
- U9: footprint Package_DIP:DIP-20_W7.62mm -> mad5150:DIP-20_W7.62mm

Commit message: Fixing stuff
Parts:
- removed U58: LS32_U58, mad5150:DIP-14_W7.62mm, symbol Mad5150_early:LS32_U58
- added U22: 74LS04, mad5150:DIP-14_W7.62mm, symbol 74xx:74LS04
Connections:
- net ~{XMEMW}': now also U22.1
- net at RN4.16: now also U22.4
- new net: U22.2, U22.3
Changed lines of the file:
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@@
     (stroke (width 0) (type default))
   )
-  (wire (pts (xy 22.86 78.105) (xy 66.675 78.105))
-    (stroke (width 0) (type default))
-  )
   (bus (pts (xy 173.99 92.075) (xy 173.99 94.615))
     (stroke (width 0) (type default))
@@
     (stroke (width 0) (type default))
   )
-  (wire (pts (xy 46.99 198.755) (xy 46.99 198.12))
-    (stroke (width 0) (type default))
-  )
   (wire (pts (xy 22.225 93.345) (xy 26.035 93.345))
     (stroke (width 0) (type default))
@@
     (stroke (width 0) (type default))
   )
+  (wire (pts (xy 22.86 80.645) (xy 48.895 80.645))
+    (stroke (width 0) (type default))
+  )
   (wire (pts (xy 56.515 373.38) (xy 76.2 373.38))
     (stroke (width 0) (type default))
@@
     (stroke (width 0) (type default))
   )
+  (wire (pts (xy 64.135 80.645) (xy 66.675 80.645))
+    (stroke (width 0) (type default))
+  )
   (wire (pts (xy 230.505 304.8) (xy 239.395 304.8))
     (stroke (width 0) (type default))
@@
     )
   )
-  (global_label "~{XMEMW}'" (shape input) (at 22.86 78.105 180) (fields_autoplaced)
+  (global_label "~{XMEMW}'" (shape input) (at 22.86 80.645 180) (fields_autoplaced)
     (effects (font (size 1.27 1.27)) (justify right))
-    (property "Intersheetrefs" "${INTERSHEET_REFS}" (at 12.5573 78.105 0)
+    (property "Intersheetrefs" "${INTERSHEET_REFS}" (at 12.5573 80.645 0)
       (effects (font (size 1.27 1.27)) (justify right) hide)
     )
@@
     )
   )
-  (symbol (lib_id "Mad5150_early:LS32_U58") (at 74.295 80.645 0) (unit 1)
-    (in_bom yes) (on_board yes) (dnp no) (fields_autoplaced)
-    (property "Reference" "U58" (at 74.295 73.66 0)
-      (effects (font (size 1.27 1.27)))
-    )
-    (property "Value" "LS32_U58" (at 74.295 76.2 0)
-      (effects (font (size 1.27 1.27)))
-    )
-    (property "Footprint" "mad5150:DIP-14_W7.62mm" (at 74.295 80.645 0)
-      (effects (font (size 1.27 1.27)) hide)
-    )
-    (property "Datasheet" "http://www.ti.com/lit/gpn/sn74LS32" (at 74.295 80.645 0)
-      (effects (font (size 1.27 1.27)) hide)
-    )
-    (pin "11")
-    (pin "5")
-    (pin "14")
-    (pin "3")
-    (pin "10")
-    (pin "13")
-    (pin "6")
-    (pin "9")
-    (pin "12")
-    (pin "2")
-    (pin "7")
-    (pin "8")
-    (pin "4")
-    (pin "1")
-    (instances
-      (project "Mad5160"
-        (path "/ac3c86ab-084e-42f6-87ca-c4b0142d8ff2/aca52fbe-2189-4f56-80e9-b8157b8b750b"
-          (reference "U58") (unit 1)
-        )
-      )
-    )
-  )
   (symbol (lib_id "Mad5150_early:64Kx1_RAM_U30_38") (at 307.34 244.475 0) (unit 1)
     (in_bom yes) (on_board yes) (dnp no) (fields_autoplaced)
@@
     )
   )
+  (symbol (lib_id "74xx:74LS04") (at 56.515 80.645 0) (unit 1)
+    (in_bom yes) (on_board yes) (dnp no) (fields_autoplaced)
+    (property "Reference" "U22" (at 56.515 73.66 0)
+      (effects (font (size 1.27 1.27)))
+    )
+    (property "Value" "74LS04" (at 56.515 76.2 0)
+      (effects (font (size 1.27 1.27)))
+    )
+    (property "Footprint" "mad5150:DIP-14_W7.62mm" (at 56.515 80.645 0)
+      (effects (font (size 1.27 1.27)) hide)
+    )
+    (property "Datasheet" "http://www.ti.com/lit/gpn/sn74LS04" (at 56.515 80.645 0)
+      (effects (font (size 1.27 1.27)) hide)
+    )
+    (pin "1")
+    (pin "2")
+    (pin "3")
+    (pin "4")
+    (pin "5")
+    (pin "6")
+    (pin "8")
+    (pin "9")
+    (pin "10")
+    (pin "11")
+    (pin "12")
+    (pin "13")
+    (pin "14")
+    (pin "7")
+    (instances
+      (project "Mad5160"
+        (path "/ac3c86ab-084e-42f6-87ca-c4b0142d8ff2/aca52fbe-2189-4f56-80e9-b8157b8b750b"
+          (reference "U22") (unit 1)
+        )
+      )
+    )
+  )
   (symbol (lib_id "power:GND") (at 321.945 114.935 90) (unit 1)
     (in_bom yes) (on_board yes) (dnp no)
@@
     )
   )
-  (symbol (lib_id "power:GND") (at 66.675 83.185 0) (unit 1)
-    (in_bom yes) (on_board yes) (dnp no) (fields_autoplaced)
-    (property "Reference" "#PWR055" (at 66.675 89.535 0)
-      (effects (font (size 1.27 1.27)) hide)
-    )
-    (property "Value" "GND" (at 66.675 87.63 0)
-      (effects (font (size 1.27 1.27)))
-    )
-    (property "Footprint" "" (at 66.675 83.185 0)
-      (effects (font (size 1.27 1.27)) hide)
-    )
-    (property "Datasheet" "" (at 66.675 83.185 0)
-      (effects (font (size 1.27 1.27)) hide)
-    )
-    (pin "1")
-    (instances
-      (project "Mad5160"
-        (path "/ac3c86ab-084e-42f6-87ca-c4b0142d8ff2/aca52fbe-2189-4f56-80e9-b8157b8b750b"
-          (reference "#PWR055") (unit 1)
-        )
-      )
-    )
-  )
   (symbol (lib_id "Mad5150_early:RN3") (at 103.505 110.49 270) (unit 1)
     (in_bom yes) (on_board yes) (dnp no)
@@
         )
       )
+    )
+  )
+  (symbol (lib_id "74xx:74LS04") (at 74.295 80.645 0) (unit 2)
+    (in_bom yes) (on_board yes) (dnp no) (fields_autoplaced)
+    (property "Reference" "U22" (at 74.295 74.295 0)
+      (effects (font (size 1.27 1.27)))
+    )
+    (property "Value" "74LS04" (at 74.295 76.835 0)
+      (effects (font (size 1.27 1.27)))
+    )
+    (property "Footprint" "mad5150:DIP-14_W7.62mm" (at 74.295 80.645 0)
+      (effects (font (size 1.27 1.27)) hide)
+    )
+    (property "Datasheet" "http://www.ti.com/lit/gpn/sn74LS04" (at 74.295 80.645 0)
+      (effects (font (size 1.27 1.27)) hide)
+    )
+    (pin "1")
+    (pin "2")
+    (pin "3")
+    (pin "4")
+    (pin "5")
+    (pin "6")
+    (pin "8")
+    (pin "9")
+    (pin "10")
+    (pin "11")
+    (pin "12")
+    (pin "13")
+    (pin "14")
+    (pin "7")
+    (instances
+      (project "Mad5160"
+        (path "/ac3c86ab-084e-42f6-87ca-c4b0142d8ff2/aca52fbe-2189-4f56-80e9-b8157b8b750b"
+          (reference "U22") (unit 2)
+        )
+      )

Commit message: Gerbers
Parts:
- U86: value S74_U70 -> 74LS74AN
Changed lines of the file:
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@@
       (effects (font (size 1.27 1.27)) (justify left))
     )
-    (property "Value" "S74_U70" (at 127.2891 196.85 0)
+    (property "Value" "74LS74AN" (at 127.2891 196.85 0)
       (effects (font (size 1.27 1.27)) (justify left))
     )
