File: sheet8.kicad_sch (KiCad schematic)
At the start: 8 parts, among them P3 SPEAKER, U21 LS175, U26 8253-5, U73 S74_U70, U85 SN75477, U87 S08_U87

Commit message: Sheet 9 finished, almost there
Parts:
- removed unit 2 of U21
- added unit 3 of U21
Connections:
- net +5V: now also U21.16 (VCC)
- net GND: now also U21.8 (GND)
- no-connect marks 10 -> 6
Changed lines of the file:
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@@
   (no_connect (at 57.15 137.795))
   (no_connect (at 149.225 33.655))
-  (no_connect (at 57.15 120.015))
-  (no_connect (at 57.15 127.635))
   (no_connect (at 31.75 136.525))
   (no_connect (at 57.15 122.555))
-  (no_connect (at 31.75 121.285))
   (no_connect (at 57.15 135.255))
-  (no_connect (at 31.75 126.365))
   (wire (pts (xy 141.605 23.495) (xy 141.605 16.51))
     (stroke (width 0) (type default))
@@
     )
   )
+  (symbol (lib_id "Mad5150_early:SN75477P_U85") (at 161.925 62.23 0) (unit 1)
+    (in_bom yes) (on_board yes) (dnp no) (fields_autoplaced)
+    (property "Reference" "U85" (at 161.925 50.8 0)
+      (effects (font (size 1.27 1.27)))
+    )
+    (property "Value" "SN75477" (at 161.925 53.34 0)
+      (effects (font (size 1.27 1.27)))
+    )
+    (property "Footprint" "Package_DIP:DIP-8_W7.62mm" (at 161.925 76.835 0)
+      (effects (font (size 1.27 1.27)) hide)
+    )
+    (property "Datasheet" "" (at 114.3 65.405 0)
+      (effects (font (size 1.27 1.27)) hide)
+    )
+    (pin "4")
+    (pin "6")
+    (pin "2")
+    (pin "1")
+    (pin "7")
+    (pin "5")
+    (pin "3")
+    (pin "8")
+    (instances
+      (project "Mad5160"
+        (path "/ac3c86ab-084e-42f6-87ca-c4b0142d8ff2/fe4ae14e-03b0-4858-831e-5da8f6de2de8"
+          (reference "U85") (unit 1)
+        )
+      )
+    )
+  )
   (symbol (lib_id "Mad5150_early:SPEAKER") (at 204.47 79.375 0) (unit 1)
     (in_bom yes) (on_board yes) (dnp no) (fields_autoplaced)
@@
     )
   )
+  (symbol (lib_id "Mad5150_early:LS175_U21") (at 44.45 130.175 0) (unit 1)
+    (in_bom yes) (on_board yes) (dnp no) (fields_autoplaced)
+    (property "Reference" "U21" (at 44.45 113.03 0)
+      (effects (font (size 1.27 1.27)))
+    )
+    (property "Value" "LS175" (at 44.45 115.57 0)
+      (effects (font (size 1.27 1.27) bold))
+    )
+    (property "Footprint" "Package_DIP:DIP-16_W7.62mm" (at 44.45 133.35 0)
+      (effects (font (size 1.27 1.27)) hide)
+    )
+    (property "Datasheet" "" (at 44.45 133.35 0)
+      (effects (font (size 1.27 1.27)) hide)
+    )
+    (pin "15")
+    (pin "3")
+    (pin "13")
+    (pin "12")
+    (pin "14")
+    (pin "4")
+    (pin "9")
+    (pin "9")
+    (pin "10")
+    (pin "6")
+    (pin "2")
+    (pin "16")
+    (pin "8")
+    (pin "1")
+    (pin "1")
+    (pin "7")
+    (pin "11")
+    (pin "5")
+    (instances
+      (project "Mad5160"
+        (path "/ac3c86ab-084e-42f6-87ca-c4b0142d8ff2/fe4ae14e-03b0-4858-831e-5da8f6de2de8"
+          (reference "U21") (unit 1)
+        )
+      )
+    )
+  )
   (symbol (lib_id "power:+5V") (at 146.05 66.04 90) (unit 1)
     (in_bom yes) (on_board yes) (dnp no) (fields_autoplaced)
@@
     )
   )
-  (symbol (lib_id "Mad5150_early:LS175_U21") (at 29.845 178.435 0) (unit 2)
-    (in_bom yes) (on_board yes) (dnp no) (fields_autoplaced)
-    (property "Reference" "U21" (at 34.29 176.8475 0)
-      (effects (font (size 1.27 1.27)) (justify left))
-    )
-    (property "Value" "LS175" (at 34.29 179.3875 0)
+  (symbol (lib_id "power:+5V") (at 78.105 55.88 90) (unit 1)
+    (in_bom yes) (on_board yes) (dnp no) (fields_autoplaced)
+    (property "Reference" "#PWR0135" (at 81.915 55.88 0)
+      (effects (font (size 1.27 1.27)) hide)
+    )
+    (property "Value" "+5V" (at 74.295 55.88 90)
+      (effects (font (size 1.27 1.27)) (justify left))
+    )
+    (property "Footprint" "" (at 78.105 55.88 0)
+      (effects (font (size 1.27 1.27)) hide)
+    )
+    (property "Datasheet" "" (at 78.105 55.88 0)
+      (effects (font (size 1.27 1.27)) hide)
+    )
+    (pin "1")
+    (instances
+      (project "Mad5160"
+        (path "/ac3c86ab-084e-42f6-87ca-c4b0142d8ff2/fe4ae14e-03b0-4858-831e-5da8f6de2de8"
+          (reference "#PWR0135") (unit 1)
+        )
+      )
+    )
+  )
+  (symbol (lib_id "power:+5V") (at 78.74 50.8 90) (unit 1)
+    (in_bom yes) (on_board yes) (dnp no) (fields_autoplaced)
+    (property "Reference" "#PWR0134" (at 82.55 50.8 0)
+      (effects (font (size 1.27 1.27)) hide)
+    )
+    (property "Value" "+5V" (at 74.93 50.8 90)
+      (effects (font (size 1.27 1.27)) (justify left))
+    )
+    (property "Footprint" "" (at 78.74 50.8 0)
+      (effects (font (size 1.27 1.27)) hide)
+    )
+    (property "Datasheet" "" (at 78.74 50.8 0)
+      (effects (font (size 1.27 1.27)) hide)
+    )
+    (pin "1")
+    (instances
+      (project "Mad5160"
+        (path "/ac3c86ab-084e-42f6-87ca-c4b0142d8ff2/fe4ae14e-03b0-4858-831e-5da8f6de2de8"
+          (reference "#PWR0134") (unit 1)
+        )
+      )
+    )
+  )
+  (symbol (lib_id "Mad5150_early:LS175_U21") (at 29.845 178.435 0) (unit 3)
+    (in_bom yes) (on_board yes) (dnp no) (fields_autoplaced)
+    (property "Reference" "U21" (at 35.56 176.8475 0)
+      (effects (font (size 1.27 1.27)) (justify left))
+    )
+    (property "Value" "LS175" (at 35.56 179.3875 0)
       (effects (font (size 1.27 1.27) bold) (justify left))
     )
@@
       (effects (font (size 1.27 1.27)) hide)
     )
+    (pin "15")
+    (pin "3")
+    (pin "13")
+    (pin "12")
+    (pin "14")
     (pin "4")
+    (pin "9")
+    (pin "9")
+    (pin "10")
     (pin "6")
-    (pin "1")
+    (pin "2")
+    (pin "16")
+    (pin "8")
+    (pin "1")
+    (pin "1")
+    (pin "7")
     (pin "11")
-    (pin "10")
-    (pin "15")
-    (pin "2")
-    (pin "14")
-    (pin "16")
-    (pin "3")
-    (pin "7")
-    (pin "13")
     (pin "5")
-    (pin "9")
-    (pin "8")
-    (pin "12")
-    (instances
-      (project "Mad5160"
-        (path "/ac3c86ab-084e-42f6-87ca-c4b0142d8ff2/fe4ae14e-03b0-4858-831e-5da8f6de2de8"
-          (reference "U21") (unit 2)
-        )
-      )
-    )
-  )
-  (symbol (lib_id "Mad5150_early:SN75477P_U85") (at 161.925 62.23 0) (unit 1)
-    (in_bom yes) (on_board yes) (dnp no)
-    (property "Reference" "U85" (at 161.925 57.785 0)
-      (effects (font (size 1.27 1.27)))
-    )
-    (property "Value" "SN75477" (at 161.925 53.975 0)
-      (effects (font (size 1.27 1.27)))
-    )
-    (property "Footprint" "Package_DIP:DIP-8_W7.62mm" (at 161.925 76.835 0)
-      (effects (font (size 1.27 1.27)) hide)
-    )
-    (property "Datasheet" "" (at 114.3 65.405 0)
-      (effects (font (size 1.27 1.27)) hide)
-    )
-    (pin "1")
-    (pin "4")
-    (pin "7")
-    (pin "6")
-    (pin "8")
-    (pin "5")
-    (instances
-      (project "Mad5160"
-        (path "/ac3c86ab-084e-42f6-87ca-c4b0142d8ff2/fe4ae14e-03b0-4858-831e-5da8f6de2de8"
-          (reference "U85") (unit 1)
-        )
-      )
-    )
-  )
-  (symbol (lib_id "power:+5V") (at 78.105 55.88 90) (unit 1)
-    (in_bom yes) (on_board yes) (dnp no) (fields_autoplaced)
-    (property "Reference" "#PWR0135" (at 81.915 55.88 0)
-      (effects (font (size 1.27 1.27)) hide)
-    )
-    (property "Value" "+5V" (at 74.295 55.88 90)
-      (effects (font (size 1.27 1.27)) (justify left))
-    )
-    (property "Footprint" "" (at 78.105 55.88 0)
-      (effects (font (size 1.27 1.27)) hide)
-    )
-    (property "Datasheet" "" (at 78.105 55.88 0)
-      (effects (font (size 1.27 1.27)) hide)
-    )
-    (pin "1")
-    (instances
-      (project "Mad5160"
-        (path "/ac3c86ab-084e-42f6-87ca-c4b0142d8ff2/fe4ae14e-03b0-4858-831e-5da8f6de2de8"
-          (reference "#PWR0135") (unit 1)
-        )
-      )
-    )
-  )
-  (symbol (lib_id "power:+5V") (at 78.74 50.8 90) (unit 1)
-    (in_bom yes) (on_board yes) (dnp no) (fields_autoplaced)
-    (property "Reference" "#PWR0134" (at 82.55 50.8 0)
-      (effects (font (size 1.27 1.27)) hide)
-    )
-    (property "Value" "+5V" (at 74.93 50.8 90)
-      (effects (font (size 1.27 1.27)) (justify left))
-    )
-    (property "Footprint" "" (at 78.74 50.8 0)
-      (effects (font (size 1.27 1.27)) hide)
-    )
-    (property "Datasheet" "" (at 78.74 50.8 0)
-      (effects (font (size 1.27 1.27)) hide)
-    )
-    (pin "1")
-    (instances
-      (project "Mad5160"
-        (path "/ac3c86ab-084e-42f6-87ca-c4b0142d8ff2/fe4ae14e-03b0-4858-831e-5da8f6de2de8"
-          (reference "#PWR0134") (unit 1)
+    (instances
+      (project "Mad5160"
+        (path "/ac3c86ab-084e-42f6-87ca-c4b0142d8ff2/fe4ae14e-03b0-4858-831e-5da8f6de2de8"
+          (reference "U21") (unit 3)
         )
       )
@@
         )
       )
-    )
-  )
-  (symbol (lib_id "Mad5150_early:LS175_U21") (at 44.45 130.175 0) (unit 1)
-    (in_bom yes) (on_board yes) (dnp no) (fields_autoplaced)
-    (property "Reference" "U21" (at 44.45 113.03 0)
-      (effects (font (size 1.27 1.27)))
-    )
-    (property "Value" "LS175" (at 44.45 115.57 0)
-      (effects (font (size 1.27 1.27) bold))
-    )
-    (property "Footprint" "Package_DIP:DIP-16_W7.62mm" (at 44.45 133.35 0)
-      (effects (font (size 1.27 1.27)) hide)
-    )
-    (property "Datasheet" "" (at 44.45 133.35 0)
-      (effects (font (size 1.27 1.27)) hide)
-    )
-    (pin "4")
-    (pin "6")
-    (pin "1")
-    (pin "11")
-    (pin "10")
-    (pin "15")
-    (pin "2")
-    (pin "14")
-    (pin "16")
-    (pin "3")
-    (pin "7")
-    (pin "13")
-    (pin "5")
-    (pin "9")
-    (pin "8")
-    (pin "12")
-    (instances
-      (project "Mad5160"
-        (path "/ac3c86ab-084e-42f6-87ca-c4b0142d8ff2/fe4ae14e-03b0-4858-831e-5da8f6de2de8"
-          (reference "U21") (unit 1)
-        )
-      )

Commit message: Sheet 10 done
Connections:
- net +5V: now also U26.14 (GATE1)
Changed lines of the file:
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@@
     )
   )
-  (symbol (lib_id "power:+5V") (at 78.105 55.88 90) (unit 1)
+  (symbol (lib_id "power:+5V") (at 78.74 55.88 90) (unit 1)
     (in_bom yes) (on_board yes) (dnp no) (fields_autoplaced)
-    (property "Reference" "#PWR0135" (at 81.915 55.88 0)
+    (property "Reference" "#PWR0135" (at 82.55 55.88 0)
       (effects (font (size 1.27 1.27)) hide)
     )
-    (property "Value" "+5V" (at 74.295 55.88 90)
+    (property "Value" "+5V" (at 74.93 55.88 90)
       (effects (font (size 1.27 1.27)) (justify left))
     )
-    (property "Footprint" "" (at 78.105 55.88 0)
+    (property "Footprint" "" (at 78.74 55.88 0)
       (effects (font (size 1.27 1.27)) hide)
     )
-    (property "Datasheet" "" (at 78.105 55.88 0)
+    (property "Datasheet" "" (at 78.74 55.88 0)
       (effects (font (size 1.27 1.27)) hide)
     )

Commit message: Begin tracing
Parts:
- C53: footprint Capacitor_THT:C_Axial_L12.0mm_D6.5mm_P15.00mm_Horizontal -> madXT_early:cap_unipolar
Changed lines of the file:
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@@
       (effects (font (size 1.27 1.27)) (justify left))
     )
-    (property "Footprint" "Capacitor_THT:C_Axial_L12.0mm_D6.5mm_P15.00mm_Horizontal" (at 178.1302 66.04 0)
+    (property "Footprint" "madXT_early:cap_unipolar" (at 178.1302 66.04 0)
       (effects (font (size 1.27 1.27)) hide)
     )

Commit message: Tracing for version 1.0 finished
Parts:
- C53: footprint madXT_early:cap_unipolar -> madXT_early:CP8
Changed lines of the file:
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@@
       (effects (font (size 1.27 1.27)) (justify left))
     )
-    (property "Footprint" "madXT_early:cap_unipolar" (at 178.1302 66.04 0)
+    (property "Footprint" "madXT_early:CP8" (at 178.1302 66.04 0)
       (effects (font (size 1.27 1.27)) hide)
     )

Commit message: Tracing finished
Parts:
- C53: footprint madXT_early:CP8 -> mad5150:CP8
- P3: footprint Connector_PinHeader_2.54mm:PinHeader_1x04_P2.54mm_Vertical -> mad5150:PinHeader_1x04_P2.54mm_Vertical
- R6: footprint madXT_early:resistor -> mad5150:resistor
- U21: footprint Package_DIP:DIP-16_W7.62mm -> mad5150:DIP-16_W7.62mm
- U26: footprint Package_DIP:DIP-24_W15.24mm -> mad5150:DIP-24_W15.24mm
- U73, U87: footprint Package_DIP:DIP-14_W7.62mm -> mad5150:DIP-14_W7.62mm
- U85: footprint Package_DIP:DIP-8_W7.62mm -> mad5150:DIP-8_W7.62mm
Changed lines of the file:
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@@
       (effects (font (size 1.27 1.27)))
     )
-    (property "Footprint" "Package_DIP:DIP-8_W7.62mm" (at 161.925 76.835 0)
+    (property "Footprint" "mad5150:DIP-8_W7.62mm" (at 161.925 76.835 0)
       (effects (font (size 1.27 1.27)) hide)
     )
@@
       (effects (font (size 1.27 1.27)) (justify left))
     )
-    (property "Footprint" "Connector_PinHeader_2.54mm:PinHeader_1x04_P2.54mm_Vertical" (at 204.47 79.375 0)
+    (property "Footprint" "mad5150:PinHeader_1x04_P2.54mm_Vertical" (at 204.47 79.375 0)
       (effects (font (size 1.27 1.27)) hide)
     )
@@
       (effects (font (size 1.27 1.27)) (justify left))
     )
-    (property "Footprint" "madXT_early:CP8" (at 178.1302 66.04 0)
+    (property "Footprint" "mad5150:CP8" (at 178.1302 66.04 0)
       (effects (font (size 1.27 1.27)) hide)
     )
@@
       (effects (font (size 1.27 1.27) bold))
     )
-    (property "Footprint" "Package_DIP:DIP-16_W7.62mm" (at 44.45 133.35 0)
+    (property "Footprint" "mad5150:DIP-16_W7.62mm" (at 44.45 133.35 0)
       (effects (font (size 1.27 1.27)) hide)
     )
@@
       (effects (font (size 1.27 1.27)) (justify left))
     )
-    (property "Footprint" "madXT_early:resistor" (at 188.087 66.04 90)
+    (property "Footprint" "mad5150:resistor" (at 188.087 66.04 90)
       (effects (font (size 1.27 1.27)) hide)
     )
@@
       (effects (font (size 1.27 1.27) bold) (justify left))
     )
-    (property "Footprint" "Package_DIP:DIP-16_W7.62mm" (at 29.845 181.61 0)
+    (property "Footprint" "mad5150:DIP-16_W7.62mm" (at 29.845 181.61 0)
       (effects (font (size 1.27 1.27)) hide)
     )
@@
       (effects (font (size 1.27 1.27)) (justify left))
     )
-    (property "Footprint" "Package_DIP:DIP-14_W7.62mm" (at 141.605 31.115 0)
+    (property "Footprint" "mad5150:DIP-14_W7.62mm" (at 141.605 31.115 0)
       (effects (font (size 1.27 1.27)) hide)
     )
@@
       (effects (font (size 1.27 1.27)))
     )
-    (property "Footprint" "Package_DIP:DIP-14_W7.62mm" (at 135.89 58.42 0)
+    (property "Footprint" "mad5150:DIP-14_W7.62mm" (at 135.89 58.42 0)
       (effects (font (size 1.27 1.27)) hide)
     )
@@
       (effects (font (size 1.27 1.27)))
     )
-    (property "Footprint" "Package_DIP:DIP-24_W15.24mm" (at 92.075 106.045 0)
-      (effects (font (size 1.27 1.27)) hide)
-    )
+    (property "Footprint" "mad5150:DIP-24_W15.24mm" (at 92.075 106.045 0)
+      (effects (font (size 1.27 1.27)) hide)
+    )

Commit message: Fixing stuff
Parts:
- added U58: LS32_U58, mad5150:DIP-14_W7.62mm, symbol Mad5150_early:LS32_U58
Connections:
- net ~{T/CCS}': now also U58.1, U58.4
- net ~{XIOR}': now also U58.2; no longer U26.22 (~{RD})
- net ~{XIOW}': now also U58.5; no longer U26.23 (~{WR})
- new net: U26.23 (~{WR}), U58.6
- new net: U26.22 (~{RD}), U58.3
Other:
- moved on the sheet: C53, P3, R6, U21A, U26, U85A, U87D

Commit message: Gerbers
Parts:
- U73: value S74_U70 -> 74LS74AN
Changed lines of the file:
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@@
       (effects (font (size 1.27 1.27)) (justify left))
     )
-    (property "Value" "S74_U70" (at 143.7991 25.4 0)
+    (property "Value" "74LS74AN" (at 143.7991 25.4 0)
       (effects (font (size 1.27 1.27)) (justify left))
     )
