File: sheet9.kicad_sch (KiCad schematic)
At the start: 18 parts, among them J9 KEYBOARD, SW1 DIP_SWITCH, U21 LS175, U27 LS322_U27, U29 8255A-5, U41 LS244, U68 7407_U68, U70 S74_U70, U71 LS04_U71, U85 SN75477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

Commit message: Sheet 10 done
Parts:
- RN5: symbol Mad5150_early:Resistor_Network -> Mad5150_early:Resistor_Network_1
Changed lines of the file:
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@@
     (stroke (width 0) (type default))
   )
-  (wire (pts (xy 110.49 92.71) (xy 223.9225 92.71))
+  (wire (pts (xy 110.49 92.71) (xy 220.345 92.71))
     (stroke (width 0) (type default))
   )
@@
     (stroke (width 0) (type default))
   )
-  (wire (pts (xy 225.1925 79.375) (xy 299.085 79.375))
+  (wire (pts (xy 224.155 79.375) (xy 299.085 79.375))
     (stroke (width 0) (type default))
   )
@@
     (stroke (width 0) (type default))
   )
-  (wire (pts (xy 222.25 114.935) (xy 224.155 114.935))
+  (wire (pts (xy 216.535 114.935) (xy 224.155 114.935))
     (stroke (width 0) (type default))
   )
@@
     (stroke (width 0) (type default))
   )
-  (wire (pts (xy 222.25 48.26) (xy 222.25 114.935))
+  (wire (pts (xy 216.535 48.26) (xy 216.535 114.935))
     (stroke (width 0) (type default))
   )
@@
     (stroke (width 0) (type default))
   )
-  (wire (pts (xy 213.36 110.49) (xy 228.6 110.49))
+  (wire (pts (xy 213.36 110.49) (xy 233.68 110.49))
     (stroke (width 0) (type default))
   )
@@
     (stroke (width 0) (type default))
   )
-  (wire (pts (xy 228.6 110.49) (xy 228.6 92.075))
+  (wire (pts (xy 233.68 110.49) (xy 233.68 92.075))
     (stroke (width 0) (type default))
   )
@@
     (stroke (width 0) (type default))
   )
-  (wire (pts (xy 223.2875 90.17) (xy 223.2875 71.755))
+  (wire (pts (xy 218.44 90.17) (xy 218.44 71.755))
     (stroke (width 0) (type default))
   )
@@
     (stroke (width 0) (type default))
   )
-  (wire (pts (xy 225.8275 100.33) (xy 225.8275 81.915))
+  (wire (pts (xy 226.06 100.33) (xy 226.06 81.915))
     (stroke (width 0) (type default))
   )
@@
     (stroke (width 0) (type default))
   )
-  (wire (pts (xy 110.49 90.17) (xy 223.2875 90.17))
+  (wire (pts (xy 110.49 90.17) (xy 218.44 90.17))
     (stroke (width 0) (type default))
   )
@@
     (stroke (width 0) (type default))
   )
-  (wire (pts (xy 110.49 97.79) (xy 225.1925 97.79))
+  (wire (pts (xy 110.49 97.79) (xy 224.155 97.79))
     (stroke (width 0) (type default))
   )
@@
     (stroke (width 0) (type default))
   )
-  (wire (pts (xy 226.4625 102.87) (xy 226.4625 84.455))
+  (wire (pts (xy 227.965 102.87) (xy 227.965 84.455))
     (stroke (width 0) (type default))
   )
@@
     (stroke (width 0) (type default))
   )
-  (wire (pts (xy 227.7325 107.95) (xy 227.7325 89.535))
+  (wire (pts (xy 231.775 107.95) (xy 231.775 89.535))
     (stroke (width 0) (type default))
   )
@@
     (stroke (width 0) (type default))
   )
-  (wire (pts (xy 160.02 48.26) (xy 222.25 48.26))
+  (wire (pts (xy 160.02 48.26) (xy 216.535 48.26))
     (stroke (width 0) (type default))
   )
@@
     (stroke (width 0) (type default))
   )
-  (wire (pts (xy 110.49 100.33) (xy 225.8275 100.33))
+  (wire (pts (xy 110.49 100.33) (xy 226.06 100.33))
     (stroke (width 0) (type default))
   )
@@
     (stroke (width 0) (type default))
   )
-  (wire (pts (xy 227.0975 105.41) (xy 227.0975 86.995))
+  (wire (pts (xy 229.87 105.41) (xy 229.87 86.995))
     (stroke (width 0) (type default))
   )
@@
     (stroke (width 0) (type default))
   )
-  (wire (pts (xy 224.5575 95.25) (xy 224.5575 76.835))
+  (wire (pts (xy 222.25 95.25) (xy 222.25 76.835))
     (stroke (width 0) (type default))
   )
@@
     (stroke (width 0) (type default))
   )
-  (wire (pts (xy 223.9225 92.71) (xy 223.9225 74.295))
+  (wire (pts (xy 220.345 92.71) (xy 220.345 74.295))
     (stroke (width 0) (type default))
   )
@@
     (stroke (width 0) (type default))
   )
-  (wire (pts (xy 226.4625 84.455) (xy 299.085 84.455))
+  (wire (pts (xy 227.965 84.455) (xy 299.085 84.455))
     (stroke (width 0) (type default))
   )
@@
     (stroke (width 0) (type default))
   )
-  (wire (pts (xy 227.0975 86.995) (xy 299.085 86.995))
+  (wire (pts (xy 229.87 86.995) (xy 299.085 86.995))
     (stroke (width 0) (type default))
   )
@@
     (stroke (width 0) (type default))
   )
-  (wire (pts (xy 223.2875 71.755) (xy 299.085 71.755))
+  (wire (pts (xy 218.44 71.755) (xy 299.085 71.755))
     (stroke (width 0) (type default))
   )
@@
     (stroke (width 0) (type default))
   )
-  (wire (pts (xy 224.5575 76.835) (xy 299.085 76.835))
+  (wire (pts (xy 222.25 76.835) (xy 299.085 76.835))
     (stroke (width 0) (type default))
   )
@@
     (stroke (width 0) (type default))
   )
-  (wire (pts (xy 110.49 107.95) (xy 227.7325 107.95))
+  (wire (pts (xy 110.49 107.95) (xy 231.775 107.95))
     (stroke (width 0) (type default))
   )
@@
     (stroke (width 0) (type default))
   )
-  (wire (pts (xy 227.7325 89.535) (xy 299.085 89.535))
+  (wire (pts (xy 231.775 89.535) (xy 299.085 89.535))
     (stroke (width 0) (type default))
   )
@@
     (stroke (width 0) (type default))
   )
-  (wire (pts (xy 110.49 102.87) (xy 226.4625 102.87))
+  (wire (pts (xy 110.49 102.87) (xy 227.965 102.87))
     (stroke (width 0) (type default))
   )
@@
     (stroke (width 0) (type default))
   )
-  (wire (pts (xy 225.1925 97.79) (xy 225.1925 79.375))
+  (wire (pts (xy 224.155 97.79) (xy 224.155 79.375))
     (stroke (width 0) (type default))
   )
@@
     (stroke (width 0) (type default))
   )
-  (wire (pts (xy 110.49 105.41) (xy 227.0975 105.41))
+  (wire (pts (xy 110.49 105.41) (xy 229.87 105.41))
     (stroke (width 0) (type default))
   )
@@
     (stroke (width 0) (type default))
   )
-  (wire (pts (xy 110.49 95.25) (xy 224.5575 95.25))
+  (wire (pts (xy 110.49 95.25) (xy 222.25 95.25))
     (stroke (width 0) (type default))
   )
@@
     (stroke (width 0) (type default))
   )
-  (wire (pts (xy 223.9225 74.295) (xy 299.085 74.295))
-    (stroke (width 0) (type default))
-  )
-  (wire (pts (xy 228.6 92.075) (xy 299.085 92.075))
+  (wire (pts (xy 220.345 74.295) (xy 299.085 74.295))
+    (stroke (width 0) (type default))
+  )
+  (wire (pts (xy 233.68 92.075) (xy 299.085 92.075))
     (stroke (width 0) (type default))
   )
@@
     (stroke (width 0) (type default))
   )
-  (wire (pts (xy 225.8275 81.915) (xy 299.085 81.915))
+  (wire (pts (xy 226.06 81.915) (xy 299.085 81.915))
     (stroke (width 0) (type default))
   )
@@
     )
   )
-  (symbol (lib_id "Mad5150_early:Resistor_Network") (at 340.995 149.86 180) (unit 4)
-    (in_bom yes) (on_board yes) (dnp no) (fields_autoplaced)
-    (property "Reference" "RN5" (at 343.535 148.59 0)
+  (symbol (lib_id "Mad5150_early:Resistor_Network_1") (at 340.995 149.86 180) (unit 4)
+    (in_bom yes) (on_board yes) (dnp no) (fields_autoplaced)
+    (property "Reference" "RN5" (at 342.9 148.59 0)
       (effects (font (size 1.27 1.27)) (justify right))
     )
-    (property "Value" "4.7K" (at 343.535 151.13 0)
+    (property "Value" "4.7K" (at 342.9 151.13 0)
       (effects (font (size 1.27 1.27)) (justify right))
     )
@@
       (effects (font (size 1.27 1.27)) hide)
     )
-    (property "Datasheet" "" (at 340.995 149.86 0)
+    (property "Datasheet" "" (at 340.36 150.495 0)
       (effects (font (size 1.27 1.27)) hide)
     )
@@
     )
   )
-  (symbol (lib_id "Mad5150_early:Resistor_Network") (at 213.995 32.385 180) (unit 9)
+  (symbol (lib_id "Mad5150_early:Resistor_Network_1") (at 213.995 32.385 180) (unit 9)
     (in_bom yes) (on_board yes) (dnp no)
     (property "Reference" "RN5" (at 215.9 31.115 0)
@@
       (effects (font (size 1.27 1.27)) hide)
     )
-    (property "Datasheet" "" (at 213.995 32.385 0)
+    (property "Datasheet" "" (at 213.36 33.02 0)
       (effects (font (size 1.27 1.27)) hide)
     )
@@
     )
   )
-  (symbol (lib_id "Mad5150_early:Resistor_Network") (at 160.02 34.29 180) (unit 8)
-    (in_bom yes) (on_board yes) (dnp no) (fields_autoplaced)
-    (property "Reference" "RN5" (at 163.83 33.02 0)
+  (symbol (lib_id "Mad5150_early:Resistor_Network_1") (at 160.02 34.29 180) (unit 8)
+    (in_bom yes) (on_board yes) (dnp no) (fields_autoplaced)
+    (property "Reference" "RN5" (at 162.56 33.02 0)
       (effects (font (size 1.27 1.27)) (justify right))
     )
-    (property "Value" "4.7K" (at 163.83 35.56 0)
+    (property "Value" "4.7K" (at 162.56 35.56 0)
       (effects (font (size 1.27 1.27)) (justify right))
     )
@@
       (effects (font (size 1.27 1.27)) hide)
     )
-    (property "Datasheet" "" (at 160.02 34.29 0)
+    (property "Datasheet" "" (at 159.385 34.925 0)
       (effects (font (size 1.27 1.27)) hide)
     )
@@
     )
   )
-  (symbol (lib_id "Mad5150_early:Resistor_Network") (at 204.47 32.385 180) (unit 11)
+  (symbol (lib_id "Mad5150_early:Resistor_Network_1") (at 204.47 32.385 180) (unit 11)
     (in_bom yes) (on_board yes) (dnp no)
     (property "Reference" "RN5" (at 206.375 31.115 0)
@@
       (effects (font (size 1.27 1.27)) hide)
     )
-    (property "Datasheet" "" (at 204.47 32.385 0)
+    (property "Datasheet" "" (at 203.835 33.02 0)
       (effects (font (size 1.27 1.27)) hide)
     )
@@
     )
   )
-  (symbol (lib_id "Mad5150_early:Resistor_Network") (at 350.52 149.86 180) (unit 3)
+  (symbol (lib_id "Mad5150_early:Resistor_Network_1") (at 350.52 149.86 180) (unit 3)
     (in_bom yes) (on_board yes) (dnp no) (fields_autoplaced)
     (property "Reference" "RN5" (at 353.06 148.59 0)
@@
       (effects (font (size 1.27 1.27)) hide)
     )
-    (property "Datasheet" "" (at 350.52 149.86 0)
-      (effects (font (size 1.27 1.27)) hide)
-    )
+    (property "Datasheet" "" (at 349.885 150.495 0)
+      (effects (font (size 1.27 1.27)) hide)
+    )

Commit message: Begin tracing
Parts:
- C2, C4, C7, C9: footprint madXT_early:Cap_unipolar_3pin -> madXT_early:cap_unipolar
Changed lines of the file:
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@@
       (effects (font (size 1.27 1.27)) (justify left))
     )
-    (property "Footprint" "madXT_early:Cap_unipolar_3pin" (at 359.7402 180.34 0)
+    (property "Footprint" "madXT_early:cap_unipolar" (at 359.7402 180.34 0)
       (effects (font (size 1.27 1.27)) hide)
     )
@@
       (effects (font (size 1.27 1.27)) (justify left))
     )
-    (property "Footprint" "madXT_early:Cap_unipolar_3pin" (at 348.3102 180.34 0)
+    (property "Footprint" "madXT_early:cap_unipolar" (at 348.3102 180.34 0)
       (effects (font (size 1.27 1.27)) hide)
     )
@@
       (effects (font (size 1.27 1.27)) (justify left))
     )
-    (property "Footprint" "madXT_early:Cap_unipolar_3pin" (at 336.8802 180.34 0)
+    (property "Footprint" "madXT_early:cap_unipolar" (at 336.8802 180.34 0)
       (effects (font (size 1.27 1.27)) hide)
     )
@@
       (effects (font (size 1.27 1.27)) (justify left))
     )
-    (property "Footprint" "madXT_early:Cap_unipolar_3pin" (at 375.6152 183.515 0)
-      (effects (font (size 1.27 1.27)) hide)
-    )
+    (property "Footprint" "madXT_early:cap_unipolar" (at 375.6152 183.515 0)
+      (effects (font (size 1.27 1.27)) hide)
+    )

Commit message: Tracing finished
Parts:
- C2, C4, C7, C9: footprint madXT_early:cap_unipolar -> mad5150:cap_unipolar
- J9: footprint madXT_early:Keyboard -> mad5150:Keyboard
- PB3: footprint Connector_PinHeader_2.54mm:PinHeader_1x03_P2.54mm_Vertical -> mad5150:PinHeader_1x03_P2.54mm_Vertical
- RN2, RN5, U21: footprint Package_DIP:DIP-16_W7.62mm -> mad5150:DIP-16_W7.62mm
- SW1: footprint madXT_early:DIP_SWITCH -> mad5150:DIP_SWITCH
- U27, U41: footprint Package_DIP:DIP-20_W7.62mm -> mad5150:DIP-20_W7.62mm
- U29: footprint Package_DIP:DIP-40_W15.24mm -> mad5150:DIP-40_W15.24mm
- U68, U70, U71, U89: footprint Package_DIP:DIP-14_W7.62mm -> mad5150:DIP-14_W7.62mm
- U85: footprint Package_DIP:DIP-8_W7.62mm -> mad5150:DIP-8_W7.62mm

Commit message: Gerbers
Parts:
- U70: value S74_U70 -> 74S74N
Changed lines of the file:
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@@
       (effects (font (size 1.27 1.27)) (justify left))
     )
-    (property "Value" "S74_U70" (at 307.975 121.92 0)
+    (property "Value" "74S74N" (at 307.975 121.92 0)
       (effects (font (size 1.27 1.27)) (justify left))
     )
