File: supporting_prj/Adlib card/Adlib.kicad_pcb (KiCad board)
At the start: 2 copper layers, 135.3 x 106.7 mm, 61 parts, among them J1 CONN_01X05, P1 IRQ, P2 ADDR, Q1 2N3904, U1 74LS109, U2 74LS138, U3 74LS138, U4 74LS245, U5 74LS04, U6 YM3812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

Commit message: Tracing for version 1.0 finished
Other:
- rule pad_to_mask_clearance: 0.2 -> 0
- board text added: "Ad Lib Inc. (replica)"
- board text added: "Ad Lib Replica Project by schlae Made by MadCat 2024"
- board text removed: "Replica of 1990 Ad Lib"
