File: supporting_prj/RNDip16/rndip16.kicad_pcb (KiCad board)
At the start: 2 copper layers, 24.4 x 21 mm, 27 parts, among them J1 Conn_01x16_Pin, J2 Conn_01x16_Pin

Commit message: Tracing for version 1.0 finished
Other:
- board text added: "Resistor network replacement MadCat 2024"
